File: brain/uc.sch (KiCad schematic (older format))
At the start: 33 parts

Commit message: updated schematic of brain board
Parts:
- added LED0, LED1, LED2, LED3: LED, symbol LED
- added R? (x4): 220, symbol R
- gave numbers to parts that had none: 1
Connections:
- net labels added: ANA_CH0_0_3v3, ANA_CH1_0_3v3, ANA_CH2_0_3v3, ANA_CH3_0_3v3, ANA_CH4_0_3v3, AX12_RX_3v3, AX12_TX_3v3, COLOR_3v3, GPIO0_3v3, GPIO10_3v3, GPIO11_3v3, GPIO1_3v3, GPIO2_3v3, GPIO3_3v3, GPIO4_3v3, GPIO5_3v3, GPIO6_3v3, GPIO7_3v3, GPIO8_3v3, GPIO9_3v3, GPIO_SHIFT_OE_3v3, GPIO_SHIFT_STCP_3v3, LED0_3v3, LED1_3v3, LED2_3v3, LED3_3v3, SLA_RX_3v3, SLA_TX_3v3, STARTER_3v3, US_CH0_E_3v3, US_CH0_T_3v3, US_CH1_E_3v3, US_CH1_T_3v3, US_CH2_E_3v3, US_CH2_T_3v3, US_CH3_E_3v3, US_CH3_T_3v3
- net labels removed: POS_SPI_CSEL_3v3, POS_SPI_CSER_3v3
- wire segments 146 -> 198
Other:
- note added: "UART1: dbg\nUART2: slave\nUART3: ax12\nSPI2: position\nSPI3: slave\nI2C1: servo\nTIM3: US ch2\nTIM4: US ch3\nTIM9: motor\nTIM10: US ch0\nTIM11: US ch1"
- moved on the sheet: R?

Commit message: footprint assignation
Parts:
- removed U?: STM32F407VG, TQFP100, symbol STM32F407VG
- added U8: STM32F407VG, Housings_QFP:LQFP-100_14x14mm_Pitch0.5mm, symbol STM32F407VG
- BOOT0, BOOT1: footprint (none) -> Pin_Headers:Pin_Header_Straight_1x02
- JTAG1: renamed from JTAG; footprint (none) -> espitall:HE10_20D
- LED0, LED1, LED2, LED3: footprint (none) -> LEDs:LED-0603
- R30, R31, R32, R33: renamed from R?; footprint (none) -> Resistors_SMD:R_0603
- UART_DBG1: renamed from UART_DBG; footprint (none) -> Sockets_MOLEX_KK-System:Socket_MOLEX-KK-RM2-54mm_Lock_5pin_straight
- Y1: renamed from Y?; footprint (none) -> Crystals:Crystal_HC49-SD_SMD
- gave numbers to parts that had none: 27
Connections:
- no-connect marks 0 -> 6

Commit message: all tracks are routed
Parts:
- removed LED3: LED, LEDs:LED-0603, symbol LED
- removed R33: 220, Resistors_SMD:R_0603, symbol R
Connections:
- net labels removed: LED3_3v3
- wire segments 198 -> 193
- no-connect marks 6 -> 4

Commit message: Brain 2018 layout
Parts:
- BOOT0, BOOT1: footprint Pin_Headers:Pin_Header_Straight_1x02 -> Pin_Headers:Pin_Header_Straight_1x02_Pitch2.54mm
- C70, C71, C72, C73, C74, C75, C76, C77, C78, C79, C80, C81, C82, C83, C84, C85, C86: symbol C -> C-RESCUE-brain
- LED0, LED1, LED2: symbol LED -> LED-RESCUE-brain
- R29, R30, R31, R32, R34, R35, R36, R37, R38, R39, R40, R41, R42: symbol R -> R-RESCUE-brain
Connections:
- net labels added: DCM_DIR_0_3v3, DCM_DIR_1_3v3, DCM_PWM_0_3v3, DCM_PWM_1_3v3
- net labels removed: AX12_RX_3v3, AX12_TX_3v3
- wire segments 193 -> 195
- no-connect marks 4 -> 3
Other:
- note added: "UART1: dbg\nUART2: slave\nUART3: ax12\nSPI2: position\nSPI3: slave\nI2C1: servo\nTIM2: DC motor\nTIM3: US ch2\nTIM4: US ch3\nTIM9: motor\nTIM10: US ch0\nTIM11: US ch1"
- note removed: "UART1: dbg\nUART2: slave\nUART3: ax12\nSPI2: position\nSPI3: slave\nI2C1: servo\nTIM3: US ch2\nTIM4: US ch3\nTIM9: motor\nTIM10: US ch0\nTIM11: US ch1"

Commit message: change shift register connector to match Cocoout and Cocoin
Connections:
- net labels added: GPIO_SHIFT_LOAD_3v3, GPIO_SHIFT_SET_3v3
- net labels removed: GPIO_SHIFT_OE_3v3, GPIO_SHIFT_STCP_3v3

Commit message: add 3d step files to brain
Parts:
- BOOT0, BOOT1: footprint Pin_Headers:Pin_Header_Straight_1x02_Pitch2.54mm -> espitall:Pin_Header_Straight_1x02_Pitch2.54mm
- C70, C71, C72, C73, C74, C75, C76, C77, C78, C79, C80, C81, C82, C83, C84, C85, C86: footprint Capacitors_SMD:C_0603 -> espitall:C_0603
- LED0, LED1, LED2: footprint LEDs:LED-0603 -> espitall:LED-0603
- R29, R30, R31, R32, R34, R35, R36, R37, R38, R39, R40, R41, R42: footprint Resistors_SMD:R_0603 -> espitall:R_0603
- U8: footprint Housings_QFP:LQFP-100_14x14mm_Pitch0.5mm -> espitall:LQFP-100_14x14mm_Pitch0.5mm
- UART_DBG1: footprint Sockets_MOLEX_KK-System:Socket_MOLEX-KK-RM2-54mm_Lock_5pin_straight -> espitall:Socket_MOLEX-KK-RM2-54mm_Lock_5pin_straight
- Y1: footprint Crystals:Crystal_HC49-SD_SMD -> espitall:Crystal_HC49-SD_SMD
Changed lines of the file:
@@
-EESchema Schematic File Version 2
+EESchema Schematic File Version 3
 LIBS:brain-rescue
-LIBS:power
-LIBS:device
-LIBS:transistors
-LIBS:conn
-LIBS:linear
-LIBS:regul
-LIBS:74xx
-LIBS:cmos4000
-LIBS:adc-dac
-LIBS:memory
-LIBS:xilinx
-LIBS:microcontrollers
-LIBS:dsp
-LIBS:microchip
-LIBS:analog_switches
-LIBS:motorola
-LIBS:texas
-LIBS:intel
-LIBS:audio
-LIBS:interface
-LIBS:digital-audio
-LIBS:philips
-LIBS:display
-LIBS:cypress
-LIBS:siliconi
-LIBS:opto
-LIBS:atmel
-LIBS:contrib
-LIBS:valves
 LIBS:espitall
 LIBS:brain-cache
-EELAYER 25 0
+EELAYER 26 0
 EELAYER END
 $Descr A3 16535 11693
@@
 F 0 "C70" H 6425 1750 50  0000 L CNN
 F 1 "4u7" H 6425 1550 50  0000 L CNN
-F 2 "Capacitors_SMD:C_0603" V 6300 1650 30  0001 C CNN
+F 2 "espitall:C_0603" V 6300 1650 30  0001 C CNN
 F 3 "" H 6400 1650 60  0000 C CNN
 	1    6400 1650
@@
 F 0 "C71" H 6725 1750 50  0000 L CNN
 F 1 "100n" H 6725 1550 50  0000 L CNN
-F 2 "Capacitors_SMD:C_0603" V 6600 1650 30  0001 C CNN
+F 2 "espitall:C_0603" V 6600 1650 30  0001 C CNN
 F 3 "" H 6700 1650 60  0000 C CNN
 	1    6700 1650
@@
 F 0 "C85" H 9325 9250 50  0000 L CNN
 F 1 "2u2" H 9325 9050 50  0000 L CNN
-F 2 "Capacitors_SMD:C_0603" V 9200 9150 30  0001 C CNN
+F 2 "espitall:C_0603" V 9200 9150 30  0001 C CNN
 F 3 "" H 9300 9150 60  0000 C CNN
 	1    9300 9150
@@
 F 0 "C86" H 9825 9250 50  0000 L CNN
 F 1 "2u2" H 9825 9050 50  0000 L CNN
-F 2 "Capacitors_SMD:C_0603" V 9700 9150 30  0001 C CNN
+F 2 "espitall:C_0603" V 9700 9150 30  0001 C CNN
 F 3 "" H 9800 9150 60  0000 C CNN
 	1    9800 9150
@@
 F 0 "Y1" H 2650 4100 50  0000 C CNN
 F 1 "8M" H 2650 3800 50  0000 C CNN
-F 2 "Crystals:Crystal_HC49-SD_SMD" H 2650 4100 60  0001 C CNN
+F 2 "espitall:Crystal_HC49-SD_SMD" H 2650 4100 60  0001 C CNN
 F 3 "" H 2650 3950 60  0000 C CNN
 	1    2650 3950
@@
 F 0 "C82" H 2675 4550 50  0000 L CNN
 F 1 "20p" H 2675 4350 50  0000 L CNN
-F 2 "Capacitors_SMD:C_0603" V 2550 4450 30  0001 C CNN
+F 2 "espitall:C_0603" V 2550 4450 30  0001 C CNN
 F 3 "" H 2650 4450 60  0000 C CNN
 	1    2650 4450
@@
 F 0 "C81" H 2375 4550 50  0000 L CNN
 F 1 "20p" H 2375 4350 50  0000 L CNN
-F 2 "Capacitors_SMD:C_0603" V 2250 4450 30  0001 C CNN
+F 2 "espitall:C_0603" V 2250 4450 30  0001 C CNN
 F 3 "" H 2350 4450 60  0000 C CNN
 	1    2350 4450
@@
 F 0 "R37" V 3180 4250 50  0000 C CNN
 F 1 "0" V 3100 4250 50  0000 C CNN
-F 2 "Resistors_SMD:R_0603" V 3030 4250 30  0001 C CNN
+F 2 "espitall:R_0603" V 3030 4250 30  0001 C CNN
 F 3 "" H 3100 4250 30  0000 C CNN
 	1    3100 4250
@@
 F 0 "BOOT0" H 1350 1500 50  0000 C CNN
 F 1 "JUMPER" H 1350 1270 50  0000 C CNN
-F 2 "Pin_Headers:Pin_Header_Straight_1x02_Pitch2.54mm" H 1350 1350 60  0001 C CNN
+F 2 "espitall:Pin_Header_Straight_1x02_Pitch2.54mm" H 1350 1350 60  0001 C CNN
 F 3 "" H 1350 1350 60  0000 C CNN
 	1    1350 1350
@@
 F 0 "BOOT1" H 1750 1500 50  0000 C CNN
 F 1 "JUMPER" H 1750 1270 50  0000 C CNN
-F 2 "Pin_Headers:Pin_Header_Straight_1x02_Pitch2.54mm" H 1750 1350 60  0001 C CNN
+F 2 "espitall:Pin_Header_Straight_1x02_Pitch2.54mm" H 1750 1350 60  0001 C CNN
 F 3 "" H 1750 1350 60  0000 C CNN
 	1    1750 1350
@@
 F 0 "R34" V 1430 2250 50  0000 C CNN
 F 1 "10k" V 1350 2250 50  0000 C CNN
-F 2 "Resistors_SMD:R_0603" V 1280 2250 30  0001 C CNN
+F 2 "espitall:R_0603" V 1280 2250 30  0001 C CNN
 F 3 "" H 1350 2250 30  0000 C CNN
 	1    1350 2250
@@
 F 0 "R35" V 1830 2250 50  0000 C CNN
 F 1 "10k" V 1750 2250 50  0000 C CNN
-F 2 "Resistors_SMD:R_0603" V 1680 2250 30  0001 C CNN
+F 2 "espitall:R_0603" V 1680 2250 30  0001 C CNN
 F 3 "" H 1750 2250 30  0000 C CNN
 	1    1750 2250
@@
 F 0 "R40" V 3030 10750 50  0000 C CNN
 F 1 "10k" V 2950 10750 50  0000 C CNN
-F 2 "Resistors_SMD:R_0603" V 2880 10750 30  0001 C CNN
+F 2 "espitall:R_0603" V 2880 10750 30  0001 C CNN
 F 3 "" H 2950 10750 30  0000 C CNN
 	1    2950 10750
@@
 F 0 "R41" V 3280 10750 50  0000 C CNN
 F 1 "10k" V 3200 10750 50  0000 C CNN
-F 2 "Resistors_SMD:R_0603" V 3130 10750 30  0001 C CNN
+F 2 "espitall:R_0603" V 3130 10750 30  0001 C CNN
 F 3 "" H 3200 10750 30  0000 C CNN
 	1    3200 10750
@@
 F 0 "R42" V 3530 10750 50  0000 C CNN
 F 1 "10k" V 3450 10750 50  0000 C CNN
-F 2 "Resistors_SMD:R_0603" V 3380 10750 30  0001 C CNN
+F 2 "espitall:R_0603" V 3380 10750 30  0001 C CNN
 F 3 "" H 3450 10750 30  0000 C CNN
 	1    3450 10750
@@
 F 0 "C72" H 7025 1750 50  0000 L CNN
 F 1 "100n" H 7025 1550 50  0000 L CNN
-F 2 "Capacitors_SMD:C_0603" V 6900 1650 30  0001 C CNN
+F 2 "espitall:C_0603" V 6900 1650 30  0001 C CNN
 F 3 "" H 7000 1650 60  0000 C CNN
 	1    7000 1650
@@
 F 0 "C73" H 7325 1750 50  0000 L CNN
 F 1 "100n" H 7325 1550 50  0000 L CNN
-F 2 "Capacitors_SMD:C_0603" V 7200 1650 30  0001 C CNN
+F 2 "espitall:C_0603" V 7200 1650 30  0001 C CNN
 F 3 "" H 7300 1650 60  0000 C CNN
 	1    7300 1650
@@
 F 0 "C74" H 7625 1750 50  0000 L CNN
 F 1 "100n" H 7625 1550 50  0000 L CNN
-F 2 "Capacitors_SMD:C_0603" V 7500 1650 30  0001 C CNN
+F 2 "espitall:C_0603" V 7500 1650 30  0001 C CNN
 F 3 "" H 7600 1650 60  0000 C CNN
 	1    7600 1650
@@
 F 0 "C75" H 7925 1750 50  0000 L CNN
 F 1 "100n" H 7925 1550 50  0000 L CNN
-F 2 "Capacitors_SMD:C_0603" V 7800 1650 30  0001 C CNN
+F 2 "espitall:C_0603" V 7800 1650 30  0001 C CNN
 F 3 "" H 7900 1650 60  0000 C CNN
 	1    7900 1650
@@
 F 0 "C76" H 8225 1750 50  0000 L CNN
 F 1 "100n" H 8225 1550 50  0000 L CNN
-F 2 "Capacitors_SMD:C_0603" V 8100 1650 30  0001 C CNN
+F 2 "espitall:C_0603" V 8100 1650 30  0001 C CNN
 F 3 "" H 8200 1650 60  0000 C CNN
 	1    8200 1650
@@
 F 0 "C77" H 8525 1750 50  0000 L CNN
 F 1 "100n" H 8525 1550 50  0000 L CNN
-F 2 "Capacitors_SMD:C_0603" V 8400 1650 30  0001 C CNN
+F 2 "espitall:C_0603" V 8400 1650 30  0001 C CNN
 F 3 "" H 8500 1650 60  0000 C CNN
 	1    8500 1650
@@
 F 0 "C78" H 8825 1750 50  0000 L CNN
 F 1 "100n" H 8825 1550 50  0000 L CNN
-F 2 "Capacitors_SMD:C_0603" V 8700 1650 30  0001 C CNN
+F 2 "espitall:C_0603" V 8700 1650 30  0001 C CNN
 F 3 "" H 8800 1650 60  0000 C CNN
 	1    8800 1650
@@
 F 0 "C79" H 9125 1750 50  0000 L CNN
 F 1 "100n" H 9125 1550 50  0000 L CNN
-F 2 "Capacitors_SMD:C_0603" V 9000 1650 30  0001 C CNN
+F 2 "espitall:C_0603" V 9000 1650 30  0001 C CNN
 F 3 "" H 9100 1650 60  0000 C CNN
 	1    9100 1650
@@
 F 0 "C80" H 2025 4550 50  0000 L CNN
 F 1 "100n" H 2025 4350 50  0000 L CNN
-F 2 "Capacitors_SMD:C_0603" V 1900 4450 30  0001 C CNN
+F 2 "espitall:C_0603" V 1900 4450 30  0001 C CNN
 F 3 "" H 2000 4450 60  0000 C CNN
 	1    2000 4450
@@
 F 0 "UART_DBG1" H 900 6350 50  0000 C CNN
 F 1 "CONN_01X05" V 1000 6050 50  0000 C CNN
-F 2 "Sockets_MOLEX_KK-System:Socket_MOLEX-KK-RM2-54mm_Lock_5pin_straight" H 900 6050 60  0001 C CNN
+F 2 "espitall:Socket_MOLEX-KK-RM2-54mm_Lock_5pin_straight" H 900 6050 60  0001 C CNN
 F 3 "" H 900 6050 60  0000 C CNN
 	1    900  6050
@@
 F 0 "C83" H 675 5400 50  0000 L CNN
 F 1 "4u7" H 675 5200 50  0000 L CNN
-F 2 "Capacitors_SMD:C_0603" V 550 5300 30  0001 C CNN
+F 2 "espitall:C_0603" V 550 5300 30  0001 C CNN
 F 3 "" H 650 5300 60  0000 C CNN
 	1    650  5300
@@
 F 0 "C84" H 925 5400 50  0000 L CNN
 F 1 "4u7" H 925 5200 50  0000 L CNN
-F 2 "Capacitors_SMD:C_0603" V 800 5300 30  0001 C CNN
+F 2 "espitall:C_0603" V 800 5300 30  0001 C CNN
 F 3 "" H 900 5300 60  0000 C CNN
 	1    900  5300
@@
 F 0 "R38" V 1380 7100 50  0000 C CNN
 F 1 "2k2" V 1300 7100 50  0000 C CNN
-F 2 "Resistors_SMD:R_0603" V 1230 7100 30  0001 C CNN
+F 2 "espitall:R_0603" V 1230 7100 30  0001 C CNN
 F 3 "" H 1300 7100 30  0000 C CNN
 	1    1300 7100
@@
 F 0 "R39" V 1580 7100 50  0000 C CNN
 F 1 "2k2" V 1500 7100 50  0000 C CNN
-F 2 "Resistors_SMD:R_0603" V 1430 7100 30  0001 C CNN
+F 2 "espitall:R_0603" V 1430 7100 30  0001 C CNN
 F 3 "" H 1500 7100 30  0000 C CNN
 	1    1500 7100
@@
 F 0 "R36" V 2880 2300 50  0000 C CNN
 F 1 "1k" V 2800 2300 50  0000 C CNN
-F 2 "Resistors_SMD:R_0603" V 2730 2300 30  0001 C CNN
+F 2 "espitall:R_0603" V 2730 2300 30  0001 C CNN
 F 3 "" H 2800 2300 30  0000 C CNN
 	1    2800 2300
@@
 F 0 "R29" V 2880 1300 50  0000 C CNN
 F 1 "10k" V 2800 1300 50  0000 C CNN
-F 2 "Resistors_SMD:R_0603" V 2730 1300 30  0001 C CNN
+F 2 "espitall:R_0603" V 2730 1300 30  0001 C CNN
 F 3 "" H 2800 1300 30  0000 C CNN
 	1    2800 1300
@@
 F 0 "R30" V 11430 1550 40  0000 C CNN
 F 1 "220" V 11357 1551 40  0000 C CNN
-F 2 "Resistors_SMD:R_0603" V 11280 1550 30  0001 C CNN
+F 2 "espitall:R_0603" V 11280 1550 30  0001 C CNN
 F 3 "" H 11350 1550 30  0000 C CNN
 	1    11350 1550
@@
 F 0 "LED0" H 11350 2200 50  0000 C CNN
 F 1 "LED" H 11350 2000 50  0000 C CNN
-F 2 "LEDs:LED-0603" H 11350 2300 60  0001 C CNN
+F 2 "espitall:LED-0603" H 11350 2300 60  0001 C CNN
 F 3 "" H 11350 2100 60  0000 C CNN
 	1    11350 2100
@@
 F 0 "R31" V 12280 1550 40  0000 C CNN
 F 1 "220" V 12207 1551 40  0000 C CNN
-F 2 "Resistors_SMD:R_0603" V 12130 1550 30  0001 C CNN
+F 2 "espitall:R_0603" V 12130 1550 30  0001 C CNN
 F 3 "" H 12200 1550 30  0000 C CNN
 	1    12200 1550
@@
 F 0 "LED1" H 12200 2200 50  0000 C CNN
 F 1 "LED" H 12200 2000 50  0000 C CNN
-F 2 "LEDs:LED-0603" H 12200 2300 60  0001 C CNN
+F 2 "espitall:LED-0603" H 12200 2300 60  0001 C CNN
 F 3 "" H 12200 2100 60  0000 C CNN
 	1    12200 2100
@@
 F 0 "R32" V 13180 1550 40  0000 C CNN
 F 1 "220" V 13107 1551 40  0000 C CNN
-F 2 "Resistors_SMD:R_0603" V 13030 1550 30  0001 C CNN
+F 2 "espitall:R_0603" V 13030 1550 30  0001 C CNN
 F 3 "" H 13100 1550 30  0000 C CNN
 	1    13100 1550
@@
 F 0 "LED2" H 13100 2200 50  0000 C CNN
 F 1 "LED" H 13100 2000 50  0000 C CNN
-F 2 "LEDs:LED-0603" H 13100 2300 60  0001 C CNN
+F 2 "espitall:LED-0603" H 13100 2300 60  0001 C CNN
 F 3 "" H 13100 2100 60  0000 C CNN
 	1    13100 2100
@@
 F 0 "U8" H 8400 5800 60  0000 C CNN
 F 1 "STM32F407VG" H 8400 5900 60  0000 C CNN
-F 2 "Housings_QFP:LQFP-100_14x14mm_Pitch0.5mm" H 8400 5700 60  0001 C CNN
+F 2 "espitall:LQFP-100_14x14mm_Pitch0.5mm" H 8400 5700 60  0001 C CNN
 F 3 "" H 8400 5800 60  0000 C CNN
 	1    8400 5800
