File: brain/uc.sch (KiCad schematic (older format))
At the start: 39 parts, among them U8 STM32F407VG, Y1 8M

Commit message: add module add footprint SPSGRF-868 for future com board
Parts:
- BOOT0, BOOT1: symbol JUMPER -> brain-rescue:JUMPER-RESCUE-brain
- C70, C71, C72, C73, C74, C75, C76, C77, C78, C79, C80, C81, C82, C83, C84, C85, C86: symbol C-RESCUE-brain -> brain-rescue:C-RESCUE-brain
- JTAG1: symbol HE10-20 -> conn:HE10-20
- LED0, LED1, LED2: symbol LED-RESCUE-brain -> brain-rescue:LED-RESCUE-brain
- R29, R30, R31, R32, R34, R35, R36, R37, R38, R39, R40, R41, R42: symbol R-RESCUE-brain -> brain-rescue:R-RESCUE-brain
- U8: symbol STM32F407VG -> espitall:STM32F407VG
- UART_DBG1: symbol CONN_01X05 -> brain-rescue:CONN_01X05-RESCUE-brain
- Y1: symbol Crystal -> device:Crystal
Connections:
- wire segments 195 -> 236
