File: brain/DC_motor.sch (KiCad schematic (older format))
At the start: 2 parts

Commit message: add 3d step files to brain
Parts:
- C30: footprint Capacitors_SMD:C_0603 -> espitall:C_0603
- DCM0: footprint Sockets_MOLEX_KK-System:Socket_MOLEX-KK-RM2-54mm_Lock_5pin_straight -> espitall:Socket_MOLEX-KK-RM2-54mm_Lock_5pin_straight
Changed lines of the file:
@@
-EESchema Schematic File Version 2
+EESchema Schematic File Version 3
 LIBS:brain-rescue
-LIBS:power
-LIBS:device
-LIBS:transistors
-LIBS:conn
-LIBS:linear
-LIBS:regul
-LIBS:74xx
-LIBS:cmos4000
-LIBS:adc-dac
-LIBS:memory
-LIBS:xilinx
-LIBS:microcontrollers
-LIBS:dsp
-LIBS:microchip
-LIBS:analog_switches
-LIBS:motorola
-LIBS:texas
-LIBS:intel
-LIBS:audio
-LIBS:interface
-LIBS:digital-audio
-LIBS:philips
-LIBS:display
-LIBS:cypress
-LIBS:siliconi
-LIBS:opto
-LIBS:atmel
-LIBS:contrib
-LIBS:valves
 LIBS:espitall
 LIBS:brain-cache
-EELAYER 25 0
+EELAYER 26 0
 EELAYER END
 $Descr A4 11693 8268
@@
 F 0 "DCM0" V 8200 3300 50  0000 C CNN
 F 1 "CONN_5" V 8300 3300 50  0000 C CNN
-F 2 "Sockets_MOLEX_KK-System:Socket_MOLEX-KK-RM2-54mm_Lock_5pin_straight" H 8250 3300 60  0001 C CNN
+F 2 "espitall:Socket_MOLEX-KK-RM2-54mm_Lock_5pin_straight" H 8250 3300 60  0001 C CNN
 F 3 "" H 8250 3300 60  0000 C CNN
 	1    8250 3300
@@
 F 0 "C30" H 8600 3400 40  0000 L CNN
 F 1 "4u7" H 8606 3215 40  0000 L CNN
-F 2 "Capacitors_SMD:C_0603" H 8638 3150 30  0001 C CNN
+F 2 "espitall:C_0603" H 8638 3150 30  0001 C CNN
 F 3 "" H 8600 3300 60  0000 C CNN
 	1    8600 3300

Commit message: add module add footprint SPSGRF-868 for future com board
Parts:
- C30: symbol C-RESCUE-brain -> brain-rescue:C-RESCUE-brain
- DCM0: symbol CONN_5 -> brain-rescue:CONN_5-RESCUE-brain
Changed lines of the file:
@@
-EESchema Schematic File Version 3
-LIBS:brain-rescue
-LIBS:espitall
+EESchema Schematic File Version 4
 LIBS:brain-cache
 EELAYER 26 0
@@
 	6950 4700 4000 4700
 $Comp
-L CONN_5 DCM0
+L brain-rescue:CONN_5-RESCUE-brain DCM0
 U 1 1 592BFB9E
 P 8250 3300
@@
 	7150 3400 7150 5000
 $Comp
-L GND-RESCUE-brain #PWR0225
+L brain-rescue:GND-RESCUE-brain #PWR0225
 U 1 1 592BFBAB
 P 7800 3700
@@
 $EndComp
 $Comp
-L +5V #PWR0226
+L power:+5V #PWR0226
 U 1 1 592BFBB1
 P 7800 2850
@@
 $EndComp
 $Comp
-L C-RESCUE-brain C30
+L brain-rescue:C-RESCUE-brain C30
 U 1 1 592BFBB7
 P 8600 3300
@@
 $EndComp
 $Comp
-L GND-RESCUE-brain #PWR0227
+L brain-rescue:GND-RESCUE-brain #PWR0227
 U 1 1 592BFBBE
 P 8600 3700
@@
 	7800 3500 7800 3700
 $Comp
-L GND-RESCUE-brain #PWR0228
+L brain-rescue:GND-RESCUE-brain #PWR0228
 U 1 1 592BFBD3
 P 7800 4950
@@
 $EndComp
 $Comp
-L +5V #PWR0229
+L power:+5V #PWR0229
 U 1 1 592BFBD9
 P 7800 4100
@@
 $EndComp
 $Comp
-L GND-RESCUE-brain #PWR0230
+L brain-rescue:GND-RESCUE-brain #PWR0230
 U 1 1 592BFBE6
 P 8600 4950
