File: brain/Servo.sch (KiCad schematic (older format))
At the start: 57 parts

Commit message: footprint assignation
Parts:
- AX12, S0, S1, S10, S11, S12, S13, S14, S15, S16, S3, S4, S5, S6, S7, S8, S9: footprint (none) -> Sockets_MOLEX_KK-System:Socket_MOLEX-KK-RM2-54mm_Lock_3pin_straight
- AX12PWR1: renamed from AX12PWR; footprint (none) -> Sockets_MOLEX_KK-System:Socket_MOLEX-KK-RM2-54mm_Lock_2pin_straight
- C35, C36, C37, C38, C39, C40, C41, C42, C43, C44, C45, C46, C47, C48, C49, C50, C51, C52, C53, C54, C55, C56: renamed from C?; footprint (none) -> Capacitors_SMD:C_0603
- D1: renamed from D?; value DIODE -> 1N4148W; footprint (none) -> Diodes_SMD:SOD-123
- I2C3v3: footprint (none) -> Sockets_MOLEX_KK-System:Socket_MOLEX-KK-RM2-54mm_Lock_5pin_straight
- I2C5V1: renamed from I2C5V; footprint (none) -> Sockets_MOLEX_KK-System:Socket_MOLEX-KK-RM2-54mm_Lock_4pin_straight
- R10, R11, R12, R13, R14, R15, R16, R9: renamed from R?; footprint (none) -> Resistors_SMD:R_0603
- SPWR0, SPWR1, SPWR2, SPWR3: footprint (none) -> Sockets_MOLEX_KK-System:Socket_MOLEX-KK-RM2-54mm_Lock_2pin_straight
- U5: renamed from U?; footprint (none) -> Power_Integrations:SO-8
- U6: renamed from U?; footprint (none) -> Housings_SSOP:TSSOP-28_4.4x9.7mm_Pitch0.65mm

Commit message: all tracks are routed
Parts:
- removed C35, C36, C37, C38, C42, C43, C44, C45, C48, C49, C50, C51, C53, C54, C55, C56: 4u7, Capacitors_SMD:C_0603, symbol C
- removed R13, R14, R16, R9: NC, Resistors_SMD:R_0603, symbol R
- removed S0, S1, S10, S11, S12, S13, S14, S15, S16, S3, S4, S5, S6, S7, S8, S9: CONN_3, Sockets_MOLEX_KK-System:Socket_MOLEX-KK-RM2-54mm_Lock_3pin_straight, symbol CONN_3
- removed SPWR0, SPWR1, SPWR2, SPWR3: CONN_2, Sockets_MOLEX_KK-System:Socket_MOLEX-KK-RM2-54mm_Lock_2pin_straight, symbol CONN_2
- added PWM1: HE10-20, espitall:HE10_20D, symbol HE10-20
Connections:
- net labels removed: S0_5V, S10_5V, S11_5V, S12_5V, S13_5V, S14_5V, S15_5V, S1_5V, S2_5V, S3_5V, S4_5V, S5_5V, S6_5V, S7_5V, S8_5V, S9_5V
- wire segments 257 -> 147

Commit message: Brain 2018 layout
Parts:
- removed AX12: CONN_3, Sockets_MOLEX_KK-System:Socket_MOLEX-KK-RM2-54mm_Lock_3pin_straight, symbol CONN_3
- removed AX12PWR1: CONN_2, Sockets_MOLEX_KK-System:Socket_MOLEX-KK-RM2-54mm_Lock_2pin_straight, symbol CONN_2
- removed D1: 1N4148W, Diodes_SMD:SOD-123, symbol DIODE
- removed PWM1: HE10-20, espitall:HE10_20D, symbol HE10-20
- removed R15: 1k, Resistors_SMD:R_0603, symbol R
- added SERVO_0-3, SERVO_4-7, SERVO_8-13: CONN_5, Sockets_MOLEX_KK-System:Socket_MOLEX-KK-RM2-54mm_Lock_5pin_straight, symbol CONN_5
- C39, C40, C41, C46, C47, C52: symbol C -> C-RESCUE-brain
- R10, R11, R12: symbol R -> R-RESCUE-brain
Connections:
- net labels removed: AX12_RX_5v, AX12_TX_5v
- wire segments 147 -> 102

Commit message: add 3d step files to brain
Parts:
- C39, C40, C41, C46, C47, C52: footprint Capacitors_SMD:C_0603 -> espitall:C_0603
- I2C3v3, SERVO_0-3, SERVO_4-7, SERVO_8-13: footprint Sockets_MOLEX_KK-System:Socket_MOLEX-KK-RM2-54mm_Lock_5pin_straight -> espitall:Socket_MOLEX-KK-RM2-54mm_Lock_5pin_straight
- I2C5V1: footprint Sockets_MOLEX_KK-System:Socket_MOLEX-KK-RM2-54mm_Lock_4pin_straight -> espitall:Socket_MOLEX-KK-RM2-54mm_Lock_4pin_straight
- R10, R11, R12: footprint Resistors_SMD:R_0603 -> espitall:R_0603
- U5: footprint Power_Integrations:SO-8 -> espitall:SO-8
- U6: footprint Housings_SSOP:TSSOP-28_4.4x9.7mm_Pitch0.65mm -> espitall:TSSOP-28_4.4x9.7mm_Pitch0.65mm
Changed lines of the file:
@@
-EESchema Schematic File Version 2
+EESchema Schematic File Version 3
 LIBS:brain-rescue
-LIBS:power
-LIBS:device
-LIBS:transistors
-LIBS:conn
-LIBS:linear
-LIBS:regul
-LIBS:74xx
-LIBS:cmos4000
-LIBS:adc-dac
-LIBS:memory
-LIBS:xilinx
-LIBS:microcontrollers
-LIBS:dsp
-LIBS:microchip
-LIBS:analog_switches
-LIBS:motorola
-LIBS:texas
-LIBS:intel
-LIBS:audio
-LIBS:interface
-LIBS:digital-audio
-LIBS:philips
-LIBS:display
-LIBS:cypress
-LIBS:siliconi
-LIBS:opto
-LIBS:atmel
-LIBS:contrib
-LIBS:valves
 LIBS:espitall
 LIBS:brain-cache
-EELAYER 25 0
+EELAYER 26 0
 EELAYER END
 $Descr A4 11693 8268
@@
 F 0 "C39" H 2300 1600 40  0000 L CNN
 F 1 "100n" H 2306 1415 40  0000 L CNN
-F 2 "Capacitors_SMD:C_0603" H 2338 1350 30  0001 C CNN
+F 2 "espitall:C_0603" H 2338 1350 30  0001 C CNN
 F 3 "" H 2300 1500 60  0000 C CNN
 	1    2300 1500
@@
 F 0 "C40" H 3150 1600 40  0000 L CNN
 F 1 "100n" H 3156 1415 40  0000 L CNN
-F 2 "Capacitors_SMD:C_0603" H 3188 1350 30  0001 C CNN
+F 2 "espitall:C_0603" H 3188 1350 30  0001 C CNN
 F 3 "" H 3150 1500 60  0000 C CNN
 	1    3150 1500
@@
 F 0 "R10" V 2980 1150 40  0000 C CNN
 F 1 "200k" V 2907 1151 40  0000 C CNN
-F 2 "Resistors_SMD:R_0603" V 2830 1150 30  0001 C CNN
+F 2 "espitall:R_0603" V 2830 1150 30  0001 C CNN
 F 3 "" H 2900 1150 30  0000 C CNN
 	1    2900 1150
@@
 F 0 "R11" V 3880 1150 40  0000 C CNN
 F 1 "2k2" V 3807 1151 40  0000 C CNN
-F 2 "Resistors_SMD:R_0603" V 3730 1150 30  0001 C CNN
+F 2 "espitall:R_0603" V 3730 1150 30  0001 C CNN
 F 3 "" H 3800 1150 30  0000 C CNN
 	1    3800 1150
@@
 F 0 "R12" V 4080 1150 40  0000 C CNN
 F 1 "2k2" V 4007 1151 40  0000 C CNN
-F 2 "Resistors_SMD:R_0603" V 3930 1150 30  0001 C CNN
+F 2 "espitall:R_0603" V 3930 1150 30  0001 C CNN
 F 3 "" H 4000 1150 30  0000 C CNN
 	1    4000 1150
@@
 F 0 "I2C5V1" V 4550 2400 50  0000 C CNN
 F 1 "CONN_4" V 4650 2400 50  0000 C CNN
-F 2 "Sockets_MOLEX_KK-System:Socket_MOLEX-KK-RM2-54mm_Lock_4pin_straight" H 4600 2400 60  0001 C CNN
+F 2 "espitall:Socket_MOLEX-KK-RM2-54mm_Lock_4pin_straight" H 4600 2400 60  0001 C CNN
 F 3 "" H 4600 2400 60  0000 C CNN
 	1    4600 2400
@@
 F 0 "C41" H 4350 1950 40  0000 L CNN
 F 1 "4u7" H 4356 1765 40  0000 L CNN
-F 2 "Capacitors_SMD:C_0603" H 4388 1700 30  0001 C CNN
+F 2 "espitall:C_0603" H 4388 1700 30  0001 C CNN
 F 3 "" H 4350 1850 60  0000 C CNN
 	1    4350 1850
@@
 F 0 "I2C3v3" V 2950 3900 50  0000 C CNN
 F 1 "CONN_5" V 3050 3900 50  0000 C CNN
-F 2 "Sockets_MOLEX_KK-System:Socket_MOLEX-KK-RM2-54mm_Lock_5pin_straight" H 3000 3900 60  0001 C CNN
+F 2 "espitall:Socket_MOLEX-KK-RM2-54mm_Lock_5pin_straight" H 3000 3900 60  0001 C CNN
 F 3 "" H 3000 3900 60  0000 C CNN
 	1    3000 3900
@@
 F 0 "C47" H 2650 3500 40  0000 L CNN
 F 1 "4u7" H 2656 3315 40  0000 L CNN
-F 2 "Capacitors_SMD:C_0603" H 2688 3250 30  0001 C CNN
+F 2 "espitall:C_0603" H 2688 3250 30  0001 C CNN
 F 3 "" H 2650 3400 60  0000 C CNN
 	1    2650 3400
@@
 F 0 "C46" H 2100 3500 40  0000 L CNN
 F 1 "4u7" H 2106 3315 40  0000 L CNN
-F 2 "Capacitors_SMD:C_0603" H 2138 3250 30  0001 C CNN
+F 2 "espitall:C_0603" H 2138 3250 30  0001 C CNN
 F 3 "" H 2100 3400 60  0000 C CNN
 	1    2100 3400
@@
 F 0 "U5" H 3000 2550 60  0000 C CNN
 F 1 "PCA9306" H 3000 1900 60  0000 C CNN
-F 2 "Power_Integrations:SO-8" H 2750 2250 60  0001 C CNN
+F 2 "espitall:SO-8" H 2750 2250 60  0001 C CNN
 F 3 "" H 2750 2250 60  0000 C CNN
 	1    2750 2250
@@
 F 0 "U6" H 4150 7350 60  0000 C CNN
 F 1 "PCA9685" H 3900 6450 60  0000 C CNN
-F 2 "Housings_SSOP:TSSOP-28_4.4x9.7mm_Pitch0.65mm" H 3900 6450 60  0001 C CNN
+F 2 "espitall:TSSOP-28_4.4x9.7mm_Pitch0.65mm" H 3900 6450 60  0001 C CNN
 F 3 "" H 3900 6450 60  0000 C CNN
 	1    3900 6450
@@
 F 0 "C52" H 3050 5250 40  0000 L CNN
 F 1 "100n" H 3056 5065 40  0000 L CNN
-F 2 "Capacitors_SMD:C_0603" H 3088 5000 30  0001 C CNN
+F 2 "espitall:C_0603" H 3088 5000 30  0001 C CNN
 F 3 "" H 3050 5150 60  0000 C CNN
 	1    3050 5150
@@
 F 0 "SERVO_0-3" V 10450 2900 50  0000 C CNN
 F 1 "CONN_5" V 10550 2900 50  0000 C CNN
-F 2 "Sockets_MOLEX_KK-System:Socket_MOLEX-KK-RM2-54mm_Lock_5pin_straight" H 10500 2900 60  0001 C CNN
+F 2 "espitall:Socket_MOLEX-KK-RM2-54mm_Lock_5pin_straight" H 10500 2900 60  0001 C CNN
 F 3 "" H 10500 2900 60  0000 C CNN
 	1    10500 2900
@@
 F 0 "SERVO_4-7" V 10450 3500 50  0000 C CNN
 F 1 "CONN_5" V 10550 3500 50  0000 C CNN
-F 2 "Sockets_MOLEX_KK-System:Socket_MOLEX-KK-RM2-54mm_Lock_5pin_straight" H 10500 3500 60  0001 C CNN
+F 2 "espitall:Socket_MOLEX-KK-RM2-54mm_Lock_5pin_straight" H 10500 3500 60  0001 C CNN
 F 3 "" H 10500 3500 60  0000 C CNN
 	1    10500 3500
@@
 F 0 "SERVO_8-13" V 10450 4100 50  0000 C CNN
 F 1 "CONN_5" V 10550 4100 50  0000 C CNN
-F 2 "Sockets_MOLEX_KK-System:Socket_MOLEX-KK-RM2-54mm_Lock_5pin_straight" H 10500 4100 60  0001 C CNN
+F 2 "espitall:Socket_MOLEX-KK-RM2-54mm_Lock_5pin_straight" H 10500 4100 60  0001 C CNN
 F 3 "" H 10500 4100 60  0000 C CNN
 	1    10500 4100

Commit message: add module add footprint SPSGRF-868 for future com board
Parts:
- C39, C40, C41, C46, C47, C52: symbol C-RESCUE-brain -> brain-rescue:C-RESCUE-brain
- I2C3v3, SERVO_0-3, SERVO_4-7, SERVO_8-13: symbol CONN_5 -> brain-rescue:CONN_5-RESCUE-brain
- I2C5V1: symbol CONN_4 -> brain-rescue:CONN_4-RESCUE-brain
- R10, R11, R12: symbol R-RESCUE-brain -> brain-rescue:R-RESCUE-brain
- U5: symbol PCA9306 -> brain-rescue:PCA9306-RESCUE-brain
- U6: symbol PCA9685 -> espitall:PCA9685
Changed lines of the file:
@@
-EESchema Schematic File Version 3
-LIBS:brain-rescue
-LIBS:espitall
+EESchema Schematic File Version 4
 LIBS:brain-cache
 EELAYER 26 0
@@
 $EndDescr
 $Comp
-L +3V3 #PWR097
+L power:+3V3 #PWR097
 U 1 1 5563D19B
 P 2600 1100
@@
 $EndComp
 $Comp
-L +5V #PWR098
+L power:+5V #PWR098
 U 1 1 5563D1B0
 P 2900 750
@@
 $EndComp
 $Comp
-L C-RESCUE-brain C39
+L brain-rescue:C-RESCUE-brain C39
 U 1 1 5563D1C5
 P 2300 1500
@@
 $EndComp
 $Comp
-L C-RESCUE-brain C40
+L brain-rescue:C-RESCUE-brain C40
 U 1 1 5563D21A
 P 3150 1500
@@
 $EndComp
 $Comp
-L GND-RESCUE-brain #PWR099
+L brain-rescue:GND-RESCUE-brain #PWR099
 U 1 1 5563D286
 P 2300 1700
@@
 $EndComp
 $Comp
-L GND-RESCUE-brain #PWR0100
+L brain-rescue:GND-RESCUE-brain #PWR0100
 U 1 1 5563D29D
 P 3150 1700
@@
 $EndComp
 $Comp
-L GND-RESCUE-brain #PWR0101
+L brain-rescue:GND-RESCUE-brain #PWR0101
 U 1 1 5563D2B4
 P 2750 2850
@@
 I2C_SDA_3v3
 $Comp
-L R-RESCUE-brain R10
+L brain-rescue:R-RESCUE-brain R10
 U 1 1 5563E278
 P 2900 1150
@@
 I2C_SDA_5v
 $Comp
-L R-RESCUE-brain R11
+L brain-rescue:R-RESCUE-brain R11
 U 1 1 5563E346
 P 3800 1150
@@
 $EndComp
 $Comp
-L R-RESCUE-brain R12
+L brain-rescue:R-RESCUE-brain R12
 U 1 1 5563E3BC
 P 4000 1150
@@
 $EndComp
 $Comp
-L +5V #PWR0102
+L power:+5V #PWR0102
 U 1 1 5563E3E2
 P 3800 750
@@
 $EndComp
 $Comp
-L +5V #PWR0103
+L power:+5V #PWR0103
 U 1 1 5563E3F9
 P 4000 750
@@
 $EndComp
 $Comp
-L GND-RESCUE-brain #PWR0104
+L brain-rescue:GND-RESCUE-brain #PWR0104
 U 1 1 5563E5FD
 P 4150 2750
@@
 $EndComp
 $Comp
-L CONN_4 I2C5V1
+L brain-rescue:CONN_4-RESCUE-brain I2C5V1
 U 1 1 5563E618
 P 4600 2400
@@
 $EndComp
 $Comp
-L C-RESCUE-brain C41
+L brain-rescue:C-RESCUE-brain C41
 U 1 1 5563E68B
 P 4350 1850
@@
 $EndComp
 $Comp
-L GND-RESCUE-brain #PWR0105
+L brain-rescue:GND-RESCUE-brain #PWR0105
 U 1 1 5563E6BE
 P 4350 2050
@@
 $EndComp
 $Comp
-L +5V #PWR0106
+L power:+5V #PWR0106
 U 1 1 5563E6F3
 P 4150 1550
@@
 $EndComp
 $Comp
-L CONN_5 I2C3v3
+L brain-rescue:CONN_5-RESCUE-brain I2C3v3
 U 1 1 5563E89C
 P 3000 3900
@@
 $EndComp
 $Comp
-L C-RESCUE-brain C47
+L brain-rescue:C-RESCUE-brain C47
 U 1 1 5563E9B2
 P 2650 3400
@@
 $EndComp
 $Comp
-L GND-RESCUE-brain #PWR0107
+L brain-rescue:GND-RESCUE-brain #PWR0107
 U 1 1 5563E9B8
 P 2650 3600
@@
 $EndComp
 $Comp
-L +5V #PWR0108
+L power:+5V #PWR0108
 U 1 1 5563E9BE
 P 2450 3000
@@
 $EndComp
 $Comp
-L +3V3 #PWR0109
+L power:+3V3 #PWR0109
 U 1 1 5563EA5E
 P 2250 3100
@@
 $EndComp
 $Comp
-L C-RESCUE-brain C46
+L brain-rescue:C-RESCUE-brain C46
 U 1 1 5563EB03
 P 2100 3400
@@
 $EndComp
 $Comp
-L GND-RESCUE-brain #PWR0110
+L brain-rescue:GND-RESCUE-brain #PWR0110
 U 1 1 5563EB8C
 P 2100 3600
@@
 $EndComp
 $Comp
-L GND-RESCUE-brain #PWR0111
+L brain-rescue:GND-RESCUE-brain #PWR0111
 U 1 1 5563ECB8
 P 2500 4200
@@
 $EndComp
 $Comp
-L PCA9306 U5
+L brain-rescue:PCA9306-RESCUE-brain U5
 U 1 1 5563FD6D
 P 2750 2250
@@
 $EndComp
 $Comp
-L PCA9685 U6
+L espitall:PCA9685 U6
 U 1 1 5563FFFB
 P 3900 6450
@@
 $EndComp
 $Comp
-L GND-RESCUE-brain #PWR0112
+L brain-rescue:GND-RESCUE-brain #PWR0112
 U 1 1 5564007E
 P 3900 7500
@@
 $EndComp
 $Comp
-L GND-RESCUE-brain #PWR0113
+L brain-rescue:GND-RESCUE-brain #PWR0113
 U 1 1 556400E9
 P 3050 5400
@@
 $EndComp
 $Comp
-L C-RESCUE-brain C52
+L brain-rescue:C-RESCUE-brain C52
 U 1 1 5564028A
 P 3050 5150
@@
 $EndComp
 $Comp
-L +5V #PWR0114
+L power:+5V #PWR0114
 U 1 1 55640425
 P 3900 4750
@@
 $EndComp
 $Comp
-L GND-RESCUE-brain #PWR0115
+L brain-rescue:GND-RESCUE-brain #PWR0115
 U 1 1 55640885
 P 2950 7500
@@
 $EndComp
 Wire Wire Line
-	2600 1100 2600 1700
+	2600 1100 2600 1200
 Wire Wire Line
 	2300 1300 2300 1200
@@
 	3050 1400 3050 1250
 Wire Wire Line
-	3050 1250 3550 1250
+	3050 1250 3150 1250
 Wire Wire Line
 	3550 1250 3550 2150
@@
 	4150 2550 4250 2550
 Wire Wire Line
-	4150 1550 4150 2250
+	4150 1550 4150 1600
 Wire Wire Line
 	4150 2250 4250 2250
@@
 Connection ~ 4150 1600
 Wire Wire Line
-	2450 3000 2450 3700
+	2450 3000 2450 3050
 Wire Wire Line
 	2650 3050 2650 3200
@@
 Connection ~ 2450 3050
 Wire Wire Line
-	2250 3100 2250 3800
+	2250 3100 2250 3150
 Wire Wire Line
 	2250 3800 2600 3800
@@
 	2500 4100 2600 4100
 Wire Wire Line
-	3900 4750 3900 5300
-Wire Wire Line
-	2850 4800 3900 4800
+	3900 4750 3900 4800
+Wire Wire Line
+	2850 4800 3050 4800
 Wire Wire Line
 	3050 4800 3050 4950
@@
 	3150 6150 2950 6150
 Wire Wire Line
-	2950 6150 2950 7500
+	2950 6150 2950 6350
 Wire Wire Line
 	3150 6350 2950 6350
@@
 	3150 6850 2850 6850
 Wire Wire Line
-	2850 4800 2850 7050
+	2850 4800 2850 6850
 Connection ~ 3050 4800
 Wire Wire Line
@@
 	4750 6450 5800 6450
 Wire Wire Line
-	3450 2450 4250 2450
-Wire Wire Line
-	3450 2350 4250 2350
-Wire Wire Line
-	1300 2450 2100 2450
-Wire Wire Line
-	1300 2350 2100 2350
+	3450 2450 3600 2450
+Wire Wire Line
+	3450 2350 3700 2350
+Wire Wire Line
+	1300 2450 1700 2450
+Wire Wire Line
+	1300 2350 1800 2350
 Wire Notes Line
 	500  4300 4800 4300
@@
 	1800 3900 1800 2350
 Wire Wire Line
-	1800 2350 1850 2350
-Connection ~ 1850 2350
-Wire Wire Line
 	1700 4000 1700 2450
 Wire Wire Line
@@
 	5700 3600 10100 3600
 $Comp
-L CONN_5 SERVO_0-3
+L brain-rescue:CONN_5-RESCUE-brain SERVO_0-3
 U 1 1 592C15A7
 P 10500 2900
@@
 $EndComp
 $Comp
-L CONN_5 SERVO_4-7
+L brain-rescue:CONN_5-RESCUE-brain SERVO_4-7
 U 1 1 592C16AE
 P 10500 3500
@@
 $EndComp
 $Comp
-L CONN_5 SERVO_8-13
+L brain-rescue:CONN_5-RESCUE-brain SERVO_8-13
 U 1 1 592C16FA
 P 10500 4100
@@
 $EndComp
 $Comp
-L GND-RESCUE-brain #PWR0116
+L brain-rescue:GND-RESCUE-brain #PWR0116
 U 1 1 592C2528
 P 10000 4750
@@
 $EndComp
 Wire Wire Line
-	10000 3100 10000 4750
+	10000 3100 10000 3700
 Wire Wire Line
 	10000 4300 10100 4300
@@
 Wire Wire Line
 	5100 2800 10100 2800
+Wire Wire Line
+	2600 1200 2600 1700
+Wire Wire Line
+	3150 1250 3550 1250
+Wire Wire Line
+	4000 2450 4250 2450
+Wire Wire Line
+	3800 2350 4250 2350
+Wire Wire Line
+	4150 1600 4150 2250
+Wire Wire Line
+	2450 3050 2450 3700
+Wire Wire Line
+	2250 3150 2250 3800
+Wire Wire Line
+	1700 2450 2100 2450
+Wire Wire Line
+	3900 4800 3900 5300
+Wire Wire Line
+	2950 6350 2950 6550
+Wire Wire Line
+	2950 6550 2950 6650
+Wire Wire Line
+	2950 6650 2950 6750
+Wire Wire Line
+	2950 6750 2950 7500
+Wire Wire Line
+	3050 4800 3900 4800
+Wire Wire Line
+	2850 6850 2850 6950
+Wire Wire Line
+	2850 6950 2850 7050
+Wire Wire Line
+	3700 2350 3800 2350
+Wire Wire Line
+	3600 2450 4000 2450
+Wire Wire Line
+	10000 4300 10000 4750
+Wire Wire Line
+	10000 3700 10000 4300
+Wire Wire Line
+	1800 2350 2100 2350
 $EndSCHEMATC
