File: brain/position.sch (KiCad schematic (older format))
At the start: 16 parts

Commit message: footprint assignation
Parts:
- C26, C29, C30, C31, C34: renamed from C?; footprint (none) -> Capacitors_SMD:C_0603
- C27, C28, C32, C33: renamed from C?; value C -> 100n; footprint (none) -> Capacitors_SMD:C_0603
- ENCL1: renamed from ENCL; footprint (none) -> Sockets_MOLEX_KK-System:Socket_MOLEX-KK-RM2-54mm_Lock_5pin_straight
- ENCR1: renamed from ENCR; footprint (none) -> Sockets_MOLEX_KK-System:Socket_MOLEX-KK-RM2-54mm_Lock_5pin_straight
- GYRO1: renamed from GYRO; footprint (none) -> Sockets_MOLEX_KK-System:Socket_MOLEX-KK-RM2-54mm_Lock_6pin_straight
- MOTL1: renamed from MOTL; footprint (none) -> Sockets_MOLEX_KK-System:Socket_MOLEX-KK-RM2-54mm_Lock_5pin_straight
- MOTR1: renamed from MOTR; footprint (none) -> Sockets_MOLEX_KK-System:Socket_MOLEX-KK-RM2-54mm_Lock_5pin_straight
- U3, U4: renamed from U?; footprint (none) -> Housings_SSOP:TSSOP-20_4.4x6.5mm_Pitch0.65mm
Connections:
- no-connect marks 0 -> 3

Commit message: Brain 2018 layout
Parts:
- removed C27, C32, C33: 100n, Capacitors_SMD:C_0603, symbol C
- removed C30: 4u7, Capacitors_SMD:C_0603, symbol C
- removed U3, U4: TXB0108, Housings_SSOP:TSSOP-20_4.4x6.5mm_Pitch0.65mm, symbol TXB0108
- added C2: 4u7, Capacitors_SMD:C_0603, symbol C-RESCUE-brain
- added C27: 100n, Capacitors_SMD:C_0603, symbol C-RESCUE-brain
- added R45, R46: 1k, Resistors_SMD:R_0603, symbol R
- added U3, U4: SN74AHCT125PW, Housings_SSOP:TSSOP-14_4.4x5mm_Pitch0.65mm, symbol SN74AHCT125PW
- C26, C28, C29, C31, C34: symbol C -> C-RESCUE-brain
Connections:
- net labels removed: +3V3, AX12_RX_3v3, AX12_RX_5v, AX12_TX_3v3, AX12_TX_5v, MOTL_DIR_5v, MOTL_PWM_5v, MOTR_DIR_5v, MOTR_PWM_5v, MOT_ENA_5v
- wire segments 105 -> 95
- no-connect marks 3 -> 0
Other:
- moved on the sheet: MOTL1, MOTR1

Commit message: add 3d step files to brain
Parts:
- C2, C26, C27, C28, C29, C31, C34: footprint Capacitors_SMD:C_0603 -> espitall:C_0603
- ENCL1, ENCR1, MOTL1, MOTR1: footprint Sockets_MOLEX_KK-System:Socket_MOLEX-KK-RM2-54mm_Lock_5pin_straight -> espitall:Socket_MOLEX-KK-RM2-54mm_Lock_5pin_straight
- GYRO1: footprint Sockets_MOLEX_KK-System:Socket_MOLEX-KK-RM2-54mm_Lock_6pin_straight -> espitall:Socket_MOLEX-KK-RM2-54mm_Lock_6pin_straight
- R45, R46: footprint Resistors_SMD:R_0603 -> espitall:R_0603
- U3, U4: footprint Housings_SSOP:TSSOP-14_4.4x5mm_Pitch0.65mm -> espitall:TSSOP-14_4.4x5mm_Pitch0.65mm
Changed lines of the file:
@@
-EESchema Schematic File Version 2
+EESchema Schematic File Version 3
 LIBS:brain-rescue
-LIBS:power
-LIBS:device
-LIBS:transistors
-LIBS:conn
-LIBS:linear
-LIBS:regul
-LIBS:74xx
-LIBS:cmos4000
-LIBS:adc-dac
-LIBS:memory
-LIBS:xilinx
-LIBS:microcontrollers
-LIBS:dsp
-LIBS:microchip
-LIBS:analog_switches
-LIBS:motorola
-LIBS:texas
-LIBS:intel
-LIBS:audio
-LIBS:interface
-LIBS:digital-audio
-LIBS:philips
-LIBS:display
-LIBS:cypress
-LIBS:siliconi
-LIBS:opto
-LIBS:atmel
-LIBS:contrib
-LIBS:valves
 LIBS:espitall
 LIBS:brain-cache
-EELAYER 25 0
+EELAYER 26 0
 EELAYER END
 $Descr A4 11693 8268
@@
 F 0 "ENCL1" V 10150 1150 50  0000 C CNN
 F 1 "CONN_5" V 10250 1150 50  0000 C CNN
-F 2 "Sockets_MOLEX_KK-System:Socket_MOLEX-KK-RM2-54mm_Lock_5pin_straight" H 10200 1150 60  0001 C CNN
+F 2 "espitall:Socket_MOLEX-KK-RM2-54mm_Lock_5pin_straight" H 10200 1150 60  0001 C CNN
 F 3 "" H 10200 1150 60  0000 C CNN
 	1    10200 1150
@@
 F 0 "C26" H 10500 1000 40  0000 L CNN
 F 1 "4u7" H 10506 815 40  0000 L CNN
-F 2 "Capacitors_SMD:C_0603" H 10538 750 30  0001 C CNN
+F 2 "espitall:C_0603" H 10538 750 30  0001 C CNN
 F 3 "" H 10500 900 60  0000 C CNN
 	1    10500 900
@@
 F 0 "ENCR1" V 10150 2700 50  0000 C CNN
 F 1 "CONN_5" V 10250 2700 50  0000 C CNN
-F 2 "Sockets_MOLEX_KK-System:Socket_MOLEX-KK-RM2-54mm_Lock_5pin_straight" H 10200 2700 60  0001 C CNN
+F 2 "espitall:Socket_MOLEX-KK-RM2-54mm_Lock_5pin_straight" H 10200 2700 60  0001 C CNN
 F 3 "" H 10200 2700 60  0000 C CNN
 	1    10200 2700
@@
 F 0 "C29" H 10500 2550 40  0000 L CNN
 F 1 "4u7" H 10506 2365 40  0000 L CNN
-F 2 "Capacitors_SMD:C_0603" H 10538 2300 30  0001 C CNN
+F 2 "espitall:C_0603" H 10538 2300 30  0001 C CNN
 F 3 "" H 10500 2450 60  0000 C CNN
 	1    10500 2450
@@
 F 0 "MOTL1" V 6400 5800 50  0000 C CNN
 F 1 "CONN_5" V 6500 5800 50  0000 C CNN
-F 2 "Sockets_MOLEX_KK-System:Socket_MOLEX-KK-RM2-54mm_Lock_5pin_straight" H 6450 5800 60  0001 C CNN
+F 2 "espitall:Socket_MOLEX-KK-RM2-54mm_Lock_5pin_straight" H 6450 5800 60  0001 C CNN
 F 3 "" H 6450 5800 60  0000 C CNN
 	1    6450 5800
@@
 F 0 "C31" H 6800 5900 40  0000 L CNN
 F 1 "4u7" H 6806 5715 40  0000 L CNN
-F 2 "Capacitors_SMD:C_0603" H 6838 5650 30  0001 C CNN
+F 2 "espitall:C_0603" H 6838 5650 30  0001 C CNN
 F 3 "" H 6800 5800 60  0000 C CNN
 	1    6800 5800
@@
 F 0 "MOTR1" V 6400 7050 50  0000 C CNN
 F 1 "CONN_5" V 6500 7050 50  0000 C CNN
-F 2 "Sockets_MOLEX_KK-System:Socket_MOLEX-KK-RM2-54mm_Lock_5pin_straight" H 6450 7050 60  0001 C CNN
+F 2 "espitall:Socket_MOLEX-KK-RM2-54mm_Lock_5pin_straight" H 6450 7050 60  0001 C CNN
 F 3 "" H 6450 7050 60  0000 C CNN
 	1    6450 7050
@@
 F 0 "C34" H 6800 7150 40  0000 L CNN
 F 1 "4u7" H 6806 6965 40  0000 L CNN
-F 2 "Capacitors_SMD:C_0603" H 6838 6900 30  0001 C CNN
+F 2 "espitall:C_0603" H 6838 6900 30  0001 C CNN
 F 3 "" H 6800 7050 60  0000 C CNN
 	1    6800 7050
@@
 F 0 "C28" H 3950 1200 40  0000 L CNN
 F 1 "100n" H 3956 1015 40  0000 L CNN
-F 2 "Capacitors_SMD:C_0603" H 3988 950 30  0001 C CNN
+F 2 "espitall:C_0603" H 3988 950 30  0001 C CNN
 F 3 "" H 3950 1100 60  0000 C CNN
 	1    3950 1100
@@
 F 0 "U3" H 3800 2600 60  0000 C CNN
 F 1 "SN74AHCT125PW" H 4100 1600 60  0000 C CNN
-F 2 "Housings_SSOP:TSSOP-14_4.4x5mm_Pitch0.65mm" H 3650 1650 60  0001 C CNN
+F 2 "espitall:TSSOP-14_4.4x5mm_Pitch0.65mm" H 3650 1650 60  0001 C CNN
 F 3 "" H 3650 1650 60  0000 C CNN
 	1    3650 2150
@@
 F 0 "R45" V 6580 3500 50  0000 C CNN
 F 1 "1k" V 6500 3500 50  0000 C CNN
-F 2 "Resistors_SMD:R_0603" V 6430 3500 50  0001 C CNN
+F 2 "espitall:R_0603" V 6430 3500 50  0001 C CNN
 F 3 "" H 6500 3500 50  0000 C CNN
 	1    6500 3500
@@
 F 0 "R46" V 6280 3750 50  0000 C CNN
 F 1 "1k" V 6200 3750 50  0000 C CNN
-F 2 "Resistors_SMD:R_0603" V 6130 3750 50  0001 C CNN
+F 2 "espitall:R_0603" V 6130 3750 50  0001 C CNN
 F 3 "" H 6200 3750 50  0000 C CNN
 	1    6200 3750
@@
 F 0 "C2" H 10550 3750 40  0000 L CNN
 F 1 "4u7" H 10556 3565 40  0000 L CNN
-F 2 "Capacitors_SMD:C_0603" H 10588 3500 30  0001 C CNN
+F 2 "espitall:C_0603" H 10588 3500 30  0001 C CNN
 F 3 "" H 10550 3650 60  0000 C CNN
 	1    10550 3650
@@
 F 0 "GYRO1" V 10150 3950 60  0000 C CNN
 F 1 "CONN_6" V 10250 3950 60  0000 C CNN
-F 2 "Sockets_MOLEX_KK-System:Socket_MOLEX-KK-RM2-54mm_Lock_6pin_straight" H 10200 3950 60  0001 C CNN
+F 2 "espitall:Socket_MOLEX-KK-RM2-54mm_Lock_6pin_straight" H 10200 3950 60  0001 C CNN
 F 3 "" H 10200 3950 60  0000 C CNN
 	1    10200 3950
@@
 F 0 "C27" H 3950 4250 40  0000 L CNN
 F 1 "100n" H 3956 4065 40  0000 L CNN
-F 2 "Capacitors_SMD:C_0603" H 3988 4000 30  0001 C CNN
+F 2 "espitall:C_0603" H 3988 4000 30  0001 C CNN
 F 3 "" H 3950 4150 60  0000 C CNN
 	1    3950 4150
@@
 F 0 "U4" H 3800 5650 60  0000 C CNN
 F 1 "SN74AHCT125PW" H 4100 4650 60  0000 C CNN
-F 2 "Housings_SSOP:TSSOP-14_4.4x5mm_Pitch0.65mm" H 3650 4700 60  0001 C CNN
+F 2 "espitall:TSSOP-14_4.4x5mm_Pitch0.65mm" H 3650 4700 60  0001 C CNN
 F 3 "" H 3650 4700 60  0000 C CNN
 	1    3650 5200

Commit message: add module add footprint SPSGRF-868 for future com board
Parts:
- C2, C26, C27, C28, C29, C31, C34: symbol C-RESCUE-brain -> brain-rescue:C-RESCUE-brain
- ENCL1, ENCR1, MOTL1, MOTR1: symbol CONN_5 -> brain-rescue:CONN_5-RESCUE-brain
- GYRO1: symbol CONN_6 -> brain-rescue:CONN_6-RESCUE-brain
- R45, R46: symbol R -> device:R
- U3, U4: symbol SN74AHCT125PW -> espitall:SN74AHCT125PW
Connections:
- wire segments 95 -> 110
Changed lines of the file:
@@
-EESchema Schematic File Version 3
-LIBS:brain-rescue
-LIBS:espitall
+EESchema Schematic File Version 4
 LIBS:brain-cache
 EELAYER 26 0
@@
 $EndDescr
 $Comp
-L CONN_5 ENCL1
+L brain-rescue:CONN_5-RESCUE-brain ENCL1
 U 1 1 5562C1E2
 P 10200 1150
@@
 $EndComp
 $Comp
-L GND-RESCUE-brain #PWR075
+L brain-rescue:GND-RESCUE-brain #PWR075
 U 1 1 5562C257
 P 9600 1550
@@
 $EndComp
 $Comp
-L +5V #PWR076
+L power:+5V #PWR076
 U 1 1 5562C27A
 P 9550 650
@@
 POS_SPI_MISO_5v
 $Comp
-L C-RESCUE-brain C26
+L brain-rescue:C-RESCUE-brain C26
 U 1 1 5562C54E
 P 10500 900
@@
 $EndComp
 $Comp
-L GND-RESCUE-brain #PWR077
+L brain-rescue:GND-RESCUE-brain #PWR077
 U 1 1 5562C591
 P 10500 1550
@@
 $EndComp
 $Comp
-L CONN_5 ENCR1
+L brain-rescue:CONN_5-RESCUE-brain ENCR1
 U 1 1 5562C68C
 P 10200 2700
@@
 $EndComp
 $Comp
-L GND-RESCUE-brain #PWR078
+L brain-rescue:GND-RESCUE-brain #PWR078
 U 1 1 5562C692
 P 9600 3100
@@
 $EndComp
 $Comp
-L +5V #PWR079
+L power:+5V #PWR079
 U 1 1 5562C698
 P 9550 2200
@@
 POS_SPI_MISO_5v
 $Comp
-L C-RESCUE-brain C29
+L brain-rescue:C-RESCUE-brain C29
 U 1 1 5562C6A8
 P 10500 2450
@@
 $EndComp
 $Comp
-L GND-RESCUE-brain #PWR080
+L brain-rescue:GND-RESCUE-brain #PWR080
 U 1 1 5562C6AE
 P 10500 3100
@@
 	8600 2600 9800 2600
 Wire Wire Line
-	9550 2200 9550 2500
+	9550 2200 9550 2250
 Wire Wire Line
 	9550 2500 9800 2500
@@
 	8600 1050 9800 1050
 Wire Wire Line
-	9550 650  9550 950
+	9550 650  9550 700
 Wire Wire Line
 	9550 950  9800 950
 $Comp
-L CONN_5 MOTL1
+L brain-rescue:CONN_5-RESCUE-brain MOTL1
 U 1 1 55633DD1
 P 6450 5800
@@
 $EndComp
 Wire Wire Line
-	5150 5700 5150 7200
+	5150 5700 5150 6950
 Wire Wire Line
 	5150 5700 6050 5700
@@
 	5350 5900 5350 7500
 $Comp
-L GND-RESCUE-brain #PWR081
+L brain-rescue:GND-RESCUE-brain #PWR081
 U 1 1 55633FDC
 P 6000 6200
@@
 $EndComp
 $Comp
-L +5V #PWR082
+L power:+5V #PWR082
 U 1 1 55633FFB
 P 6000 5350
@@
 $EndComp
 $Comp
-L C-RESCUE-brain C31
+L brain-rescue:C-RESCUE-brain C31
 U 1 1 5563401A
 P 6800 5800
@@
 $EndComp
 $Comp
-L GND-RESCUE-brain #PWR083
+L brain-rescue:GND-RESCUE-brain #PWR083
 U 1 1 55634096
 P 6800 6200
@@
 	6800 5400 6000 5400
 Wire Wire Line
-	6000 5350 6000 5600
+	6000 5350 6000 5400
 Wire Wire Line
 	6000 5600 6050 5600
@@
 	6000 6000 6000 6200
 $Comp
-L CONN_5 MOTR1
+L brain-rescue:CONN_5-RESCUE-brain MOTR1
 U 1 1 55634312
 P 6450 7050
@@
 $EndComp
 $Comp
-L GND-RESCUE-brain #PWR084
+L brain-rescue:GND-RESCUE-brain #PWR084
 U 1 1 5563431B
 P 6000 7450
@@
 $EndComp
 $Comp
-L +5V #PWR085
+L power:+5V #PWR085
 U 1 1 55634321
 P 6000 6600
@@
 $EndComp
 $Comp
-L C-RESCUE-brain C34
+L brain-rescue:C-RESCUE-brain C34
 U 1 1 55634327
 P 6800 7050
@@
 $EndComp
 $Comp
-L GND-RESCUE-brain #PWR086
+L brain-rescue:GND-RESCUE-brain #PWR086
 U 1 1 5563432D
 P 6800 7450
@@
 	6800 6650 6000 6650
 Wire Wire Line
-	6000 6600 6000 6850
+	6000 6600 6000 6650
 Wire Wire Line
 	6000 6850 6050 6850
@@
 	5550 7150 5550 7600
 $Comp
-L +5V #PWR087
+L power:+5V #PWR087
 U 1 1 55634D8A
 P 3650 700
@@
 $EndComp
 $Comp
-L C-RESCUE-brain C28
+L brain-rescue:C-RESCUE-brain C28
 U 1 1 55634D96
 P 3950 1100
@@
 $EndComp
 $Comp
-L GND-RESCUE-brain #PWR088
+L brain-rescue:GND-RESCUE-brain #PWR088
 U 1 1 55634DA8
 P 3950 1300
@@
 POS_SPI_MISO_5v
 $Comp
-L GND-RESCUE-brain #PWR089
+L brain-rescue:GND-RESCUE-brain #PWR089
 U 1 1 55634DB0
 P 3650 3300
@@
 	4350 2150 5750 2150
 Wire Wire Line
-	5000 3500 6350 3500
+	5000 3500 6200 3500
 Wire Wire Line
 	3000 2350 1900 2350
@@
 	3000 1950 1900 1950
 Wire Wire Line
-	3650 2950 3650 3300
+	3650 2950 3650 3050
 Wire Wire Line
 	4350 2050 5750 2050
@@
 POS_SPI_MOSI_3v3
 $Comp
-L SN74AHCT125PW U3
+L espitall:SN74AHCT125PW U3
 U 1 1 58D98F44
 P 3650 2150
@@
 	2900 3050 3650 3050
 Wire Wire Line
-	2900 1850 2900 3050
+	2900 1850 2900 2050
 Wire Wire Line
 	2900 1850 3000 1850
@@
 Connection ~ 2900 2450
 $Comp
-L R R45
+L device:R R45
 U 1 1 58D999E6
 P 6500 3500
@@
 $EndComp
 $Comp
-L R R46
+L device:R R46
 U 1 1 58D99A40
 P 6200 3750
@@
 $EndComp
 $Comp
-L GND-RESCUE-brain #PWR090
+L brain-rescue:GND-RESCUE-brain #PWR090
 U 1 1 58D99A8A
 P 6200 4000
@@
 Connection ~ 6200 3500
 $Comp
-L GND-RESCUE-brain #PWR091
+L brain-rescue:GND-RESCUE-brain #PWR091
 U 1 1 5929DFCD
 P 9650 4450
@@
 POS_SPI_MISO_5v
 $Comp
-L C-RESCUE-brain C2
+L brain-rescue:C-RESCUE-brain C2
 U 1 1 5929DFDC
 P 10550 3650
@@
 $EndComp
 $Comp
-L GND-RESCUE-brain #PWR092
+L brain-rescue:GND-RESCUE-brain #PWR092
 U 1 1 5929DFE2
 P 10550 4450
@@
 	8350 3800 9850 3800
 Wire Wire Line
-	9600 3400 9600 3700
+	9600 3400 9600 3450
 Wire Wire Line
 	9600 3700 9850 3700
 $Comp
-L CONN_6 GYRO1
+L brain-rescue:CONN_6-RESCUE-brain GYRO1
 U 1 1 5929E01E
 P 10200 3950
@@
 	4900 6600 4900 5000
 $Comp
-L +5V #PWR093
+L power:+5V #PWR093
 U 1 1 5929FD76
 P 3650 3750
@@
 $EndComp
 $Comp
-L C-RESCUE-brain C27
+L brain-rescue:C-RESCUE-brain C27
 U 1 1 5929FD7C
 P 3950 4150
@@
 $EndComp
 $Comp
-L GND-RESCUE-brain #PWR094
+L brain-rescue:GND-RESCUE-brain #PWR094
 U 1 1 5929FD82
 P 3950 4350
@@
 $EndComp
 $Comp
-L GND-RESCUE-brain #PWR095
+L brain-rescue:GND-RESCUE-brain #PWR095
 U 1 1 5929FD89
 P 3650 6350
@@
 	3000 5000 1900 5000
 Wire Wire Line
-	3650 6000 3650 6350
+	3650 6000 3650 6100
 Wire Wire Line
 	4350 4900 8350 4900
@@
 	3650 3750 3650 4500
 $Comp
-L SN74AHCT125PW U4
+L espitall:SN74AHCT125PW U4
 U 1 1 5929FDA8
 P 3650 5200
@@
 	2900 6100 3650 6100
 Wire Wire Line
-	2900 4900 2900 6100
+	2900 4900 2900 5100
 Wire Wire Line
 	2900 4900 3000 4900
@@
 	8350 4900 8350 3800
 $Comp
-L +5V #PWR096
+L power:+5V #PWR096
 U 1 1 592B1B39
 P 9600 3400
@@
 	1    0    0    -1
 $EndComp
+Wire Wire Line
+	9550 2250 9550 2500
+Wire Wire Line
+	9550 700  9550 950
+Wire Wire Line
+	6000 5400 6000 5600
+Wire Wire Line
+	6000 6650 6000 6850
+Wire Wire Line
+	5150 6950 5150 7200
+Wire Wire Line
+	3650 3050 3650 3300
+Wire Wire Line
+	2900 2050 2900 2250
+Wire Wire Line
+	2900 2250 2900 2450
+Wire Wire Line
+	2900 2450 2900 3050
+Wire Wire Line
+	6200 3500 6350 3500
+Wire Wire Line
+	9600 3450 9600 3700
+Wire Wire Line
+	3650 6100 3650 6350
+Wire Wire Line
+	2900 5100 2900 5300
+Wire Wire Line
+	2900 5300 2900 5500
+Wire Wire Line
+	2900 5500 2900 6100
 $EndSCHEMATC
