File: brain/slave.sch (KiCad schematic (older format))
At the start: 14 parts

Commit message: updated schematic of brain board
Parts:
- added C? (x2): 4u7, symbol C
- added SLA4: HE10-16, symbol HE10-16
- gave numbers to parts that had none: 4
Connections:
- net labels added: SLA_SPI_CS10_3v3, SLA_SPI_CS11_3v3, SLA_SPI_CS12_3v3, SLA_SPI_CS4_3v3, SLA_SPI_CS5_3v3, SLA_SPI_CS6_3v3, SLA_SPI_CS7_3v3, SLA_SPI_CS8_3v3, SLA_SPI_CS9_3v3
- net labels removed: SLA_SPI_CS0_3v3
- wire segments 61 -> 97

Commit message: footprint assignation
Parts:
- added C90, C91: 4u7, Capacitors_SMD:C_0603, symbol C
- added SLAUART1: CONN_01X05, Sockets_MOLEX_KK-System:Socket_MOLEX-KK-RM2-54mm_Lock_5pin_straight, symbol CONN_01X05
- C15, C16, C17, C18, C19, C20, C21, C22, C23, C24, C25: renamed from C?; footprint (none) -> Capacitors_SMD:C_0603
- SLA0, SLA1, SLA2, SLA3: footprint (none) -> espitall:Socket_MOLEX-KK-RM2-54mm_Lock_8pin_straight
- SLA4: footprint (none) -> espitall:HE10_16D
- U2: renamed from U?; footprint (none) -> Housings_SOIC:SOIC-24_7.5x15.4mm_Pitch1.27mm
Connections:
- net labels added: SLA_RX_3v3, SLA_TX_3v3
- wire segments 97 -> 109
- no-connect marks 0 -> 4

Commit message: all tracks are routed
Changed lines of the file:
@@
 Connection ~ 6650 2000
-Wire Wire Line
-	6550 2200 6550 5350
-Connection ~ 6550 2200
 Wire Wire Line
 	6650 3750 9950 3750
@@
 Text Label 6450 3950 0    60   ~ 0
 SLA_SPI_CS3_3v3
-Wire Wire Line
-	6350 2200 7400 2200
 Wire Wire Line
 	9950 2200 8900 2200
@@
 Text HLabel 2750 6750 2    60   Output ~ 0
 SLA_RX_3v3
+Wire Wire Line
+	6550 2100 6550 5350
+Connection ~ 6550 2100
+Wire Wire Line
+	7400 2200 6350 2200
 $EndSCHEMATC

Commit message: Brain 2018 layout
Parts:
- C15, C16, C17, C18, C19, C20, C21, C22, C23, C24, C25, C90, C91: symbol C -> C-RESCUE-brain

Commit message: add 3d step files to brain
Parts:
- C15, C16, C17, C18, C19, C20, C21, C22, C23, C24, C25, C90, C91: footprint Capacitors_SMD:C_0603 -> espitall:C_0603
- SLAUART1: footprint Sockets_MOLEX_KK-System:Socket_MOLEX-KK-RM2-54mm_Lock_5pin_straight -> espitall:Socket_MOLEX-KK-RM2-54mm_Lock_5pin_straight
- U2: footprint Housings_SOIC:SOIC-24_7.5x15.4mm_Pitch1.27mm -> espitall:SOIC-24_7.5x15.4mm_Pitch1.27mm
Changed lines of the file:
@@
-EESchema Schematic File Version 2
+EESchema Schematic File Version 3
 LIBS:brain-rescue
-LIBS:power
-LIBS:device
-LIBS:transistors
-LIBS:conn
-LIBS:linear
-LIBS:regul
-LIBS:74xx
-LIBS:cmos4000
-LIBS:adc-dac
-LIBS:memory
-LIBS:xilinx
-LIBS:microcontrollers
-LIBS:dsp
-LIBS:microchip
-LIBS:analog_switches
-LIBS:motorola
-LIBS:texas
-LIBS:intel
-LIBS:audio
-LIBS:interface
-LIBS:digital-audio
-LIBS:philips
-LIBS:display
-LIBS:cypress
-LIBS:siliconi
-LIBS:opto
-LIBS:atmel
-LIBS:contrib
-LIBS:valves
 LIBS:espitall
 LIBS:brain-cache
-EELAYER 25 0
+EELAYER 26 0
 EELAYER END
 $Descr A4 11693 8268
@@
 F 0 "U2" H 3250 3300 60  0000 C CNN
 F 1 "74HC154" H 3000 2400 60  0000 C CNN
-F 2 "Housings_SOIC:SOIC-24_7.5x15.4mm_Pitch1.27mm" H 3000 2400 60  0001 C CNN
+F 2 "espitall:SOIC-24_7.5x15.4mm_Pitch1.27mm" H 3000 2400 60  0001 C CNN
 F 3 "" H 3000 2400 60  0000 C CNN
 	1    3000 2400
@@
 F 0 "C15" H 2750 1250 40  0000 L CNN
 F 1 "100n" H 2756 1065 40  0000 L CNN
-F 2 "Capacitors_SMD:C_0603" H 2788 1000 30  0001 C CNN
+F 2 "espitall:C_0603" H 2788 1000 30  0001 C CNN
 F 3 "" H 2750 1150 60  0000 C CNN
 	1    2750 1150
@@
 F 0 "C18" H 9400 1350 40  0000 L CNN
 F 1 "100n" H 9406 1165 40  0000 L CNN
-F 2 "Capacitors_SMD:C_0603" H 9438 1100 30  0001 C CNN
+F 2 "espitall:C_0603" H 9438 1100 30  0001 C CNN
 F 3 "" H 9400 1250 60  0000 C CNN
 	1    9400 1250
@@
 F 0 "C19" H 9900 1350 40  0000 L CNN
 F 1 "100n" H 9906 1165 40  0000 L CNN
-F 2 "Capacitors_SMD:C_0603" H 9938 1100 30  0001 C CNN
+F 2 "espitall:C_0603" H 9938 1100 30  0001 C CNN
 F 3 "" H 9900 1250 60  0000 C CNN
 	1    9900 1250
@@
 F 0 "C22" H 9400 3100 40  0000 L CNN
 F 1 "100n" H 9406 2915 40  0000 L CNN
-F 2 "Capacitors_SMD:C_0603" H 9438 2850 30  0001 C CNN
+F 2 "espitall:C_0603" H 9438 2850 30  0001 C CNN
 F 3 "" H 9400 3000 60  0000 C CNN
 	1    9400 3000
@@
 F 0 "C23" H 9900 3100 40  0000 L CNN
 F 1 "100n" H 9906 2915 40  0000 L CNN
-F 2 "Capacitors_SMD:C_0603" H 9938 2850 30  0001 C CNN
+F 2 "espitall:C_0603" H 9938 2850 30  0001 C CNN
 F 3 "" H 9900 3000 60  0000 C CNN
 	1    9900 3000
@@
 F 0 "C16" H 6850 1350 40  0000 L CNN
 F 1 "100n" H 6856 1165 40  0000 L CNN
-F 2 "Capacitors_SMD:C_0603" H 6888 1100 30  0001 C CNN
+F 2 "espitall:C_0603" H 6888 1100 30  0001 C CNN
 F 3 "" H 6850 1250 60  0000 C CNN
 	1    6850 1250
@@
 F 0 "C17" H 7350 1350 40  0000 L CNN
 F 1 "100n" H 7356 1165 40  0000 L CNN
-F 2 "Capacitors_SMD:C_0603" H 7388 1100 30  0001 C CNN
+F 2 "espitall:C_0603" H 7388 1100 30  0001 C CNN
 F 3 "" H 7350 1250 60  0000 C CNN
 	1    7350 1250
@@
 F 0 "C20" H 6850 3100 40  0000 L CNN
 F 1 "100n" H 6856 2915 40  0000 L CNN
-F 2 "Capacitors_SMD:C_0603" H 6888 2850 30  0001 C CNN
+F 2 "espitall:C_0603" H 6888 2850 30  0001 C CNN
 F 3 "" H 6850 3000 60  0000 C CNN
 	1    6850 3000
@@
 F 0 "C21" H 7350 3100 40  0000 L CNN
 F 1 "100n" H 7356 2915 40  0000 L CNN
-F 2 "Capacitors_SMD:C_0603" H 7388 2850 30  0001 C CNN
+F 2 "espitall:C_0603" H 7388 2850 30  0001 C CNN
 F 3 "" H 7350 3000 60  0000 C CNN
 	1    7350 3000
@@
 F 0 "C25" H 7350 6200 40  0000 L CNN
 F 1 "4u7" H 7356 6015 40  0000 L CNN
-F 2 "Capacitors_SMD:C_0603" H 7388 5950 30  0001 C CNN
+F 2 "espitall:C_0603" H 7388 5950 30  0001 C CNN
 F 3 "" H 7350 6100 60  0000 C CNN
 	1    7350 6100
@@
 F 0 "C24" H 7000 6200 40  0000 L CNN
 F 1 "4u7" H 7006 6015 40  0000 L CNN
-F 2 "Capacitors_SMD:C_0603" H 7038 5950 30  0001 C CNN
+F 2 "espitall:C_0603" H 7038 5950 30  0001 C CNN
 F 3 "" H 7000 6100 60  0000 C CNN
 	1    7000 6100
@@
 F 0 "SLAUART1" H 1950 6950 50  0000 C CNN
 F 1 "CONN_01X05" V 2050 6650 50  0000 C CNN
-F 2 "Sockets_MOLEX_KK-System:Socket_MOLEX-KK-RM2-54mm_Lock_5pin_straight" H 1950 6650 60  0001 C CNN
+F 2 "espitall:Socket_MOLEX-KK-RM2-54mm_Lock_5pin_straight" H 1950 6650 60  0001 C CNN
 F 3 "" H 1950 6650 60  0000 C CNN
 	1    1950 6650
@@
 F 0 "C90" H 1725 6000 50  0000 L CNN
 F 1 "4u7" H 1725 5800 50  0000 L CNN
-F 2 "Capacitors_SMD:C_0603" V 1600 5900 30  0001 C CNN
+F 2 "espitall:C_0603" V 1600 5900 30  0001 C CNN
 F 3 "" H 1700 5900 60  0000 C CNN
 	1    1700 5900
@@
 F 0 "C91" H 1975 6000 50  0000 L CNN
 F 1 "4u7" H 1975 5800 50  0000 L CNN
-F 2 "Capacitors_SMD:C_0603" V 1850 5900 30  0001 C CNN
+F 2 "espitall:C_0603" V 1850 5900 30  0001 C CNN
 F 3 "" H 1950 5900 60  0000 C CNN
 	1    1950 5900

Commit message: add module add footprint SPSGRF-868 for future com board
Parts:
- C15, C16, C17, C18, C19, C20, C21, C22, C23, C24, C25, C90, C91: symbol C-RESCUE-brain -> brain-rescue:C-RESCUE-brain
- SLA0, SLA1, SLA2, SLA3: symbol CONN_8 -> brain-rescue:CONN_8-RESCUE-brain
- SLA4: symbol HE10-16 -> conn:HE10-16
- SLAUART1: symbol CONN_01X05 -> brain-rescue:CONN_01X05-RESCUE-brain
- U2: symbol 74HC154 -> espitall:74HC154
Connections:
- wire segments 109 -> 131
