File: brain/supply.sch (KiCad schematic (older format))
At the start: 6 parts

Commit message: footprint assignation
Parts:
- C87, C89: renamed from C?; footprint (none) -> Capacitors_SMD:C_0603
- C88: renamed from C?; footprint (none) -> Capacitors_SMD:c_elec_6.3x7.7
- PWR1: renamed from PWR; footprint (none) -> Sockets_MOLEX_KK-System:Socket_MOLEX-KK-RM2-54mm_Lock_2pin_straight
- U10, U9: renamed from U?; footprint (none) -> espitall:TSR-1
Changed lines of the file:
@@
 LIBS:contrib
 LIBS:valves
-LIBS:stm32
 LIBS:espitall
 LIBS:brain-cache
@@
 $EndDescr
 $Comp
-L CONN_2 PWR
+L CONN_2 PWR1
 U 1 1 556E624F
 P 3750 3700
-F 0 "PWR" V 3700 3700 40  0000 C CNN
+F 0 "PWR1" V 3700 3700 40  0000 C CNN
 F 1 "CONN_2" V 3800 3700 40  0000 C CNN
-F 2 "" H 3750 3700 60  0000 C CNN
+F 2 "Sockets_MOLEX_KK-System:Socket_MOLEX-KK-RM2-54mm_Lock_2pin_straight" H 3750 3700 60  0001 C CNN
 F 3 "" H 3750 3700 60  0000 C CNN
 	1    3750 3700
@@
 $EndComp
 $Comp
-L GND #PWR?
+L GND #PWR0258
 U 1 1 556E62AE
 P 4200 4100
-F 0 "#PWR?" H 4200 4100 30  0001 C CNN
+F 0 "#PWR0258" H 4200 4100 30  0001 C CNN
 F 1 "GND" H 4200 4030 30  0001 C CNN
 F 2 "" H 4200 4100 60  0000 C CNN
@@
 $EndComp
 $Comp
-L +BATT #PWR?
+L +BATT #PWR0259
 U 1 1 556E62C3
 P 4250 3150
-F 0 "#PWR?" H 4250 3100 20  0001 C CNN
+F 0 "#PWR0259" H 4250 3100 20  0001 C CNN
 F 1 "+BATT" H 4250 3250 30  0000 C CNN
 F 2 "" H 4250 3150 60  0000 C CNN
@@
 	4200 3800 4200 4100
 $Comp
-L C C?
+L C C88
 U 1 1 556E6F4F
 P 4450 3650
-F 0 "C?" H 4450 3750 40  0000 L CNN
+F 0 "C88" H 4450 3750 40  0000 L CNN
 F 1 "100u" H 4456 3565 40  0000 L CNN
-F 2 "" H 4488 3500 30  0000 C CNN
+F 2 "Capacitors_SMD:c_elec_6.3x7.7" H 4488 3500 30  0001 C CNN
 F 3 "" H 4450 3650 60  0000 C CNN
 	1    4450 3650
@@
 Connection ~ 4250 3350
 $Comp
-L TSR1-2450 U?
+L TSR1-2450 U9
 U 1 1 556E764E
 P 6450 2850
-F 0 "U?" H 6600 2654 60  0000 C CNN
+F 0 "U9" H 6600 2654 60  0000 C CNN
 F 1 "TSR1-2450" H 6450 3050 60  0000 C CNN
-F 2 "" H 6450 2850 60  0000 C CNN
+F 2 "espitall:TSR-1" H 6450 2850 60  0001 C CNN
 F 3 "" H 6450 2850 60  0000 C CNN
 	1    6450 2850
@@
 $EndComp
 $Comp
-L GND #PWR?
+L GND #PWR0260
 U 1 1 556E7685
 P 6450 3500
-F 0 "#PWR?" H 6450 3500 30  0001 C CNN
+F 0 "#PWR0260" H 6450 3500 30  0001 C CNN
 F 1 "GND" H 6450 3430 30  0001 C CNN
 F 2 "" H 6450 3500 60  0000 C CNN
@@
 $EndComp
 $Comp
-L C C?
+L C C87
 U 1 1 556E7699
 P 7150 3150
-F 0 "C?" H 7150 3250 40  0000 L CNN
+F 0 "C87" H 7150 3250 40  0000 L CNN
 F 1 "4u7" H 7156 3065 40  0000 L CNN
-F 2 "" H 7188 3000 30  0000 C CNN
+F 2 "Capacitors_SMD:C_0603" H 7188 3000 30  0001 C CNN
 F 3 "" H 7150 3150 60  0000 C CNN
 	1    7150 3150
@@
 $EndComp
 $Comp
-L +BATT #PWR?
+L +BATT #PWR0261
 U 1 1 556E76EB
 P 5850 2650
-F 0 "#PWR?" H 5850 2600 20  0001 C CNN
+F 0 "#PWR0261" H 5850 2600 20  0001 C CNN
 F 1 "+BATT" H 5850 2750 30  0000 C CNN
 F 2 "" H 5850 2650 60  0000 C CNN
@@
 	6450 3100 6450 3500
 $Comp
-L GND #PWR?
+L GND #PWR0262
 U 1 1 556E7736
 P 7150 3450
-F 0 "#PWR?" H 7150 3450 30  0001 C CNN
+F 0 "#PWR0262" H 7150 3450 30  0001 C CNN
 F 1 "GND" H 7150 3380 30  0001 C CNN
 F 2 "" H 7150 3450 60  0000 C CNN
@@
 	7150 2800 6850 2800
 $Comp
-L GND #PWR?
+L GND #PWR0263
 U 1 1 556E78DB
 P 6450 4750
-F 0 "#PWR?" H 6450 4750 30  0001 C CNN
+F 0 "#PWR0263" H 6450 4750 30  0001 C CNN
 F 1 "GND" H 6450 4680 30  0001 C CNN
 F 2 "" H 6450 4750 60  0000 C CNN
@@
 $EndComp
 $Comp
-L C C?
+L C C89
 U 1 1 556E78E1
 P 7150 4400
-F 0 "C?" H 7150 4500 40  0000 L CNN
+F 0 "C89" H 7150 4500 40  0000 L CNN
 F 1 "4u7" H 7156 4315 40  0000 L CNN
-F 2 "" H 7188 4250 30  0000 C CNN
+F 2 "Capacitors_SMD:C_0603" H 7188 4250 30  0001 C CNN
 F 3 "" H 7150 4400 60  0000 C CNN
 	1    7150 4400
@@
 $EndComp
 $Comp
-L +BATT #PWR?
+L +BATT #PWR0264
 U 1 1 556E78E7
 P 5850 3900
-F 0 "#PWR?" H 5850 3850 20  0001 C CNN
+F 0 "#PWR0264" H 5850 3850 20  0001 C CNN
 F 1 "+BATT" H 5850 4000 30  0000 C CNN
 F 2 "" H 5850 3900 60  0000 C CNN
@@
 	6450 4350 6450 4750
 $Comp
-L GND #PWR?
+L GND #PWR0265
 U 1 1 556E78F0
 P 7150 4700
-F 0 "#PWR?" H 7150 4700 30  0001 C CNN
+F 0 "#PWR0265" H 7150 4700 30  0001 C CNN
 F 1 "GND" H 7150 4630 30  0001 C CNN
 F 2 "" H 7150 4700 60  0000 C CNN
@@
 	7150 4050 6850 4050
 $Comp
-L TSR1-2433 U?
+L TSR1-2433 U10
 U 1 1 556E7AB0
 P 6450 4100
-F 0 "U?" H 6600 3904 60  0000 C CNN
+F 0 "U10" H 6600 3904 60  0000 C CNN
 F 1 "TSR1-2433" H 6450 4300 60  0000 C CNN
-F 2 "" H 6450 4100 60  0000 C CNN
+F 2 "espitall:TSR-1" H 6450 4100 60  0001 C CNN
 F 3 "" H 6450 4100 60  0000 C CNN
 	1    6450 4100
@@
 $EndComp
 $Comp
-L +5V #PWR?
+L +5V #PWR0266
 U 1 1 556E7ACF
 P 7150 2550
-F 0 "#PWR?" H 7150 2640 20  0001 C CNN
+F 0 "#PWR0266" H 7150 2640 20  0001 C CNN
 F 1 "+5V" H 7150 2640 30  0000 C CNN
 F 2 "" H 7150 2550 60  0000 C CNN
@@
 $EndComp
 $Comp
-L +3V3 #PWR?
+L +3V3 #PWR0267
 U 1 1 556E7AE9
 P 7150 4000
-F 0 "#PWR?" H 7150 3850 50  0001 C CNN
+F 0 "#PWR0267" H 7150 3850 50  0001 C CNN
 F 1 "+3V3" H 7150 4140 50  0000 C CNN
 F 2 "" H 7150 4000 60  0000 C CNN

Commit message: Brain 2018 layout
Parts:
- C87, C88, C89: symbol C -> C-RESCUE-brain
Changed lines of the file:
@@
 EESchema Schematic File Version 2
+LIBS:brain-rescue
 LIBS:power
 LIBS:device
@@
 LIBS:memory
 LIBS:xilinx
-LIBS:special
 LIBS:microcontrollers
 LIBS:dsp
@@
 $Descr A4 11693 8268
 encoding utf-8
-Sheet 8 8
-Title ""
-Date ""
-Rev ""
-Comp ""
-Comment1 ""
+Sheet 8 9
+Title "Brain"
+Date "2017-05-28"
+Rev "2018"
+Comp "Cocobot"
+Comment1 "Board for eurobot 2018 (French edition)"
 Comment2 ""
 Comment3 ""
@@
 $EndComp
 $Comp
-L GND #PWR227
+L GND-RESCUE-brain #PWR0214
 U 1 1 556E62AE
 P 4200 4100
-F 0 "#PWR227" H 4200 4100 30  0001 C CNN
+F 0 "#PWR0214" H 4200 4100 30  0001 C CNN
 F 1 "GND" H 4200 4030 30  0001 C CNN
 F 2 "" H 4200 4100 60  0000 C CNN
@@
 $EndComp
 $Comp
-L +BATT #PWR222
+L +BATT #PWR0215
 U 1 1 556E62C3
 P 4250 3150
-F 0 "#PWR222" H 4250 3100 20  0001 C CNN
+F 0 "#PWR0215" H 4250 3100 20  0001 C CNN
 F 1 "+BATT" H 4250 3250 30  0000 C CNN
 F 2 "" H 4250 3150 60  0000 C CNN
@@
 	4200 3800 4200 4100
 $Comp
-L C C88
+L C-RESCUE-brain C88
 U 1 1 556E6F4F
 P 4450 3650
@@
 $EndComp
 $Comp
-L GND #PWR224
+L GND-RESCUE-brain #PWR0216
 U 1 1 556E7685
 P 6450 3500
-F 0 "#PWR224" H 6450 3500 30  0001 C CNN
+F 0 "#PWR0216" H 6450 3500 30  0001 C CNN
 F 1 "GND" H 6450 3430 30  0001 C CNN
 F 2 "" H 6450 3500 60  0000 C CNN
@@
 $EndComp
 $Comp
-L C C87
+L C-RESCUE-brain C87
 U 1 1 556E7699
 P 7150 3150
@@
 $EndComp
 $Comp
-L +BATT #PWR221
+L +BATT #PWR0217
 U 1 1 556E76EB
 P 5850 2650
-F 0 "#PWR221" H 5850 2600 20  0001 C CNN
+F 0 "#PWR0217" H 5850 2600 20  0001 C CNN
 F 1 "+BATT" H 5850 2750 30  0000 C CNN
 F 2 "" H 5850 2650 60  0000 C CNN
@@
 	6450 3100 6450 3500
 $Comp
-L GND #PWR223
+L GND-RESCUE-brain #PWR0218
 U 1 1 556E7736
 P 7150 3450
-F 0 "#PWR223" H 7150 3450 30  0001 C CNN
+F 0 "#PWR0218" H 7150 3450 30  0001 C CNN
 F 1 "GND" H 7150 3380 30  0001 C CNN
 F 2 "" H 7150 3450 60  0000 C CNN
@@
 	7150 2800 6850 2800
 $Comp
-L GND #PWR229
+L GND-RESCUE-brain #PWR0219
 U 1 1 556E78DB
 P 6450 4750
-F 0 "#PWR229" H 6450 4750 30  0001 C CNN
+F 0 "#PWR0219" H 6450 4750 30  0001 C CNN
 F 1 "GND" H 6450 4680 30  0001 C CNN
 F 2 "" H 6450 4750 60  0000 C CNN
@@
 $EndComp
 $Comp
-L C C89
+L C-RESCUE-brain C89
 U 1 1 556E78E1
 P 7150 4400
@@
 $EndComp
 $Comp
-L +BATT #PWR225
+L +BATT #PWR0220
 U 1 1 556E78E7
 P 5850 3900
-F 0 "#PWR225" H 5850 3850 20  0001 C CNN
+F 0 "#PWR0220" H 5850 3850 20  0001 C CNN
 F 1 "+BATT" H 5850 4000 30  0000 C CNN
 F 2 "" H 5850 3900 60  0000 C CNN
@@
 	6450 4350 6450 4750
 $Comp
-L GND #PWR228
+L GND-RESCUE-brain #PWR0221
 U 1 1 556E78F0
 P 7150 4700
-F 0 "#PWR228" H 7150 4700 30  0001 C CNN
+F 0 "#PWR0221" H 7150 4700 30  0001 C CNN
 F 1 "GND" H 7150 4630 30  0001 C CNN
 F 2 "" H 7150 4700 60  0000 C CNN
@@
 $EndComp
 $Comp
-L +5V #PWR220
+L +5V #PWR0222
 U 1 1 556E7ACF
 P 7150 2550
-F 0 "#PWR220" H 7150 2640 20  0001 C CNN
+F 0 "#PWR0222" H 7150 2640 20  0001 C CNN
 F 1 "+5V" H 7150 2640 30  0000 C CNN
 F 2 "" H 7150 2550 60  0000 C CNN
@@
 $EndComp
 $Comp
-L +3V3 #PWR226
+L +3V3 #PWR0223
 U 1 1 556E7AE9
 P 7150 4000
-F 0 "#PWR226" H 7150 3850 50  0001 C CNN
+F 0 "#PWR0223" H 7150 3850 50  0001 C CNN
 F 1 "+3V3" H 7150 4140 50  0000 C CNN
 F 2 "" H 7150 4000 60  0000 C CNN

Commit message: add 3d step files to brain
Parts:
- C87, C89: footprint Capacitors_SMD:C_0603 -> espitall:C_0603
- C88: footprint Capacitors_SMD:c_elec_6.3x7.7 -> espitall:c_elec_6.3x7.7
- PWR1: footprint Sockets_MOLEX_KK-System:Socket_MOLEX-KK-RM2-54mm_Lock_2pin_straight -> espitall:Socket_MOLEX-KK-RM2-54mm_Lock_2pin_straight
Changed lines of the file:
@@
-EESchema Schematic File Version 2
+EESchema Schematic File Version 3
 LIBS:brain-rescue
-LIBS:power
-LIBS:device
-LIBS:transistors
-LIBS:conn
-LIBS:linear
-LIBS:regul
-LIBS:74xx
-LIBS:cmos4000
-LIBS:adc-dac
-LIBS:memory
-LIBS:xilinx
-LIBS:microcontrollers
-LIBS:dsp
-LIBS:microchip
-LIBS:analog_switches
-LIBS:motorola
-LIBS:texas
-LIBS:intel
-LIBS:audio
-LIBS:interface
-LIBS:digital-audio
-LIBS:philips
-LIBS:display
-LIBS:cypress
-LIBS:siliconi
-LIBS:opto
-LIBS:atmel
-LIBS:contrib
-LIBS:valves
 LIBS:espitall
 LIBS:brain-cache
-EELAYER 25 0
+EELAYER 26 0
 EELAYER END
 $Descr A4 11693 8268
@@
 F 0 "PWR1" V 3700 3700 40  0000 C CNN
 F 1 "CONN_2" V 3800 3700 40  0000 C CNN
-F 2 "Sockets_MOLEX_KK-System:Socket_MOLEX-KK-RM2-54mm_Lock_2pin_straight" H 3750 3700 60  0001 C CNN
+F 2 "espitall:Socket_MOLEX-KK-RM2-54mm_Lock_2pin_straight" H 3750 3700 60  0001 C CNN
 F 3 "" H 3750 3700 60  0000 C CNN
 	1    3750 3700
@@
 F 0 "C88" H 4450 3750 40  0000 L CNN
 F 1 "100u" H 4456 3565 40  0000 L CNN
-F 2 "Capacitors_SMD:c_elec_6.3x7.7" H 4488 3500 30  0001 C CNN
+F 2 "espitall:c_elec_6.3x7.7" H 4488 3500 30  0001 C CNN
 F 3 "" H 4450 3650 60  0000 C CNN
 	1    4450 3650
@@
 F 0 "C87" H 7150 3250 40  0000 L CNN
 F 1 "4u7" H 7156 3065 40  0000 L CNN
-F 2 "Capacitors_SMD:C_0603" H 7188 3000 30  0001 C CNN
+F 2 "espitall:C_0603" H 7188 3000 30  0001 C CNN
 F 3 "" H 7150 3150 60  0000 C CNN
 	1    7150 3150
@@
 F 0 "C89" H 7150 4500 40  0000 L CNN
 F 1 "4u7" H 7156 4315 40  0000 L CNN
-F 2 "Capacitors_SMD:C_0603" H 7188 4250 30  0001 C CNN
+F 2 "espitall:C_0603" H 7188 4250 30  0001 C CNN
 F 3 "" H 7150 4400 60  0000 C CNN
 	1    7150 4400

Commit message: add module add footprint SPSGRF-868 for future com board
Parts:
- C87, C88, C89: symbol C-RESCUE-brain -> brain-rescue:C-RESCUE-brain
- PWR1: symbol CONN_2 -> brain-rescue:CONN_2-RESCUE-brain
- U10: symbol TSR1-2433 -> espitall:TSR1-2433
- U9: symbol TSR1-2450 -> espitall:TSR1-2450
Changed lines of the file:
@@
-EESchema Schematic File Version 3
-LIBS:brain-rescue
-LIBS:espitall
+EESchema Schematic File Version 4
 LIBS:brain-cache
 EELAYER 26 0
@@
 $EndDescr
 $Comp
-L CONN_2 PWR1
+L brain-rescue:CONN_2-RESCUE-brain PWR1
 U 1 1 556E624F
 P 3750 3700
@@
 $EndComp
 $Comp
-L GND-RESCUE-brain #PWR0215
+L brain-rescue:GND-RESCUE-brain #PWR0215
 U 1 1 556E62AE
 P 4200 4100
@@
 $EndComp
 $Comp
-L +BATT #PWR0216
+L power:+BATT #PWR0216
 U 1 1 556E62C3
 P 4250 3150
@@
 $EndComp
 Wire Wire Line
-	4250 3150 4250 3600
+	4250 3150 4250 3350
 Wire Wire Line
 	4250 3600 4100 3600
@@
 	4100 3800 4200 3800
 Wire Wire Line
-	4200 3800 4200 4100
-$Comp
-L C-RESCUE-brain C88
+	4200 3800 4200 3950
+$Comp
+L brain-rescue:C-RESCUE-brain C88
 U 1 1 556E6F4F
 P 4450 3650
@@
 Connection ~ 4250 3350
 $Comp
-L TSR1-2450 U9
+L espitall:TSR1-2450 U9
 U 1 1 556E764E
 P 6450 2850
@@
 $EndComp
 $Comp
-L GND-RESCUE-brain #PWR0217
+L brain-rescue:GND-RESCUE-brain #PWR0217
 U 1 1 556E7685
 P 6450 3500
@@
 $EndComp
 $Comp
-L C-RESCUE-brain C87
+L brain-rescue:C-RESCUE-brain C87
 U 1 1 556E7699
 P 7150 3150
@@
 $EndComp
 $Comp
-L +BATT #PWR0218
+L power:+BATT #PWR0218
 U 1 1 556E76EB
 P 5850 2650
@@
 	6450 3100 6450 3500
 $Comp
-L GND-RESCUE-brain #PWR0219
+L brain-rescue:GND-RESCUE-brain #PWR0219
 U 1 1 556E7736
 P 7150 3450
@@
 	7150 3450 7150 3350
 Wire Wire Line
-	7150 2550 7150 2950
+	7150 2550 7150 2800
 Wire Wire Line
 	7150 2800 6850 2800
 $Comp
-L GND-RESCUE-brain #PWR0220
+L brain-rescue:GND-RESCUE-brain #PWR0220
 U 1 1 556E78DB
 P 6450 4750
@@
 $EndComp
 $Comp
-L C-RESCUE-brain C89
+L brain-rescue:C-RESCUE-brain C89
 U 1 1 556E78E1
 P 7150 4400
@@
 $EndComp
 $Comp
-L +BATT #PWR0221
+L power:+BATT #PWR0221
 U 1 1 556E78E7
 P 5850 3900
@@
 	6450 4350 6450 4750
 $Comp
-L GND-RESCUE-brain #PWR0222
+L brain-rescue:GND-RESCUE-brain #PWR0222
 U 1 1 556E78F0
 P 7150 4700
@@
 	7150 4700 7150 4600
 Wire Wire Line
-	7150 4000 7150 4200
+	7150 4000 7150 4050
 Wire Wire Line
 	7150 4050 6850 4050
 $Comp
-L TSR1-2433 U10
+L espitall:TSR1-2433 U10
 U 1 1 556E7AB0
 P 6450 4100
@@
 $EndComp
 $Comp
-L +5V #PWR0223
+L power:+5V #PWR0223
 U 1 1 556E7ACF
 P 7150 2550
@@
 $EndComp
 $Comp
-L +3V3 #PWR0224
+L power:+3V3 #PWR0224
 U 1 1 556E7AE9
 P 7150 4000
@@
 Connection ~ 7150 4050
 Connection ~ 7150 2800
+Wire Wire Line
+	4200 3950 4200 4100
+Wire Wire Line
+	4250 3350 4250 3600
+Wire Wire Line
+	7150 4050 7150 4200
+Wire Wire Line
+	7150 2800 7150 2950
 $EndSCHEMATC
