File: brain/usir.sch (KiCad schematic (older format))
At the start: 31 parts

Commit message: updated schematic of brain board
Parts:
- R? (x8): value R -> 1k
Changed lines of the file:
@@
 $Descr A4 11693 8268
 encoding utf-8
-Sheet 3 4
+Sheet 2 8
 Title ""
 Date ""
@@
 P 8450 3050
 F 0 "R?" V 8530 3050 40  0000 C CNN
-F 1 "R" V 8457 3051 40  0000 C CNN
+F 1 "1k" V 8457 3051 40  0000 C CNN
 F 2 "" V 8380 3050 30  0000 C CNN
 F 3 "" H 8450 3050 30  0000 C CNN
@@
 P 9050 3400
 F 0 "R?" V 9130 3400 40  0000 C CNN
-F 1 "R" V 9057 3401 40  0000 C CNN
+F 1 "1k" V 9057 3401 40  0000 C CNN
 F 2 "" V 8980 3400 30  0000 C CNN
 F 3 "" H 9050 3400 30  0000 C CNN
@@
 P 8450 4950
 F 0 "R?" V 8530 4950 40  0000 C CNN
-F 1 "R" V 8457 4951 40  0000 C CNN
+F 1 "1k" V 8457 4951 40  0000 C CNN
 F 2 "" V 8380 4950 30  0000 C CNN
 F 3 "" H 8450 4950 30  0000 C CNN
@@
 P 9050 5300
 F 0 "R?" V 9130 5300 40  0000 C CNN
-F 1 "R" V 9057 5301 40  0000 C CNN
+F 1 "1k" V 9057 5301 40  0000 C CNN
 F 2 "" V 8980 5300 30  0000 C CNN
 F 3 "" H 9050 5300 30  0000 C CNN
@@
 P 4650 4950
 F 0 "R?" V 4730 4950 40  0000 C CNN
-F 1 "R" V 4657 4951 40  0000 C CNN
+F 1 "1k" V 4657 4951 40  0000 C CNN
 F 2 "" V 4580 4950 30  0000 C CNN
 F 3 "" H 4650 4950 30  0000 C CNN
@@
 P 5250 5300
 F 0 "R?" V 5330 5300 40  0000 C CNN
-F 1 "R" V 5257 5301 40  0000 C CNN
+F 1 "1k" V 5257 5301 40  0000 C CNN
 F 2 "" V 5180 5300 30  0000 C CNN
 F 3 "" H 5250 5300 30  0000 C CNN
@@
 P 4650 6850
 F 0 "R?" V 4730 6850 40  0000 C CNN
-F 1 "R" V 4657 6851 40  0000 C CNN
+F 1 "1k" V 4657 6851 40  0000 C CNN
 F 2 "" V 4580 6850 30  0000 C CNN
 F 3 "" H 4650 6850 30  0000 C CNN
@@
 P 5250 7200
 F 0 "R?" V 5330 7200 40  0000 C CNN
-F 1 "R" V 5257 7201 40  0000 C CNN
+F 1 "1k" V 5257 7201 40  0000 C CNN
 F 2 "" V 5180 7200 30  0000 C CNN
 F 3 "" H 5250 7200 30  0000 C CNN

Commit message: footprint assignation
Parts:
- C1, C10, C11, C12, C13, C14, C2, C3, C4, C5, C6, C7, C8, C9: renamed from C?; footprint (none) -> Capacitors_SMD:C_0603
- IR0: footprint (none) -> Sockets_MOLEX_KK-System:Socket_MOLEX-KK-RM2-54mm_Lock_3pin_straight
- IR1, IR2, IR3: renamed from IR?; footprint (none) -> Sockets_MOLEX_KK-System:Socket_MOLEX-KK-RM2-54mm_Lock_3pin_straight
- R1, R2, R3, R4, R5, R6, R7, R8: renamed from R?; footprint (none) -> Resistors_SMD:R_0603
- U1: renamed from U?; footprint (none) -> Housings_SSOP:TSSOP-20_4.4x6.5mm_Pitch0.65mm
- US0, US1, US2, US3: footprint (none) -> Sockets_MOLEX_KK-System:Socket_MOLEX-KK-RM2-54mm_Lock_4pin_straight

Commit message: Brain 2018 layout
Parts:
- removed C2: 100n, Capacitors_SMD:C_0603, symbol C
- removed U1: TXB0108, Housings_SSOP:TSSOP-20_4.4x6.5mm_Pitch0.65mm, symbol TXB0108
- added R13, R14, R15, R16, R33, R43, R44, R9: 1k, Resistors_SMD:R_0603, symbol R-RESCUE-brain
- added U1: SN74AHCT125PW, Housings_SSOP:TSSOP-14_4.4x5mm_Pitch0.65mm, symbol SN74AHCT125PW
- C1, C10, C11, C12, C13, C14, C3, C4, C5, C6, C7, C8, C9: symbol C -> C-RESCUE-brain
- R1, R2, R3, R4, R5, R6, R7, R8: symbol R -> R-RESCUE-brain
Connections:
- net labels removed: +3V3
- wire segments 113 -> 118

Commit message: add 3d step files to brain
Parts:
- C1, C10, C11, C12, C13, C14, C3, C4, C5, C6, C7, C8, C9: footprint Capacitors_SMD:C_0603 -> espitall:C_0603
- IR0, IR1, IR2, IR3: footprint Sockets_MOLEX_KK-System:Socket_MOLEX-KK-RM2-54mm_Lock_3pin_straight -> espitall:Socket_MOLEX-KK-RM2-54mm_Lock_3pin_straight
- R1, R13, R14, R15, R16, R2, R3, R33, R4, R43, R44, R5, R6, R7, R8, R9: footprint Resistors_SMD:R_0603 -> espitall:R_0603
- U1: footprint Housings_SSOP:TSSOP-14_4.4x5mm_Pitch0.65mm -> espitall:TSSOP-14_4.4x5mm_Pitch0.65mm
- US0, US1, US2, US3: footprint Sockets_MOLEX_KK-System:Socket_MOLEX-KK-RM2-54mm_Lock_4pin_straight -> espitall:Socket_MOLEX-KK-RM2-54mm_Lock_4pin_straight

Commit message: add module add footprint SPSGRF-868 for future com board
Parts:
- C1, C10, C11, C12, C13, C14, C3, C4, C5, C6, C7, C8, C9: symbol C-RESCUE-brain -> brain-rescue:C-RESCUE-brain
- IR0, IR1, IR2, IR3: symbol CONN_3 -> brain-rescue:CONN_3-RESCUE-brain
- R1, R13, R14, R15, R16, R2, R3, R33, R4, R43, R44, R5, R6, R7, R8, R9: symbol R-RESCUE-brain -> brain-rescue:R-RESCUE-brain
- U1: symbol SN74AHCT125PW -> espitall:SN74AHCT125PW
- US0, US1, US2, US3: symbol CONN_4 -> brain-rescue:CONN_4-RESCUE-brain
Connections:
- wire segments 118 -> 143
