File: cocoout/Cocoout.kicad_pcb (KiCad board)
At the start: 2 copper layers, 50 x 50 mm, 55 parts, among them P0 CONN_01X04, P1 CONN_01X04, P2 CONN_01X04, P3 CONN_01X04, P4 CONN_01X04, P5 CONN_01X04, P6 CONN_01X04, P7 CONN_01X03, P8 CONN_01X07, P9 CONN_01X07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

Commit message: ad 3d step files to cocoout
Parts:
- C1: footprint Capacitors_SMD:C_0805_HandSoldering -> espitall:C_0805_HandSoldering
- C2: footprint Capacitors_SMD:C_0603_HandSoldering -> espitall:C_0603_HandSoldering
- D0, D1, D16, D2, D3, D4, D5, D6, D7: footprint Diodes_SMD:D_0805 -> espitall:D_0805
- D10, D11, D12, D14, D15, D8, D9: footprint Diodes_SMD:D_SMA_Handsoldering -> espitall:D_SMA_Handsoldering
- H1, H2, H3: footprint Mounting_Holes:MountingHole_3.2mm_M3_Pad -> Mounting_Holes:MountingHole_3.2mm_M3
- P0, P1, P2, P3, P4, P5, P6: footprint Sockets_MOLEX_KK-System:Socket_MOLEX-KK-RM2-54mm_Lock_4pin_straight -> espitall:Socket_MOLEX-KK-RM2-54mm_Lock_4pin_straight
- P7: footprint Sockets_MOLEX_KK-System:Socket_MOLEX-KK-RM2-54mm_Lock_3pin_straight -> espitall:Socket_MOLEX-KK-RM2-54mm_Lock_3pin_straight
- Q1, Q2, Q3, Q4, Q5, Q7, Q8: footprint TO_SOT_Packages_SMD:SOT-23 -> espitall:SOT-23
- R1, R11, R12, R13, R14, R15, R16, R17, R2, R3, R4, R5, R6, R7, R8, R9: footprint Resistors_SMD:R_0603_HandSoldering -> espitall:R_0603_HandSoldering
- U1: footprint Housings_SSOP:TSSOP-16_4.4x5mm_Pitch0.65mm -> espitall:TSSOP-16_4.4x5mm_Pitch0.65mm
Connections:
- H1 pad 1: (no net) -> Net-(H1-Pad1)
- H2 pad 1: (no net) -> Net-(H2-Pad1)
- H3 pad 1: (no net) -> Net-(H3-Pad1)
