File: cocoout/Cocoout.sch (KiCad schematic (older format))
At the start: 58 parts, among them P0 CONN_01X04, P1 CONN_01X04, P2 CONN_01X04, P3 CONN_01X04, P4 CONN_01X04, P5 CONN_01X04, P6 CONN_01X04, P7 CONN_01X04, P8 CONN_01X07, P9 CONN_01X07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

Commit message: Schematic and footprint asignment of CocoOUT board
Parts:
- removed Q1, Q2, Q3, Q4, Q5, Q6, Q7, Q8: Q_NMOS_GDSD, symbol Q_NMOS_GDSD
- added C2: 100n, Capacitors_SMD:C_0603_HandSoldering, symbol C
- added Q1, Q2, Q3, Q4, Q5, Q6, Q7, Q8: DMN2041L-7, TO_SOT_Packages_SMD:SOT-23, symbol Q_NMOS_GSD
- C1: footprint (none) -> Capacitors_SMD:C_0805_HandSoldering
- D0, D1, D16, D2, D3, D4, D5, D6, D7: footprint (none) -> Diodes_SMD:D_0805; symbol LED -> LED-RESCUE-Cocoout
- D10, D11, D12, D13, D14, D15, D8, D9: footprint (none) -> Diodes_SMD:D_SMA_Handsoldering
- H1, H2, H3, H4: footprint (none) -> Mounting_Holes:MountingHole_3.2mm_M3_Pad
- P0, P1, P2, P3, P4, P5, P6, P7: footprint (none) -> Sockets_MOLEX_KK-System:Socket_MOLEX-KK-RM2-54mm_Lock_4pin_straight
- P8, P9: footprint (none) -> espitall:Socket_MOLEX-KK-RM2-54mm_Lock_7pin_straight
- R1, R10, R11, R12, R13, R14, R15, R16, R17, R2, R3, R4, R5, R6, R7, R8, R9: footprint (none) -> Resistors_SMD:R_0603_HandSoldering
- U1: footprint (none) -> Housings_SSOP:TSSOP-16_4.4x5mm_Pitch0.65mm
Connections:
- wire segments 211 -> 205

Commit message: Layout of CocoOUT board
Parts:
- removed D13: D, Diodes_SMD:D_SMA_Handsoldering, symbol D
- removed H4: CONN_01X01, Mounting_Holes:MountingHole_3.2mm_M3_Pad, symbol CONN_01X01
- removed P7: CONN_01X04, Sockets_MOLEX_KK-System:Socket_MOLEX-KK-RM2-54mm_Lock_4pin_straight, symbol CONN_01X04
- removed Q6: DMN2041L-7, TO_SOT_Packages_SMD:SOT-23, symbol Q_NMOS_GSD
- removed R10: R, Resistors_SMD:R_0603_HandSoldering, symbol R
- added P7: CONN_01X03, Sockets_MOLEX_KK-System:Socket_MOLEX-KK-RM2-54mm_Lock_3pin_straight, symbol CONN_01X03
Connections:
- net labels removed: VDD
- wire segments 205 -> 194

Commit message: ad 3d step files to cocoout
Parts:
- C1: footprint Capacitors_SMD:C_0805_HandSoldering -> espitall:C_0805_HandSoldering
- C2: footprint Capacitors_SMD:C_0603_HandSoldering -> espitall:C_0603_HandSoldering
- D0, D1, D16, D2, D3, D4, D5, D6, D7: footprint Diodes_SMD:D_0805 -> espitall:D_0805
- D10, D11, D12, D14, D15, D8, D9: footprint Diodes_SMD:D_SMA_Handsoldering -> espitall:D_SMA_Handsoldering
- H1, H2, H3: footprint Mounting_Holes:MountingHole_3.2mm_M3_Pad -> Mounting_Holes:MountingHole_3.2mm_M3
- P0, P1, P2, P3, P4, P5, P6: footprint Sockets_MOLEX_KK-System:Socket_MOLEX-KK-RM2-54mm_Lock_4pin_straight -> espitall:Socket_MOLEX-KK-RM2-54mm_Lock_4pin_straight
- P7: footprint Sockets_MOLEX_KK-System:Socket_MOLEX-KK-RM2-54mm_Lock_3pin_straight -> espitall:Socket_MOLEX-KK-RM2-54mm_Lock_3pin_straight
- Q1, Q2, Q3, Q4, Q5, Q7, Q8: footprint TO_SOT_Packages_SMD:SOT-23 -> espitall:SOT-23
- R1, R11, R12, R13, R14, R15, R16, R17, R2, R3, R4, R5, R6, R7, R8, R9: footprint Resistors_SMD:R_0603_HandSoldering -> espitall:R_0603_HandSoldering
- U1: footprint Housings_SSOP:TSSOP-16_4.4x5mm_Pitch0.65mm -> espitall:TSSOP-16_4.4x5mm_Pitch0.65mm
