File: cocoin/Cocoin.sch (KiCad schematic (older format))
At the start: 42 parts, among them P0 CONN_01X03, P1 CONN_01X03, P2 CONN_01X03, P3 CONN_01X03, P4 CONN_01X03, P5 CONN_01X03, P6 CONN_01X03, P7 CONN_01X03, P8 CONN_01X07, P9 CONN_01X07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

Commit message: schematic and layout of CocoIN 2018
Parts:
- removed H4: CONN_01X01, symbol CONN_01X01
- added C10: 100n, Capacitors_SMD:C_0603_HandSoldering, symbol C
- C1: footprint (none) -> Capacitors_SMD:C_0805_HandSoldering
- C2, C3, C4, C5, C6, C7, C8, C9: footprint (none) -> Capacitors_SMD:C_0603_HandSoldering
- D16: footprint (none) -> LEDs:LED_0805; symbol LED -> LED-RESCUE-Cocoin
- H1, H2, H3: footprint (none) -> Mounting_Holes:MountingHole_3.2mm_M3_Pad
- P0, P1, P2, P3, P4, P5, P6, P7: footprint (none) -> Sockets_MOLEX_KK-System:Socket_MOLEX-KK-RM2-54mm_Lock_3pin_straight
- P8, P9: footprint (none) -> espitall:Socket_MOLEX-KK-RM2-54mm_Lock_7pin_straight
- R1, R10, R11, R12, R13, R14, R15, R16, R17, R2, R3, R4, R5, R6, R7, R8, R9: footprint (none) -> Resistors_SMD:R_0603_HandSoldering
- U1: footprint (none) -> Housings_SSOP:TSSOP-16_4.4x5mm_Pitch0.65mm
Connections:
- wire segments 119 -> 121
- no-connect marks 5 -> 4
Other:
- note added: "Inputs"
- note removed: "Input"

Commit message: ad 3d step files to cocoin
Parts:
- C1: footprint Capacitors_SMD:C_0805_HandSoldering -> espitall:C_0805_HandSoldering
- C10, C2, C3, C4, C5, C6, C7, C8, C9: footprint Capacitors_SMD:C_0603_HandSoldering -> espitall:C_0603_HandSoldering
- D16: footprint LEDs:LED_0805 -> espitall:LED_0805
- H1, H2, H3: footprint Mounting_Holes:MountingHole_3.2mm_M3_Pad -> Mounting_Holes:MountingHole_3.2mm_M3
- P0, P1, P2, P3, P4, P5, P6, P7: footprint Sockets_MOLEX_KK-System:Socket_MOLEX-KK-RM2-54mm_Lock_3pin_straight -> espitall:Socket_MOLEX-KK-RM2-54mm_Lock_3pin_straight
- R1, R10, R11, R12, R13, R14, R15, R16, R17, R2, R3, R4, R5, R6, R7, R8, R9: footprint Resistors_SMD:R_0603_HandSoldering -> espitall:R_0603_HandSoldering
- U1: footprint Housings_SSOP:TSSOP-16_4.4x5mm_Pitch0.65mm -> espitall:TSSOP-16_4.4x5mm_Pitch0.65mm
