File: cocoservo/Cocoservo.sch (KiCad schematic (older format))
At the start: 21 parts, among them P0 CONN_01X03, P1 CONN_01X03, P2 CONN_01X03, P3 CONN_01X03, P4 CONN_01X02, P5 CONN_01X02, P6 CONN_01X05, U1 TSR1-2450

Commit message: layout of cocoservo 2018 board
Parts:
- removed H4: CONN_01X01, symbol CONN_01X01
- C1, C2: footprint (none) -> Capacitors_SMD:C_0805_HandSoldering
- C3: footprint (none) -> Capacitors_SMD:C_0603_HandSoldering
- D1: footprint (none) -> LEDs:LED_0805; symbol LED -> LED-RESCUE-Cocoservo
- H1, H2, H3: footprint (none) -> Mounting_Holes:MountingHole_3.2mm_M3_Pad
- PIN1: renamed from P4; footprint (none) -> Connectors_Molex:Molex_KK-6410-02_02x2.54mm_Straight
- POUT1: renamed from P5; footprint (none) -> Connectors_Molex:Molex_KK-6410-02_02x2.54mm_Straight
- R1, R2, R3, R4, R5: footprint (none) -> Resistors_SMD:R_0603_HandSoldering
- S0: renamed from P0; footprint (none) -> Connectors_Molex:Molex_KK-6410-03_03x2.54mm_Straight
- S1: renamed from P1; footprint (none) -> Connectors_Molex:Molex_KK-6410-03_03x2.54mm_Straight
- S2: renamed from P2; footprint (none) -> Connectors_Molex:Molex_KK-6410-03_03x2.54mm_Straight
- S3: renamed from P3; footprint (none) -> Connectors_Molex:Molex_KK-6410-03_03x2.54mm_Straight
- SIN1: renamed from P6; footprint (none) -> Connectors_Molex:Molex_KK-6410-05_05x2.54mm_Straight
- U1: footprint (none) -> espitall:TSR-1
Connections:
- net labels added: servo_0_5v, servo_1_5v, servo_2_5v, servo_3_5v
- net labels removed: servo_0_3v3, servo_1_3v3, servo_2_3v3, servo_3_3v3
- no-connect marks 4 -> 0
Other:
- moved on the sheet: H3
Changed lines of the file:
@@
 EESchema Schematic File Version 2
+LIBS:Cocoservo-rescue
 LIBS:xilinx
 LIBS:video
@@
 $EndComp
 $Comp
-L LED D1
+L LED-RESCUE-Cocoservo D1
 U 1 1 573CEA8D
 P 6650 1700
 F 0 "D1" H 6650 1800 50  0000 C CNN
 F 1 "LED" H 6650 1600 50  0000 C CNN
-F 2 "" H 6650 1700 50  0000 C CNN
+F 2 "LEDs:LED_0805" H 6650 1700 50  0001 C CNN
 F 3 "" H 6650 1700 50  0000 C CNN
 	1    6650 1700
@@
 F 0 "R1" V 6730 1300 50  0000 C CNN
 F 1 "330" V 6650 1300 50  0000 C CNN
-F 2 "" H 6650 1300 50  0000 C CNN
+F 2 "Resistors_SMD:R_0603_HandSoldering" H 6650 1300 50  0001 C CNN
 F 3 "" H 6650 1300 50  0000 C CNN
 	1    6650 1300
@@
 F 0 "H1" H 9200 1400 50  0000 C CNN
 F 1 "CONN_01X01" V 9300 1300 50  0000 C CNN
-F 2 "" H 9200 1300 50  0000 C CNN
+F 2 "Mounting_Holes:MountingHole_3.2mm_M3_Pad" H 9200 1300 50  0001 C CNN
 F 3 "" H 9200 1300 50  0000 C CNN
 	1    9200 1300
@@
 F 0 "H2" H 9800 1400 50  0000 C CNN
 F 1 "CONN_01X01" V 9900 1300 50  0000 C CNN
-F 2 "" H 9800 1300 50  0000 C CNN
+F 2 "Mounting_Holes:MountingHole_3.2mm_M3_Pad" H 9800 1300 50  0001 C CNN
 F 3 "" H 9800 1300 50  0000 C CNN
 	1    9800 1300
@@
 Text Notes 9100 850  0    60   ~ 0
 Mouting holes
-NoConn ~ 9200 1500
-NoConn ~ 9800 1500
 $Comp
 L C C1
@@
 F 0 "C1" H 3200 1600 50  0000 C CNN
 F 1 "10u" V 3250 1350 50  0000 C CNN
-F 2 "" H 3150 1500 50  0000 C CNN
+F 2 "Capacitors_SMD:C_0805_HandSoldering" H 3150 1500 50  0001 C CNN
 F 3 "" H 3150 1500 50  0000 C CNN
 	1    3150 1500
@@
 Power led
 Text Label 1200 1600 0    60   ~ 0
-servo_3_3v3
+servo_3_5v
 Text Label 1200 1500 0    60   ~ 0
-servo_2_3v3
+servo_2_5v
 Text Label 1200 1400 0    60   ~ 0
-servo_1_3v3
+servo_1_5v
 Text Label 1200 1300 0    60   ~ 0
-servo_0_3v3
+servo_0_5v
 Text Notes 600  2750 0    60   ~ 0
 Servo output
@@
 L CONN_01X01 H3
 U 1 1 57889E4C
-P 9200 1800
-F 0 "H3" H 9200 1900 50  0000 C CNN
-F 1 "CONN_01X01" V 9300 1800 50  0000 C CNN
-F 2 "" H 9200 1800 50  0000 C CNN
-F 3 "" H 9200 1800 50  0000 C CNN
-	1    9200 1800
+P 9200 1950
+F 0 "H3" H 9200 2050 50  0000 C CNN
+F 1 "CONN_01X01" V 9300 1950 50  0000 C CNN
+F 2 "Mounting_Holes:MountingHole_3.2mm_M3_Pad" H 9200 1950 50  0001 C CNN
+F 3 "" H 9200 1950 50  0000 C CNN
+	1    9200 1950
 	0    -1   -1   0
 $EndComp
 $Comp
-L CONN_01X01 H4
-U 1 1 57889E52
-P 9800 1800
-F 0 "H4" H 9800 1900 50  0000 C CNN
-F 1 "CONN_01X01" V 9900 1800 50  0000 C CNN
-F 2 "" H 9800 1800 50  0000 C CNN
-F 3 "" H 9800 1800 50  0000 C CNN
-	1    9800 1800
-	0    -1   -1   0
-$EndComp
-NoConn ~ 9200 2000
-NoConn ~ 9800 2000
-$Comp
-L CONN_01X03 P0
+L CONN_01X03 S0
 U 1 1 5787B6B2
 P 4850 4000
-F 0 "P0" H 4850 4200 50  0000 C CNN
+F 0 "S0" H 4850 4200 50  0000 C CNN
 F 1 "CONN_01X03" V 4950 4000 50  0000 C CNN
-F 2 "" H 4850 4000 50  0000 C CNN
+F 2 "Connectors_Molex:Molex_KK-6410-03_03x2.54mm_Straight" H 4850 4000 50  0001 C CNN
 F 3 "" H 4850 4000 50  0000 C CNN
 	1    4850 4000
@@
 F 0 "R2" V 4380 3750 50  0000 C CNN
 F 1 "10k" V 4300 3750 50  0000 C CNN
-F 2 "" V 4230 3750 50  0000 C CNN
+F 2 "Resistors_SMD:R_0603_HandSoldering" V 4230 3750 50  0001 C CNN
 F 3 "" H 4300 3750 50  0000 C CNN
 	1    4300 3750
@@
 Connection ~ 4300 4000
 Text Label 3300 4000 0    60   ~ 0
-servo_0_3v3
-$Comp
-L CONN_01X03 P1
+servo_0_5v
+$Comp
+L CONN_01X03 S1
 U 1 1 5787D99C
 P 6750 4000
-F 0 "P1" H 6750 4200 50  0000 C CNN
+F 0 "S1" H 6750 4200 50  0000 C CNN
 F 1 "CONN_01X03" V 6850 4000 50  0000 C CNN
-F 2 "" H 6750 4000 50  0000 C CNN
+F 2 "Connectors_Molex:Molex_KK-6410-03_03x2.54mm_Straight" H 6750 4000 50  0001 C CNN
 F 3 "" H 6750 4000 50  0000 C CNN
 	1    6750 4000
@@
 F 0 "R3" V 6280 3750 50  0000 C CNN
 F 1 "10k" V 6200 3750 50  0000 C CNN
-F 2 "" V 6130 3750 50  0000 C CNN
+F 2 "Resistors_SMD:R_0603_HandSoldering" V 6130 3750 50  0001 C CNN
 F 3 "" H 6200 3750 50  0000 C CNN
 	1    6200 3750
@@
 Connection ~ 6200 4000
 Text Label 5200 4000 0    60   ~ 0
-servo_1_3v3
-$Comp
-L CONN_01X03 P2
+servo_1_5v
+$Comp
+L CONN_01X03 S2
 U 1 1 5787DBB0
 P 4850 5650
-F 0 "P2" H 4850 5850 50  0000 C CNN
+F 0 "S2" H 4850 5850 50  0000 C CNN
 F 1 "CONN_01X03" V 4950 5650 50  0000 C CNN
-F 2 "" H 4850 5650 50  0000 C CNN
+F 2 "Connectors_Molex:Molex_KK-6410-03_03x2.54mm_Straight" H 4850 5650 50  0001 C CNN
 F 3 "" H 4850 5650 50  0000 C CNN
 	1    4850 5650
@@
 F 0 "R4" V 4380 5400 50  0000 C CNN
 F 1 "10k" V 4300 5400 50  0000 C CNN
-F 2 "" V 4230 5400 50  0000 C CNN
+F 2 "Resistors_SMD:R_0603_HandSoldering" V 4230 5400 50  0001 C CNN
 F 3 "" H 4300 5400 50  0000 C CNN
 	1    4300 5400
@@
 Connection ~ 4300 5650
 Text Label 3300 5650 0    60   ~ 0
-servo_2_3v3
-$Comp
-L CONN_01X03 P3
+servo_2_5v
+$Comp
+L CONN_01X03 S3
 U 1 1 5787DBD3
 P 6750 5650
-F 0 "P3" H 6750 5850 50  0000 C CNN
+F 0 "S3" H 6750 5850 50  0000 C CNN
 F 1 "CONN_01X03" V 6850 5650 50  0000 C CNN
-F 2 "" H 6750 5650 50  0000 C CNN
+F 2 "Connectors_Molex:Molex_KK-6410-03_03x2.54mm_Straight" H 6750 5650 50  0001 C CNN
 F 3 "" H 6750 5650 50  0000 C CNN
 	1    6750 5650
@@
 F 0 "R5" V 6280 5400 50  0000 C CNN
 F 1 "10k" V 6200 5400 50  0000 C CNN
-F 2 "" V 6130 5400 50  0000 C CNN
+F 2 "Resistors_SMD:R_0603_HandSoldering" V 6130 5400 50  0001 C CNN
 F 3 "" H 6200 5400 50  0000 C CNN
 	1    6200 5400
@@
 Connection ~ 6200 5650
 Text Label 5200 5650 0    60   ~ 0
-servo_3_3v3
-$Comp
-L CONN_01X05 P6
+servo_3_5v
+$Comp
+L CONN_01X05 SIN1
 U 1 1 5787DF50
 P 950 1500
-F 0 "P6" H 950 1800 50  0000 C CNN
+F 0 "SIN1" H 950 1800 50  0000 C CNN
 F 1 "CONN_01X05" V 1050 1500 50  0000 C CNN
-F 2 "" H 950 1500 50  0000 C CNN
+F 2 "Connectors_Molex:Molex_KK-6410-05_05x2.54mm_Straight" H 950 1500 50  0001 C CNN
 F 3 "" H 950 1500 50  0000 C CNN
 	1    950  1500
@@
 F 0 "U1" H 4300 1104 60  0000 C CNN
 F 1 "TSR1-2450" H 4150 1500 60  0000 C CNN
-F 2 "" H 4150 1300 60  0000 C CNN
+F 2 "espitall:TSR-1" H 4150 1300 60  0001 C CNN
 F 3 "" H 4150 1300 60  0000 C CNN
 	1    4150 1300
@@
 F 0 "C2" H 4900 1600 50  0000 C CNN
 F 1 "10u" V 4950 1350 50  0000 C CNN
-F 2 "" H 4850 1500 50  0000 C CNN
+F 2 "Capacitors_SMD:C_0805_HandSoldering" H 4850 1500 50  0001 C CNN
 F 3 "" H 4850 1500 50  0000 C CNN
 	1    4850 1500
@@
 F 0 "C3" H 5200 1600 50  0000 C CNN
 F 1 "100n" V 5250 1350 50  0000 C CNN
-F 2 "" H 5150 1500 50  0000 C CNN
+F 2 "Capacitors_SMD:C_0603_HandSoldering" H 5150 1500 50  0001 C CNN
 F 3 "" H 5150 1500 50  0000 C CNN
 	1    5150 1500
@@
 	2400 500  2400 2600
 $Comp
-L CONN_01X02 P4
+L CONN_01X02 PIN1
 U 1 1 5787F44A
 P 2750 1250
-F 0 "P4" H 2750 1400 50  0000 C CNN
+F 0 "PIN1" H 2750 1400 50  0000 C CNN
 F 1 "CONN_01X02" V 2850 1250 50  0000 C CNN
-F 2 "" H 2750 1250 50  0000 C CNN
+F 2 "Connectors_Molex:Molex_KK-6410-02_02x2.54mm_Straight" H 2750 1250 50  0001 C CNN
 F 3 "" H 2750 1250 50  0000 C CNN
 	1    2750 1250
@@
 Connection ~ 3150 1200
 $Comp
-L CONN_01X02 P5
+L CONN_01X02 POUT1
 U 1 1 5787F6B6
 P 5650 1250
-F 0 "P5" H 5650 1400 50  0000 C CNN
+F 0 "POUT1" H 5650 1400 50  0000 C CNN
 F 1 "CONN_01X02" V 5750 1250 50  0000 C CNN
-F 2 "" H 5650 1250 50  0000 C CNN
+F 2 "Connectors_Molex:Molex_KK-6410-02_02x2.54mm_Straight" H 5650 1250 50  0001 C CNN
 F 3 "" H 5650 1250 50  0000 C CNN
 	1    5650 1250
@@
 Wire Wire Line
 	5350 1300 5450 1300
+$Comp
+L GND #PWR020
+U 1 1 592C8E28
+P 9200 2150
+F 0 "#PWR020" H 9200 1900 50  0001 C CNN
+F 1 "GND" H 9200 2000 50  0000 C CNN
+F 2 "" H 9200 2150 50  0000 C CNN
+F 3 "" H 9200 2150 50  0000 C CNN
+	1    9200 2150
+	1    0    0    -1
+$EndComp
+$Comp
+L GND #PWR021
+U 1 1 592C8EE6
+P 9800 1500
+F 0 "#PWR021" H 9800 1250 50  0001 C CNN
+F 1 "GND" H 9800 1350 50  0000 C CNN
+F 2 "" H 9800 1500 50  0000 C CNN
+F 3 "" H 9800 1500 50  0000 C CNN
+	1    9800 1500
+	1    0    0    -1
+$EndComp
+$Comp
+L GND #PWR022
+U 1 1 592C8F45
+P 9200 1500
+F 0 "#PWR022" H 9200 1250 50  0001 C CNN
+F 1 "GND" H 9200 1350 50  0000 C CNN
+F 2 "" H 9200 1500 50  0000 C CNN
+F 3 "" H 9200 1500 50  0000 C CNN
+	1    9200 1500
+	1    0    0    -1
+$EndComp
 $EndSCHEMATC

Commit message: ad 3d step files to cocoservo
Parts:
- C1, C2: footprint Capacitors_SMD:C_0805_HandSoldering -> espitall:C_0805_HandSoldering
- C3: footprint Capacitors_SMD:C_0603_HandSoldering -> espitall:C_0603_HandSoldering
- D1: footprint LEDs:LED_0805 -> espitall:LED_0805
- H1, H2, H3: footprint Mounting_Holes:MountingHole_3.2mm_M3_Pad -> Mounting_Holes:MountingHole_3.2mm_M3
- PIN1, POUT1: footprint Connectors_Molex:Molex_KK-6410-02_02x2.54mm_Straight -> espitall:Socket_MOLEX-KK-RM2-54mm_Lock_2pin_straight
- R1, R2, R3, R4, R5: footprint Resistors_SMD:R_0603_HandSoldering -> espitall:R_0603_HandSoldering
- S0, S1, S2, S3: footprint Connectors_Molex:Molex_KK-6410-03_03x2.54mm_Straight -> espitall:Socket_MOLEX-KK-RM2-54mm_Lock_3pin_straight
- SIN1: footprint Connectors_Molex:Molex_KK-6410-05_05x2.54mm_Straight -> espitall:Socket_MOLEX-KK-RM2-54mm_Lock_5pin_straight
Changed lines of the file:
@@
-EESchema Schematic File Version 2
+EESchema Schematic File Version 3
 LIBS:Cocoservo-rescue
-LIBS:xilinx
-LIBS:video
-LIBS:valves
-LIBS:ttl_ieee
-LIBS:transistors
-LIBS:transf
-LIBS:texas
-LIBS:switches
-LIBS:supertex
-LIBS:stm8
-LIBS:stm32
-LIBS:siliconi
-LIBS:silabs
-LIBS:sensors
-LIBS:rfcom
-LIBS:relays
-LIBS:regul
-LIBS:references
-LIBS:powerint
-LIBS:power
-LIBS:philips
-LIBS:opto
-LIBS:onsemi
-LIBS:nxp_armmcu
-LIBS:nordicsemi
-LIBS:msp430
-LIBS:motorola
-LIBS:motor_drivers
-LIBS:microcontrollers
-LIBS:microchip_pic32mcu
-LIBS:microchip_pic18mcu
-LIBS:microchip_pic16mcu
-LIBS:microchip_pic12mcu
-LIBS:microchip_pic10mcu
-LIBS:microchip_dspic33dsc
-LIBS:microchip
-LIBS:memory
-LIBS:maxim
-LIBS:logo
-LIBS:linear
-LIBS:ir
-LIBS:interface
-LIBS:intel
-LIBS:hc11
-LIBS:graphic
-LIBS:gennum
-LIBS:ftdi
-LIBS:elec-unifil
-LIBS:dsp
-LIBS:display
-LIBS:diode
-LIBS:digital-audio
-LIBS:device
-LIBS:dc-dc
-LIBS:cypress
-LIBS:contrib
-LIBS:conn
-LIBS:cmos_ieee
-LIBS:cmos4000
-LIBS:brooktre
-LIBS:audio
-LIBS:atmel
-LIBS:analog_switches
-LIBS:analog_devices
-LIBS:adc-dac
-LIBS:actel
-LIBS:ac-dc
-LIBS:Zilog
-LIBS:Xicor
-LIBS:Power_Management
-LIBS:Oscillators
-LIBS:Lattice
-LIBS:ESD_Protection
-LIBS:Altera
-LIBS:74xx
-LIBS:74xgxx
-LIBS:Symbols_Transformer-Diskrete_RevA
-LIBS:Symbols_Socket-DIN41612_RevA
-LIBS:Symbols_Microcontroller_Philips-NXP_RevA_06Oct2013
-LIBS:Symbols_ICs-Opto_RevB_16Sep2013
-LIBS:Symbols_ICs-Diskrete_RevD10
-LIBS:Symbols_EN60617_13Mar2013
-LIBS:Symbols_EN60617-10_HF-Radio_DRAFT_12Sep2013
-LIBS:Symbols_DCDC-ACDC-Converter_RevC_20Jul2012
-LIBS:SymbolsSimilarEN60617+oldDIN617-RevE8
 LIBS:espitall
 LIBS:Cocoservo-cache
-EELAYER 25 0
+EELAYER 26 0
 EELAYER END
 $Descr A4 11693 8268
@@
 F 0 "D1" H 6650 1800 50  0000 C CNN
 F 1 "LED" H 6650 1600 50  0000 C CNN
-F 2 "LEDs:LED_0805" H 6650 1700 50  0001 C CNN
+F 2 "espitall:LED_0805" H 6650 1700 50  0001 C CNN
 F 3 "" H 6650 1700 50  0000 C CNN
 	1    6650 1700
@@
 F 0 "R1" V 6730 1300 50  0000 C CNN
 F 1 "330" V 6650 1300 50  0000 C CNN
-F 2 "Resistors_SMD:R_0603_HandSoldering" H 6650 1300 50  0001 C CNN
+F 2 "espitall:R_0603_HandSoldering" H 6650 1300 50  0001 C CNN
 F 3 "" H 6650 1300 50  0000 C CNN
 	1    6650 1300
@@
 F 0 "H1" H 9200 1400 50  0000 C CNN
 F 1 "CONN_01X01" V 9300 1300 50  0000 C CNN
-F 2 "Mounting_Holes:MountingHole_3.2mm_M3_Pad" H 9200 1300 50  0001 C CNN
+F 2 "Mounting_Holes:MountingHole_3.2mm_M3" H 9200 1300 50  0001 C CNN
 F 3 "" H 9200 1300 50  0000 C CNN
 	1    9200 1300
@@
 F 0 "H2" H 9800 1400 50  0000 C CNN
 F 1 "CONN_01X01" V 9900 1300 50  0000 C CNN
-F 2 "Mounting_Holes:MountingHole_3.2mm_M3_Pad" H 9800 1300 50  0001 C CNN
+F 2 "Mounting_Holes:MountingHole_3.2mm_M3" H 9800 1300 50  0001 C CNN
 F 3 "" H 9800 1300 50  0000 C CNN
 	1    9800 1300
@@
 F 0 "C1" H 3200 1600 50  0000 C CNN
 F 1 "10u" V 3250 1350 50  0000 C CNN
-F 2 "Capacitors_SMD:C_0805_HandSoldering" H 3150 1500 50  0001 C CNN
+F 2 "espitall:C_0805_HandSoldering" H 3150 1500 50  0001 C CNN
 F 3 "" H 3150 1500 50  0000 C CNN
 	1    3150 1500
@@
 F 0 "H3" H 9200 2050 50  0000 C CNN
 F 1 "CONN_01X01" V 9300 1950 50  0000 C CNN
-F 2 "Mounting_Holes:MountingHole_3.2mm_M3_Pad" H 9200 1950 50  0001 C CNN
+F 2 "Mounting_Holes:MountingHole_3.2mm_M3" H 9200 1950 50  0001 C CNN
 F 3 "" H 9200 1950 50  0000 C CNN
 	1    9200 1950
@@
 F 0 "S0" H 4850 4200 50  0000 C CNN
 F 1 "CONN_01X03" V 4950 4000 50  0000 C CNN
-F 2 "Connectors_Molex:Molex_KK-6410-03_03x2.54mm_Straight" H 4850 4000 50  0001 C CNN
+F 2 "espitall:Socket_MOLEX-KK-RM2-54mm_Lock_3pin_straight" H 4850 4000 50  0001 C CNN
 F 3 "" H 4850 4000 50  0000 C CNN
 	1    4850 4000
@@
 F 0 "R2" V 4380 3750 50  0000 C CNN
 F 1 "10k" V 4300 3750 50  0000 C CNN
-F 2 "Resistors_SMD:R_0603_HandSoldering" V 4230 3750 50  0001 C CNN
+F 2 "espitall:R_0603_HandSoldering" V 4230 3750 50  0001 C CNN
 F 3 "" H 4300 3750 50  0000 C CNN
 	1    4300 3750
@@
 F 0 "S1" H 6750 4200 50  0000 C CNN
 F 1 "CONN_01X03" V 6850 4000 50  0000 C CNN
-F 2 "Connectors_Molex:Molex_KK-6410-03_03x2.54mm_Straight" H 6750 4000 50  0001 C CNN
+F 2 "espitall:Socket_MOLEX-KK-RM2-54mm_Lock_3pin_straight" H 6750 4000 50  0001 C CNN
 F 3 "" H 6750 4000 50  0000 C CNN
 	1    6750 4000
@@
 F 0 "R3" V 6280 3750 50  0000 C CNN
 F 1 "10k" V 6200 3750 50  0000 C CNN
-F 2 "Resistors_SMD:R_0603_HandSoldering" V 6130 3750 50  0001 C CNN
+F 2 "espitall:R_0603_HandSoldering" V 6130 3750 50  0001 C CNN
 F 3 "" H 6200 3750 50  0000 C CNN
 	1    6200 3750
@@
 F 0 "S2" H 4850 5850 50  0000 C CNN
 F 1 "CONN_01X03" V 4950 5650 50  0000 C CNN
-F 2 "Connectors_Molex:Molex_KK-6410-03_03x2.54mm_Straight" H 4850 5650 50  0001 C CNN
+F 2 "espitall:Socket_MOLEX-KK-RM2-54mm_Lock_3pin_straight" H 4850 5650 50  0001 C CNN
 F 3 "" H 4850 5650 50  0000 C CNN
 	1    4850 5650
@@
 F 0 "R4" V 4380 5400 50  0000 C CNN
 F 1 "10k" V 4300 5400 50  0000 C CNN
-F 2 "Resistors_SMD:R_0603_HandSoldering" V 4230 5400 50  0001 C CNN
+F 2 "espitall:R_0603_HandSoldering" V 4230 5400 50  0001 C CNN
 F 3 "" H 4300 5400 50  0000 C CNN
 	1    4300 5400
@@
 F 0 "S3" H 6750 5850 50  0000 C CNN
 F 1 "CONN_01X03" V 6850 5650 50  0000 C CNN
-F 2 "Connectors_Molex:Molex_KK-6410-03_03x2.54mm_Straight" H 6750 5650 50  0001 C CNN
+F 2 "espitall:Socket_MOLEX-KK-RM2-54mm_Lock_3pin_straight" H 6750 5650 50  0001 C CNN
 F 3 "" H 6750 5650 50  0000 C CNN
 	1    6750 5650
@@
 F 0 "R5" V 6280 5400 50  0000 C CNN
 F 1 "10k" V 6200 5400 50  0000 C CNN
-F 2 "Resistors_SMD:R_0603_HandSoldering" V 6130 5400 50  0001 C CNN
+F 2 "espitall:R_0603_HandSoldering" V 6130 5400 50  0001 C CNN
 F 3 "" H 6200 5400 50  0000 C CNN
 	1    6200 5400
@@
 F 0 "SIN1" H 950 1800 50  0000 C CNN
 F 1 "CONN_01X05" V 1050 1500 50  0000 C CNN
-F 2 "Connectors_Molex:Molex_KK-6410-05_05x2.54mm_Straight" H 950 1500 50  0001 C CNN
+F 2 "espitall:Socket_MOLEX-KK-RM2-54mm_Lock_5pin_straight" H 950 1500 50  0001 C CNN
 F 3 "" H 950 1500 50  0000 C CNN
 	1    950  1500
@@
 F 0 "C2" H 4900 1600 50  0000 C CNN
 F 1 "10u" V 4950 1350 50  0000 C CNN
-F 2 "Capacitors_SMD:C_0805_HandSoldering" H 4850 1500 50  0001 C CNN
+F 2 "espitall:C_0805_HandSoldering" H 4850 1500 50  0001 C CNN
 F 3 "" H 4850 1500 50  0000 C CNN
 	1    4850 1500
@@
 F 0 "C3" H 5200 1600 50  0000 C CNN
 F 1 "100n" V 5250 1350 50  0000 C CNN
-F 2 "Capacitors_SMD:C_0603_HandSoldering" H 5150 1500 50  0001 C CNN
+F 2 "espitall:C_0603_HandSoldering" H 5150 1500 50  0001 C CNN
 F 3 "" H 5150 1500 50  0000 C CNN
 	1    5150 1500
@@
 F 0 "PIN1" H 2750 1400 50  0000 C CNN
 F 1 "CONN_01X02" V 2850 1250 50  0000 C CNN
-F 2 "Connectors_Molex:Molex_KK-6410-02_02x2.54mm_Straight" H 2750 1250 50  0001 C CNN
+F 2 "espitall:Socket_MOLEX-KK-RM2-54mm_Lock_2pin_straight" H 2750 1250 50  0001 C CNN
 F 3 "" H 2750 1250 50  0000 C CNN
 	1    2750 1250
@@
 F 0 "POUT1" H 5650 1400 50  0000 C CNN
 F 1 "CONN_01X02" V 5750 1250 50  0000 C CNN
-F 2 "Connectors_Molex:Molex_KK-6410-02_02x2.54mm_Straight" H 5650 1250 50  0001 C CNN
+F 2 "espitall:Socket_MOLEX-KK-RM2-54mm_Lock_2pin_straight" H 5650 1250 50  0001 C CNN
 F 3 "" H 5650 1250 50  0000 C CNN
 	1    5650 1250
