File: motor/motor.kicad_pcb (KiCad board)
At the start: 2 copper layers, 45 x 50 mm, 23 parts, among them U1 LMD18200T

Commit message: 3d view of motor board
Parts:
- C1: footprint Capacitors_SMD:CP_Elec_10x10 -> espitall:CP_Elec_10x10
- C2, C3, C4: footprint Capacitors_SMD:C_0805 -> espitall:C_0805
- D1, D2, D3: footprint LEDs:LED_0805 -> espitall:LED_0805
- ERROR1: footprint Sockets_MOLEX_KK-System:Socket_MOLEX-KK-RM2-54mm_Lock_2pin_straight -> espitall:Socket_MOLEX-KK-RM2-54mm_Lock_2pin_straight
- LOGIC1: footprint Sockets_MOLEX_KK-System:Socket_MOLEX-KK-RM2-54mm_Lock_5pin_straight -> espitall:Socket_MOLEX-KK-RM2-54mm_Lock_5pin_straight
- MOTOR1, POWER1: footprint Connectors_Terminal_Blocks:TerminalBlock_WAGO-236_2Stift_RM5mm_2pol -> espitall:TerminalBlock_WAGO-236_2Stift_RM5mm_2pol
- R1, R2, R3, R4, R5, R6, R7: footprint Resistors_SMD:R_0603 -> espitall:R_0603
- moved C4 3.91 mm to (81.4, 64.3)
- moved C3 3.89 mm to (63.5, 64.3)
- moved ERROR1 3.46 mm to (89.1, 70.7)
- moved R1 3.25 mm to (88.4, 66.8)
- turned MOTOR1 to 90 degrees
- turned POWER1 to 270 degrees
Connections:
- MOTOR1 pad 1: Net-(C3-Pad1) -> Net-(C4-Pad1)
- MOTOR1 pad 2: Net-(C4-Pad1) -> Net-(C3-Pad1)
- POWER1 pad 1: +BATT -> GND
- POWER1 pad 2: GND -> +BATT
Routing:
- net +5V: track 49.9 -> 67.0 mm
- net Net-(C3-Pad1): track 45.5 -> 54.1 mm
- net GND: track 241.1 -> 232.6 mm
- net /dir: track 14.0 -> 16.8 mm
- net /err: track 42.3 -> 40.0 mm
- net /brake: track 19.8 -> 17.5 mm
- net Net-(R2-Pad2): track 1.77 -> 3.33 mm
- net Net-(C4-Pad2): track 3.50 -> 2.41 mm
- net Net-(C3-Pad2): track 3.43 -> 2.45 mm
- net +BATT: track 73.4 -> 74.3 mm
- net Net-(C4-Pad1): track 32.9 -> 33.7 mm
- net /PWM: track 19.0 -> 19.7 mm
