File: motor/motor.sch (KiCad schematic (older format))
At the start: 12 parts, among them U1 LMD18200T

Commit message: motor (HV) board layout
Parts:
- removed HEATSINK1: CONN_2, Sockets_MOLEX_KK-System:Socket_MOLEX-KK-RM2-54mm_Lock_2pin_straight, symbol CONN_2
- added D1, D2: LED_Green, LEDs:LED_0805, symbol LED
- added D3: LED_red, LEDs:LED_0805, symbol LED
- added H1, H2, H3: CONN_01X01, Mounting_Holes:MountingHole_3.2mm_M3, symbol CONN_01X01
- added HS1: CONN_01X01, espitall:SK409-25_4STC, symbol CONN_01X01
- added R3, R4: 10k, Resistors_SMD:R_0603, symbol R-RESCUE-motor
- added R5: 330, Resistors_SMD:R_0603, symbol R-RESCUE-motor
- added R6, R7: 2k2, Resistors_SMD:R_0603, symbol R-RESCUE-motor
- C1: value 1m -> 220u; footprint Capacitors_ThroughHole:C_Radial_D10_L20_P5 -> Capacitors_SMD:CP_Elec_10x10; symbol C -> C-RESCUE-motor
- C2: value 1u -> 470n; symbol C -> C-RESCUE-motor
- C3, C4: symbol C -> C-RESCUE-motor
- MOTOR1, POWER1: footprint Terminal_Blocks:TerminalBlock_WAGO-804_RM5mm_2pol -> Connectors_Terminal_Blocks:TerminalBlock_WAGO-236_2Stift_RM5mm_2pol
- R1: symbol R -> R-RESCUE-motor
- R2: value 2k7 -> 2k2; symbol R -> R-RESCUE-motor
Connections:
- net +5V: now also D1.2 (A)
- net +BATT: now also D2.2 (A), D3.2 (A)
- net GND: now also H1.1 (P1), H2.1 (P1), H3.1 (P1), HS1.1 (P1), R3.1, R4.1, R5.1, R6.1
- net dir: now reaches LOGIC1.3, U1.3 (DIR)
- net brake: now reaches LOGIC1.2, U1.4 (BRAKE)
- net brake: now also R4.2
- net PWM: now reaches LOGIC1.4, U1.5 (PWM)
- net PWM: now also R3.2
- net err: now reaches ERROR1.2 (PM), U1.9 (THERMAL)
- net err: now also R7.1
- new net: D1.1 (K), R5.2
- new net: D2.1 (K), R6.2
- new net: D3.1 (K), R7.2

Commit message: 3d view of motor board
Parts:
- C1: footprint Capacitors_SMD:CP_Elec_10x10 -> espitall:CP_Elec_10x10; symbol C-RESCUE-motor -> motor-rescue:C-RESCUE-motor
- C2, C3, C4: footprint Capacitors_SMD:C_0805 -> espitall:C_0805; symbol C-RESCUE-motor -> motor-rescue:C-RESCUE-motor
- D1, D2, D3: footprint LEDs:LED_0805 -> espitall:LED_0805; symbol LED -> motor-rescue:LED-RESCUE-motor
- ERROR1: footprint Sockets_MOLEX_KK-System:Socket_MOLEX-KK-RM2-54mm_Lock_2pin_straight -> espitall:Socket_MOLEX-KK-RM2-54mm_Lock_2pin_straight; symbol CONN_2 -> motor-rescue:CONN_2-RESCUE-motor
- H1, H2, H3, HS1: symbol CONN_01X01 -> motor-rescue:CONN_01X01-RESCUE-motor
- LOGIC1: footprint Sockets_MOLEX_KK-System:Socket_MOLEX-KK-RM2-54mm_Lock_5pin_straight -> espitall:Socket_MOLEX-KK-RM2-54mm_Lock_5pin_straight; symbol CONN_5 -> motor-rescue:CONN_5-RESCUE-motor
- MOTOR1, POWER1: footprint Connectors_Terminal_Blocks:TerminalBlock_WAGO-236_2Stift_RM5mm_2pol -> espitall:TerminalBlock_WAGO-236_2Stift_RM5mm_2pol; symbol CONN_2 -> motor-rescue:CONN_2-RESCUE-motor
- R1, R2, R3, R4, R5, R6, R7: footprint Resistors_SMD:R_0603 -> espitall:R_0603; symbol R-RESCUE-motor -> motor-rescue:R-RESCUE-motor
- U1: symbol LMD18200T -> motor-rescue:LMD18200T-RESCUE-motor
Connections:
- net +BATT: now also POWER1.2 (PM); no longer POWER1.1 (P1)
- net GND: now also POWER1.1 (P1); no longer POWER1.2 (PM)
- net at C4.1, U1.10 (OUPUT_2): now also MOTOR1.1 (P1); no longer MOTOR1.2 (PM)
- net at C3.1, U1.2 (OUTPUT_1): now also MOTOR1.2 (PM); no longer MOTOR1.1 (P1)
