File: alim/alim/alim.sch (KiCad schematic (older format))
At the start: 15 parts

Commit message: schematic modified
Parts:
- added C2, C6, C? (x2): C, mods:CAPCP2012X100N, symbol device:C
- added C4: C, espitall:C_0805_HandSoldering, symbol device:C
- added C?: Chimique (OSEF de la valeur et la taille, juste u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, symbol device:C
- added L2: INDUCTOR, 15µH Wurth 74457115 (ou equivalent), symbol INDUCTOR:INDUCTOR
- added P5: CONN_2_PWR, espitall:TerminalBlock_WAGO-236_2Stift_RM5mm_2pol, symbol espitall:CONN_2_PWR
- added Q3, Q?: STTH30R08 (PPACK56), TRANS_SIR422DP-T1-GE3, symbol SIR422DP-T1-GE3:SIR422DP-T1-GE3
- added R4, R5: R, espitall:R_0603_HandSoldering, symbol device:R
- added U2: TPS5430DDA, HSOIC8, symbol dc-dc:TPS5430DDA
- L1: renamed from L?; value INDUCTOR -> 15µH Wurth 74457115 (ou equivalent); footprint mods:INDC3218X180N -> (none)
- Q1: renamed from Q?; value SIR422DP-T1-GE3 -> BSC046N10NS3 (PPACK56)
- Q2: renamed from Q?; value SIR422DP-T1-GE3 -> STTH30R08 (PPACK56)
- gave numbers to parts that had none: 12
Connections:
- wire segments 88 -> 172

Commit message: Prepare alim board for layout
Parts:
- removed L1: 15µH Wurth 74457115 (ou equivalent), symbol INDUCTOR:INDUCTOR
- removed Q1: BSC046N10NS3 (PPACK56), TRANS_SIR422DP-T1-GE3, symbol SIR422DP-T1-GE3:SIR422DP-T1-GE3
- removed Q2, Q3, Q?: STTH30R08 (PPACK56), TRANS_SIR422DP-T1-GE3, symbol SIR422DP-T1-GE3:SIR422DP-T1-GE3
- added L1: INDUCTOR, Inductors_SMD:L_Wuerth_WE-PD4-Typ-X, symbol alim-rescue:INDUCTOR-INDUCTOR
- added Q1, Q2, Q3, Q4: BSC046N10NS3, espitall:TDSON-8-1_HandSoldering, symbol espitall:BSC046N10NS3
- C1, C2, C3, C4, C5, C6: symbol device:C -> alim-rescue:C-device
- C7: renamed from C?; footprint (none) -> espitall:c_elec_6.3x7.7; symbol device:C -> alim-rescue:C-device
- C8, C9: renamed from C?; symbol device:C -> alim-rescue:C-device
- D1: symbol DIODEZENER:DIODEZENER -> alim-rescue:DIODEZENER-DIODEZENER
- L2: footprint 15µH Wurth 74457115 (ou equivalent) -> Inductors_SMD:L_Wuerth_WE-PD4-Typ-X; symbol INDUCTOR:INDUCTOR -> alim-rescue:INDUCTOR-INDUCTOR; Field4 (none) -> 15µH Wurth 74457115 (ou equivalent)
- P5: footprint espitall:TerminalBlock_WAGO-236_2Stift_RM5mm_2pol -> espitall:Socket_MOLEX-KK-RM2-54mm_Lock_2pin_straight
- R1, R2, R3, R4, R5: symbol device:R -> alim-rescue:R-device
- U1, U2: footprint HSOIC8 -> espitall:SOIC-8-PowerPAD; symbol dc-dc:TPS5430DDA -> alim-rescue:TPS5430DDA-dc-dc
Connections:
- wire segments 172 -> 150

Commit message: Add missing C1210 footprint
Parts:
- C1, C2, C5, C6, C8, C9: footprint mods:CAPCP2012X100N -> espitall:C_1210_HandSoldering
Connections:
- wire segments 150 -> 145
Changed lines of the file:
@@
 F 0 "C3" V 6511 2100 40  0000 C CNN
 F 1 "C" V 6587 2100 40  0000 C CNN
-F 2 "espitall:C_0805_HandSoldering" V 6655 2100 30  0000 C CNN
+F 2 "espitall:C_0805_HandSoldering" V 6655 2100 30  0001 C CNN
 F 3 "" H 6800 2100 60  0000 C CNN
 	1    6800 2100
@@
 Wire Wire Line
 	8250 2250 8250 2300
-Wire Wire Line
-	6950 2850 6950 2800
-Wire Wire Line
-	6950 2800 6950 2250
 Connection ~ 6950 2250
 Wire Wire Line
@@
 F 0 "C5" H 8535 2882 40  0000 R CNN
 F 1 "C" H 8535 2958 40  0000 R CNN
-F 2 "mods:CAPCP2012X100N" H 8535 3026 30  0000 R CNN
+F 2 "espitall:C_1210_HandSoldering" H 8535 3026 30  0001 R CNN
 F 3 "" H 8650 2950 60  0000 C CNN
 	1    8650 2950
@@
 F 0 "C1" H 4935 2832 40  0000 R CNN
 F 1 "C" H 4935 2908 40  0000 R CNN
-F 2 "mods:CAPCP2012X100N" H 4935 2976 30  0000 R CNN
+F 2 "espitall:C_1210_HandSoldering" H 4935 2976 30  0001 R CNN
 F 3 "" H 5050 2900 60  0000 C CNN
 	1    5050 2900
@@
 F 0 "C4" V 6511 4450 40  0000 C CNN
 F 1 "C" V 6587 4450 40  0000 C CNN
-F 2 "espitall:C_0805_HandSoldering" V 6655 4450 30  0000 C CNN
+F 2 "espitall:C_0805_HandSoldering" V 6655 4450 30  0001 C CNN
 F 3 "" H 6800 4450 60  0000 C CNN
 	1    6800 4450
@@
 Wire Wire Line
 	8250 4600 8250 4650
-Wire Wire Line
-	6950 5200 6950 5150
-Wire Wire Line
-	6950 5150 6950 4600
 Connection ~ 6950 4600
 Wire Wire Line
@@
 F 0 "C6" H 8535 5232 40  0000 R CNN
 F 1 "C" H 8535 5308 40  0000 R CNN
-F 2 "mods:CAPCP2012X100N" H 8535 5376 30  0000 R CNN
+F 2 "espitall:C_1210_HandSoldering" H 8535 5376 30  0001 R CNN
 F 3 "" H 8650 5300 60  0000 C CNN
 	1    8650 5300
@@
 F 0 "C2" H 4935 5182 40  0000 R CNN
 F 1 "C" H 4935 5258 40  0000 R CNN
-F 2 "mods:CAPCP2012X100N" H 4935 5326 30  0000 R CNN
+F 2 "espitall:C_1210_HandSoldering" H 4935 5326 30  0001 R CNN
 F 3 "" H 5050 5250 60  0000 C CNN
 	1    5050 5250
@@
 	9450 1200 9450 850
 Wire Wire Line
-	9450 850  8700 850
-Wire Wire Line
-	8500 850  8600 850
-Wire Wire Line
 	8600 1000 8600 850
 Connection ~ 8600 850
-Wire Wire Line
-	8600 850  8700 850
-Wire Wire Line
-	8500 850  8400 850
 Wire Wire Line
 	4300 1200 4300 850
@@
 Connection ~ 5800 850
 Wire Wire Line
-	5800 850  8400 850
-Wire Wire Line
 	5800 1450 5800 1650
 Connection ~ 5800 1650
@@
 F 0 "C8" H 8985 2882 40  0000 R CNN
 F 1 "C" H 8985 2958 40  0000 R CNN
-F 2 "mods:CAPCP2012X100N" H 8985 3026 30  0000 R CNN
+F 2 "espitall:C_1210_HandSoldering" H 8985 3026 30  0001 R CNN
 F 3 "" H 9100 2950 60  0000 C CNN
 	1    9100 2950
@@
 F 0 "C9" H 8935 5232 40  0000 R CNN
 F 1 "C" H 8935 5308 40  0000 R CNN
-F 2 "mods:CAPCP2012X100N" H 8935 5376 30  0000 R CNN
+F 2 "espitall:C_1210_HandSoldering" H 8935 5376 30  0001 R CNN
 F 3 "" H 9050 5300 60  0000 C CNN
 	1    9050 5300
@@
 	1    0    0    -1
 $EndComp
+Wire Wire Line
+	6950 2250 6950 2850
+Wire Wire Line
+	6950 4600 6950 5200
+Wire Wire Line
+	8600 850  9450 850
+Wire Wire Line
+	5800 850  8600 850
 $EndSCHEMATC

Commit message: prerouting placement
Parts:
- added H1, H2, H3, H4: CONN_1, symbol conn:CONN_1
- L1, L2: footprint Inductors_SMD:L_Wuerth_WE-PD4-Typ-X -> espitall:L_Wuerth_WE-PD4-Typ-X
Connections:
- wire segments 145 -> 153
Changed lines of the file:
@@
 F 0 "L2" H 7450 4800 40  0000 C CNN
 F 1 "INDUCTOR" H 7450 4700 40  0000 C CNN
-F 2 "Inductors_SMD:L_Wuerth_WE-PD4-Typ-X" H 7450 4694 60  0001 C CNN
+F 2 "espitall:L_Wuerth_WE-PD4-Typ-X" H 7450 4694 60  0001 C CNN
 F 3 "" H 7450 4600 60  0000 C CNN
 F 4 "15µH Wurth 74457115 (ou equivalent)" H 7450 4600 50  0001 C CNN "Field4"
@@
 F 0 "L1" H 7450 2450 40  0000 C CNN
 F 1 "INDUCTOR" H 7450 2350 40  0000 C CNN
-F 2 "Inductors_SMD:L_Wuerth_WE-PD4-Typ-X" H 7450 2344 60  0001 C CNN
+F 2 "espitall:L_Wuerth_WE-PD4-Typ-X" H 7450 2344 60  0001 C CNN
 F 3 "" H 7450 2250 60  0000 C CNN
 F 4 "15µH Wurth 74457115 (ou equivalent)" H 7450 2250 50  0001 C CNN "Field4"
@@
 Wire Wire Line
 	5800 850  8600 850
+$Comp
+L conn:CONN_1 H1
+U 1 1 5A783F3B
+P 1900 5700
+F 0 "H1" H 1959 5700 40  0000 L CNN
+F 1 "CONN_1" H 1900 5755 30  0001 C CNN
+F 2 "" H 1900 5700 50  0001 C CNN
+F 3 "" H 1900 5700 50  0001 C CNN
+	1    1900 5700
+	1    0    0    -1
+$EndComp
+$Comp
+L conn:CONN_1 H2
+U 1 1 5A784078
+P 1900 5850
+F 0 "H2" H 1959 5850 40  0000 L CNN
+F 1 "CONN_1" H 1900 5905 30  0001 C CNN
+F 2 "" H 1900 5850 50  0001 C CNN
+F 3 "" H 1900 5850 50  0001 C CNN
+	1    1900 5850
+	1    0    0    -1
+$EndComp
+$Comp
+L conn:CONN_1 H3
+U 1 1 5A7840D2
+P 1900 6000
+F 0 "H3" H 1959 6000 40  0000 L CNN
+F 1 "CONN_1" H 1900 6055 30  0001 C CNN
+F 2 "" H 1900 6000 50  0001 C CNN
+F 3 "" H 1900 6000 50  0001 C CNN
+	1    1900 6000
+	1    0    0    -1
+$EndComp
+$Comp
+L conn:CONN_1 H4
+U 1 1 5A784122
+P 1900 6200
+F 0 "H4" H 1959 6200 40  0000 L CNN
+F 1 "CONN_1" H 1900 6255 30  0001 C CNN
+F 2 "" H 1900 6200 50  0001 C CNN
+F 3 "" H 1900 6200 50  0001 C CNN
+	1    1900 6200
+	1    0    0    -1
+$EndComp
+$Comp
+L alim-rescue:GND-power #PWR02
+U 1 1 5A784256
+P 1500 6450
+F 0 "#PWR02" H 1500 6450 30  0001 C CNN
+F 1 "GND" H 1500 6380 30  0001 C CNN
+F 2 "" H 1500 6450 50  0001 C CNN
+F 3 "" H 1500 6450 50  0001 C CNN
+	1    1500 6450
+	1    0    0    -1
+$EndComp
+Wire Wire Line
+	1750 5700 1500 5700
+Wire Wire Line
+	1500 5700 1500 5850
+Wire Wire Line
+	1750 5850 1500 5850
+Connection ~ 1500 5850
+Wire Wire Line
+	1500 5850 1500 6000
+Wire Wire Line
+	1750 6000 1500 6000
+Connection ~ 1500 6000
+Wire Wire Line
+	1500 6000 1500 6200
+Wire Wire Line
+	1750 6200 1500 6200
+Connection ~ 1500 6200
+Wire Wire Line
+	1500 6200 1500 6450
 $EndSCHEMATC
