File: score/score.kicad_pcb (KiCad board)
At the start: 2 copper layers, 62 x 46 mm, 47 parts, among them J1 Conn_01x02, P8 CONN_01X07, P9 CONN_01X07, U1 74HC595T16-13, U2 HDSP-C8A1, U3 HDSP-C8A1, U4 HDSP-C8A1, U5 74HC595T16-13, U6 74HC595T16-13, U7 TSR1-2433

Commit message: quick modification on pads. Do not use this revision
Parts:
- removed U5, U6: 74HC595T16-13, espitall:TSSOP-16_4.4x5mm_Pitch0.65mm
- added U1: 74HC595T16-13, espitall:TSSOP-16_4.4x5mm_Pitch0.65mm, B.Cu at (101.7, 63.8)
- added U1: 74HC595T16-13, espitall:TSSOP-16_4.4x5mm_Pitch0.65mm, B.Cu at (81.8, 63.0)
Routing:
- net Net-(U5-Pad9): track 33.1 -> 0.00 mm, vias 2 -> 0
- net (no net): track 0.00 -> 33.1 mm, vias 0 -> 2
