File: com/com.sch (KiCad schematic (older format))
At the start: 3 parts, among them U1 SPSGRF-868

Commit message: full schematic
Parts:
- added U2: TSR1-2433, symbol espitall:TSR1-2433
- C1: footprint (none) -> espitall:C_0805; symbol device:C -> com-rescue:C-device
- C2: footprint (none) -> espitall:C_0603; symbol device:C -> com-rescue:C-device
Connections:
- wire segments 18 -> 35
Changed lines of the file:
@@
 	9950 4750 9950 4550
 $Comp
-L device:C C1
+L com-rescue:C-device C1
 U 1 1 5AFB1A84
 P 10250 2600
 F 0 "C1" H 10365 2646 50  0000 L CNN
 F 1 "10u" H 10365 2555 50  0000 L CNN
-F 2 "" H 10288 2450 50  0001 C CNN
+F 2 "espitall:C_0805" H 10288 2450 50  0001 C CNN
 F 3 "" H 10250 2600 50  0001 C CNN
 	1    10250 2600
@@
 	10250 2850 10250 2750
 $Comp
-L device:C C2
+L com-rescue:C-device C2
 U 1 1 5AFB1C41
 P 10650 2600
 F 0 "C2" H 10765 2646 50  0000 L CNN
 F 1 "100n" H 10765 2555 50  0000 L CNN
-F 2 "" H 10688 2450 50  0001 C CNN
+F 2 "espitall:C_0603" H 10688 2450 50  0001 C CNN
 F 3 "" H 10650 2600 50  0001 C CNN
 	1    10650 2600
@@
 F0 "Computer" 50
 F1 "computer.sch" 50
+F2 "rx_3v3" O R 4550 2200 50
+F3 "tx_3v3" I R 4550 2100 50
+F4 "5v" O R 4550 1900 50
 $EndSheet
 $Sheet
@@
 F0 "Robot" 50
 F1 "robot.sch" 50
+F2 "rx_3v3" O R 4550 3900 50
+F3 "tx_3v3" I R 4550 3800 50
+F4 "5v" O R 4550 3650 50
 $EndSheet
+Wire Wire Line
+	4550 3800 5600 3800
+Wire Wire Line
+	5600 3800 5600 3300
+Wire Wire Line
+	5600 3300 6450 3300
+Wire Wire Line
+	6450 3400 5700 3400
+Wire Wire Line
+	5700 3400 5700 3900
+Wire Wire Line
+	5700 3900 4550 3900
+Wire Wire Line
+	4550 2100 5600 2100
+Wire Wire Line
+	5600 2100 5600 3300
+Connection ~ 5600 3300
+Wire Wire Line
+	4550 2200 5700 2200
+Wire Wire Line
+	5700 2200 5700 3400
+Connection ~ 5700 3400
+$Comp
+L espitall:TSR1-2433 U2
+U 1 1 5AFEE66F
+P 6950 1950
+F 0 "U2" H 6950 2287 60  0000 C CNN
+F 1 "TSR1-2433" H 6950 2181 60  0000 C CNN
+F 2 "" H 6950 1950 60  0000 C CNN
+F 3 "" H 6950 1950 60  0000 C CNN
+	1    6950 1950
+	1    0    0    -1
+$EndComp
+$Comp
+L power:GND #PWR05
+U 1 1 5AFEE676
+P 6950 2500
+F 0 "#PWR05" H 6950 2250 50  0001 C CNN
+F 1 "GND" H 6955 2327 50  0000 C CNN
+F 2 "" H 6950 2500 50  0001 C CNN
+F 3 "" H 6950 2500 50  0001 C CNN
+	1    6950 2500
+	1    0    0    -1
+$EndComp
+Wire Wire Line
+	6950 2500 6950 2200
+$Comp
+L power:+3V3 #PWR06
+U 1 1 5AFEE67E
+P 7450 1700
+F 0 "#PWR06" H 7450 1550 50  0001 C CNN
+F 1 "+3V3" H 7465 1873 50  0000 C CNN
+F 2 "" H 7450 1700 50  0001 C CNN
+F 3 "" H 7450 1700 50  0001 C CNN
+	1    7450 1700
+	1    0    0    -1
+$EndComp
+Wire Wire Line
+	7450 1700 7450 1900
+Wire Wire Line
+	7450 1900 7350 1900
+Wire Wire Line
+	4550 1900 5800 1900
+Wire Wire Line
+	4550 3650 5800 3650
+Wire Wire Line
+	5800 3650 5800 1900
+Connection ~ 5800 1900
+Wire Wire Line
+	5800 1900 6550 1900
 $EndSCHEMATC

Commit message: footprint assignation
Parts:
- added J6, J7, J8, J9: Conn_01x01, Mounting_Holes:MountingHole_3.2mm_M3, symbol Connector_Generic:Conn_01x01
- U2: footprint (none) -> espitall:TSR-1
Changed lines of the file:
@@
 F 0 "U2" H 6950 2287 60  0000 C CNN
 F 1 "TSR1-2433" H 6950 2181 60  0000 C CNN
-F 2 "" H 6950 1950 60  0000 C CNN
+F 2 "espitall:TSR-1" H 6950 1950 60  0001 C CNN
 F 3 "" H 6950 1950 60  0000 C CNN
 	1    6950 1950
@@
 Wire Wire Line
 	5800 1900 6550 1900
+$Comp
+L Connector_Generic:Conn_01x01 J6
+U 1 1 5B046ECC
+P 900 7050
+F 0 "J6" H 820 6825 50  0000 C CNN
+F 1 "Conn_01x01" H 820 6916 50  0000 C CNN
+F 2 "Mounting_Holes:MountingHole_3.2mm_M3" H 900 7050 50  0001 C CNN
+F 3 "~" H 900 7050 50  0001 C CNN
+	1    900  7050
+	-1   0    0    1
+$EndComp
+$Comp
+L Connector_Generic:Conn_01x01 J8
+U 1 1 5B046F52
+P 900 7400
+F 0 "J8" H 820 7175 50  0000 C CNN
+F 1 "Conn_01x01" H 820 7266 50  0000 C CNN
+F 2 "Mounting_Holes:MountingHole_3.2mm_M3" H 900 7400 50  0001 C CNN
+F 3 "~" H 900 7400 50  0001 C CNN
+	1    900  7400
+	-1   0    0    1
+$EndComp
+$Comp
+L Connector_Generic:Conn_01x01 J7
+U 1 1 5B046F92
+P 1500 7050
+F 0 "J7" H 1420 6825 50  0000 C CNN
+F 1 "Conn_01x01" H 1420 6916 50  0000 C CNN
+F 2 "Mounting_Holes:MountingHole_3.2mm_M3" H 1500 7050 50  0001 C CNN
+F 3 "~" H 1500 7050 50  0001 C CNN
+	1    1500 7050
+	-1   0    0    1
+$EndComp
+$Comp
+L Connector_Generic:Conn_01x01 J9
+U 1 1 5B046FEE
+P 1500 7400
+F 0 "J9" H 1420 7175 50  0000 C CNN
+F 1 "Conn_01x01" H 1420 7266 50  0000 C CNN
+F 2 "Mounting_Holes:MountingHole_3.2mm_M3" H 1500 7400 50  0001 C CNN
+F 3 "~" H 1500 7400 50  0001 C CNN
+	1    1500 7400
+	-1   0    0    1
+$EndComp
 $EndSCHEMATC

Commit message: add CAN output on com board
Connections:
- wire segments 35 -> 43
Changed lines of the file:
@@
 $Descr A4 11693 8268
 encoding utf-8
-Sheet 1 4
+Sheet 1 5
 Title ""
 Date ""
@@
 	10650 2350 10250 2350
 Connection ~ 10250 2350
-$Sheet
-S 6450 3050 1800 1400
-U 5AFB1EE6
-F0 "uc" 50
-F1 "uc.sch" 50
-F2 "rf_spi_sck_3v3" O R 8250 4050 50
-F3 "rf_spi_miso_3v3" I R 8250 3950 50
-F4 "rf_spi_mosi_3v3" O R 8250 3850 50
-F5 "tx_3v3" O L 6450 3300 50
-F6 "rx_3v3" I L 6450 3400 50
-F7 "rf_spi_cs_3v3" O R 8250 3750 50
-F8 "rf_gpio3_3v3" O R 8250 3250 50
-F9 "rf_gpio2_3v3" O R 8250 3350 50
-F10 "rf_gpio1_3v3" O R 8250 3450 50
-F11 "rf_gpio0_3v3" O R 8250 3550 50
-F12 "rf_sdn_3v3" O R 8250 4250 50
-$EndSheet
 Wire Wire Line
 	9250 3950 8250 3950
@@
 F3 "tx_3v3" I R 4550 3800 50
 F4 "5v" O R 4550 3650 50
+F5 "can_h" B L 2700 4300 50
+F6 "can_l" B L 2700 4400 50
 $EndSheet
 Wire Wire Line
@@
 	-1   0    0    1
 $EndComp
+$Sheet
+S 6450 3050 1800 3000
+U 5AFB1EE6
+F0 "uc" 50
+F1 "uc.sch" 50
+F2 "rf_spi_sck_3v3" O R 8250 4050 50
+F3 "rf_spi_miso_3v3" I R 8250 3950 50
+F4 "rf_spi_mosi_3v3" O R 8250 3850 50
+F5 "tx_3v3" O L 6450 3300 50
+F6 "rx_3v3" I L 6450 3400 50
+F7 "rf_spi_cs_3v3" O R 8250 3750 50
+F8 "rf_gpio3_3v3" O R 8250 3250 50
+F9 "rf_gpio2_3v3" O R 8250 3350 50
+F10 "rf_gpio1_3v3" O R 8250 3450 50
+F11 "rf_gpio0_3v3" O R 8250 3550 50
+F12 "rf_sdn_3v3" O R 8250 4250 50
+F13 "can_tx_3v3" O L 6450 5300 50
+F14 "can_rx_3v3" I L 6450 5400 50
+$EndSheet
+$Sheet
+S 2700 5100 1850 950
+U 5B0C6E1B
+F0 "CAN" 50
+F1 "can.sch" 50
+F2 "can_tx_3v3" I R 4550 5300 50
+F3 "can_rx_3v3" O R 4550 5400 50
+F4 "can_h" B L 2700 5300 50
+F5 "can_l" B L 2700 5400 50
+$EndSheet
+Wire Wire Line
+	6450 5400 4550 5400
+Wire Wire Line
+	4550 5300 6450 5300
+Wire Wire Line
+	2700 4300 2250 4300
+Wire Wire Line
+	2250 4300 2250 5300
+Wire Wire Line
+	2250 5300 2700 5300
+Wire Wire Line
+	2700 5400 2350 5400
+Wire Wire Line
+	2350 5400 2350 4400
+Wire Wire Line
+	2350 4400 2700 4400
 $EndSCHEMATC
