File: com/computer.sch (KiCad schematic (older format))
At the start: 0 parts

Commit message: full schematic
Parts:
- added C3: 10n, espitall:C_0603, symbol Device:C
- added C4: 4u7, espitall:C_0805, symbol Device:C
- added C5, C6: 100n, espitall:C_0603, symbol Device:C
- added J4: USB_B_Micro, symbol Connector_Specialized:USB_B_Micro
- added L1: Ferrite_Bead, symbol Device:Ferrite_Bead
- added R21: 10k, espitall:C_0603, symbol Device:R
- added U3: FT232RL, Package_SO:SSOP-28_5.3x10.2mm_P0.65mm, symbol Interface_USB:FT232RL
Connections:
- net labels added: +3V3, 5v, GND, rx_3v3, tx_3v3
- wire segments 0 -> 46

Commit message: footprint assignation
Parts:
- J4: footprint (none) -> Connectors:USB_Micro-B_10103594-0001LF
- L1: footprint (none) -> espitall:C_0805
Changed lines of the file:
@@
 F 0 "J4" H 2155 3867 50  0000 C CNN
 F 1 "USB_B_Micro" H 2155 3776 50  0000 C CNN
-F 2 "" H 2250 3350 50  0001 C CNN
+F 2 "Connectors:USB_Micro-B_10103594-0001LF" H 2250 3350 50  0001 C CNN
 F 3 "~" H 2250 3350 50  0001 C CNN
 	1    2100 3400
@@
 F 0 "L1" V 3726 1950 50  0000 C CNN
 F 1 "Ferrite_Bead" V 3817 1950 50  0000 C CNN
-F 2 "" V 3930 1950 50  0001 C CNN
+F 2 "espitall:C_0805" V 3930 1950 50  0001 C CNN
 F 3 "~" H 4000 1950 50  0001 C CNN
 	1    4000 1950

Commit message: add CAN output on com board
Parts:
- U3: footprint Package_SO:SSOP-28_5.3x10.2mm_P0.65mm -> Housings_SSOP:SSOP-28_5.3x10.2mm_Pitch0.65mm
Changed lines of the file:
@@
 $Descr A4 11693 8268
 encoding utf-8
-Sheet 3 4
+Sheet 3 5
 Title ""
 Date ""
@@
 F 0 "U3" H 7450 4500 50  0000 C CNN
 F 1 "FT232RL" H 7550 2700 50  0000 C CNN
-F 2 "Package_SO:SSOP-28_5.3x10.2mm_P0.65mm" H 7000 3600 50  0001 C CNN
+F 2 "Housings_SSOP:SSOP-28_5.3x10.2mm_Pitch0.65mm" H 7000 3600 50  0001 C CNN
 F 3 "http://www.ftdichip.com/Products/ICs/FT232RL.htm" H 7000 3600 50  0001 C CNN
 	1    7000 3600

Commit message: com board: silkscreen and 3d
Parts:
- J4: footprint Connectors:USB_Micro-B_10103594-0001LF -> espitall:USB_Micro-B_10103594-0001LF
Changed lines of the file:
@@
 $Descr A4 11693 8268
 encoding utf-8
-Sheet 3 5
-Title ""
-Date ""
-Rev ""
-Comp ""
+Sheet 2 5
+Title "Com"
+Date "2018-05-27"
+Rev "2019"
+Comp "Cocobot"
 Comment1 ""
 Comment2 ""
@@
 F 0 "J4" H 2155 3867 50  0000 C CNN
 F 1 "USB_B_Micro" H 2155 3776 50  0000 C CNN
-F 2 "Connectors:USB_Micro-B_10103594-0001LF" H 2250 3350 50  0001 C CNN
+F 2 "espitall:USB_Micro-B_10103594-0001LF" H 2250 3350 50  0001 C CNN
 F 3 "~" H 2250 3350 50  0001 C CNN
 	1    2100 3400
