File: com/can.sch (KiCad schematic (older format))
At the start: 3 parts, among them U5 MAX3051ESA

Commit message: add electrical protection on CAN bus
Parts:
- added C15, C16, C17, C18: C, espitall:C_0603, symbol Device:C
- added D2: NUP2105LT1G, espitall:SOT-23, symbol espitall:NUP2105LT1G
- added FL1: DR331-113BE, espitall:DR331, symbol espitall:DR331-113BE
Connections:
- wire segments 15 -> 46
