File: com/robot.sch (KiCad schematic (older format))
At the start: 3 parts

Commit message: full schematic
Parts:
- removed U?: TSR1-2433, symbol espitall:TSR1-2433
- added C10, C11, C12, C7, C9: 100n, espitall:C_0603, symbol Device:C
- added R22, R23: 0, espitall:R_0603, symbol Device:R
- added U4: MAX3232, symbol Interface_UART:MAX3232
- C8: renamed from C?; footprint (none) -> espitall:C_0805; symbol device:C -> com-rescue:C-device
- J5: renamed from J?; symbol conn:Conn_01x04 -> com-rescue:Conn_01x04-conn
Connections:
- net labels added: 5v, rx_3v3, tx_3v3
- net labels removed: +5V
- wire segments 12 -> 54

Commit message: footprint assignation
Parts:
- J5: footprint (none) -> Connectors_JST:JST_PH_S4B-PH-SM4-TB_04x2.00mm_Angled
- U4: value MAX3232 -> MAX3232CPW; footprint (none) -> Housings_SSOP:TSSOP-16_4.4x5mm_Pitch0.65mm
Changed lines of the file:
@@
 F 0 "J5" H 2630 3292 50  0000 L CNN
 F 1 "Conn_01x04" H 2630 3201 50  0000 L CNN
-F 2 "" H 2550 3300 50  0001 C CNN
+F 2 "Connectors_JST:JST_PH_S4B-PH-SM4-TB_04x2.00mm_Angled" H 2550 3300 50  0001 C CNN
 F 3 "~" H 2550 3300 50  0001 C CNN
 	1    2550 3300
@@
 P 7350 3650
 F 0 "U4" H 7550 4750 50  0000 C CNN
-F 1 "MAX3232" H 7650 2600 50  0000 C CNN
-F 2 "" H 7400 2600 50  0001 L CNN
+F 1 "MAX3232CPW" H 7650 2600 50  0000 C CNN
+F 2 "Housings_SSOP:TSSOP-16_4.4x5mm_Pitch0.65mm" H 7400 2600 50  0001 L CNN
 F 3 "https://datasheets.maximintegrated.com/en/ds/MAX3222-MAX3241.pdf" H 7350 3750 50  0001 C CNN
 	1    7350 3650

Commit message: add CAN output on com board
Connections:
- net labels added: can_h, can_l
- wire segments 54 -> 56
Changed lines of the file:
@@
 $Descr A4 11693 8268
 encoding utf-8
-Sheet 4 4
+Sheet 3 5
 Title ""
 Date ""
@@
 Text HLabel 2950 2100 1    50   Output ~ 0
 5v
+Text HLabel 4000 3300 2    50   BiDi ~ 0
+can_h
+Text HLabel 4000 3400 2    50   BiDi ~ 0
+can_l
+Wire Wire Line
+	4000 3400 3600 3400
+Connection ~ 3600 3400
+Wire Wire Line
+	3700 3300 4000 3300
+Connection ~ 3700 3300
 $EndSCHEMATC

Commit message: com board: silkscreen and 3d
Parts:
- J5: footprint Connectors_JST:JST_PH_S4B-PH-SM4-TB_04x2.00mm_Angled -> espitall:JST_PH_S4B-PH-SM4-TB_04x2.00mm_Angled
Changed lines of the file:
@@
 encoding utf-8
 Sheet 3 5
-Title ""
-Date ""
-Rev ""
-Comp ""
+Title "Com"
+Date "2018-05-27"
+Rev "2019"
+Comp "Cocobot"
 Comment1 ""
 Comment2 ""
@@
 F 0 "J5" H 2630 3292 50  0000 L CNN
 F 1 "Conn_01x04" H 2630 3201 50  0000 L CNN
-F 2 "Connectors_JST:JST_PH_S4B-PH-SM4-TB_04x2.00mm_Angled" H 2550 3300 50  0001 C CNN
+F 2 "espitall:JST_PH_S4B-PH-SM4-TB_04x2.00mm_Angled" H 2550 3300 50  0001 C CNN
 F 3 "~" H 2550 3300 50  0001 C CNN
 	1    2550 3300

Commit message: create specific connector for CAN bus
Parts:
- removed J5: Conn_01x04, espitall:JST_PH_S4B-PH-SM4-TB_04x2.00mm_Angled, symbol com-rescue:Conn_01x04-conn
- added J2: CocobotCAN, espitall:JST_PH_S4B-PH-SM4-TB_04x2.00mm_Angled, symbol espitall:CocobotCAN
Connections:
- wire segments 56 -> 57
Changed lines of the file:
@@
 $EndDescr
-$Comp
-L com-rescue:Conn_01x04-conn J5
-U 1 1 5B7F7A0D
-P 2550 3300
-F 0 "J5" H 2630 3292 50  0000 L CNN
-F 1 "Conn_01x04" H 2630 3201 50  0000 L CNN
-F 2 "espitall:JST_PH_S4B-PH-SM4-TB_04x2.00mm_Angled" H 2550 3300 50  0001 C CNN
-F 3 "~" H 2550 3300 50  0001 C CNN
-	1    2550 3300
-	-1   0    0    -1
-$EndComp
 $Comp
 L power:GND #PWR017
@@
 	3700 3300 4000 3300
 Connection ~ 3700 3300
+$Comp
+L espitall:CocobotCAN J2
+U 1 1 5B0BC194
+P 2550 3300
+F 0 "J2" H 2570 3625 50  0000 C CNN
+F 1 "CocobotCAN" H 2570 3534 50  0000 C CNN
+F 2 "espitall:JST_PH_S4B-PH-SM4-TB_04x2.00mm_Angled" H 2500 3500 50  0001 C CNN
+F 3 "~" H 2550 3300 50  0001 C CNN
+	1    2550 3300
+	-1   0    0    -1
+$EndComp
+$Comp
+L power:GND #PWR0105
+U 1 1 5B0BCE4A
+P 2450 3950
+F 0 "#PWR0105" H 2450 3700 50  0001 C CNN
+F 1 "GND" H 2455 3777 50  0000 C CNN
+F 2 "" H 2450 3950 50  0001 C CNN
+F 3 "" H 2450 3950 50  0001 C CNN
+	1    2450 3950
+	1    0    0    -1
+$EndComp
+Wire Wire Line
+	2450 3950 2450 3700
 $EndSCHEMATC

Commit message: update com board with new CAN connector
Parts:
- J2: footprint espitall:JST_PH_S4B-PH-SM4-TB_04x2.00mm_Angled -> espitall:JST_PH_S5B-PH-SM4-TB_05x2.00mm_Angled
Connections:
- wire segments 57 -> 59
Changed lines of the file:
@@
 $EndComp
 Wire Wire Line
-	2950 3950 2950 3500
+	2950 3950 2950 3600
 Wire Wire Line
 	2950 3500 2750 3500
@@
 Connection ~ 3700 3300
 $Comp
-L espitall:CocobotCAN J2
-U 1 1 5B0BC194
-P 2550 3300
-F 0 "J2" H 2570 3625 50  0000 C CNN
-F 1 "CocobotCAN" H 2570 3534 50  0000 C CNN
-F 2 "espitall:JST_PH_S4B-PH-SM4-TB_04x2.00mm_Angled" H 2500 3500 50  0001 C CNN
-F 3 "~" H 2550 3300 50  0001 C CNN
-	1    2550 3300
-	-1   0    0    -1
-$EndComp
-$Comp
 L power:GND #PWR0105
 U 1 1 5B0BCE4A
@@
 	1    0    0    -1
 $EndComp
-Wire Wire Line
-	2450 3950 2450 3700
+$Comp
+L espitall:CocobotCAN J2
+U 1 1 5B24549B
+P 2550 3300
+F 0 "J2" H 2589 3625 50  0000 C CNN
+F 1 "CocobotCAN" H 2589 3534 50  0000 C CNN
+F 2 "espitall:JST_PH_S5B-PH-SM4-TB_05x2.00mm_Angled" H 2500 3500 50  0001 C CNN
+F 3 "~" H 2550 3300 50  0001 C CNN
+	1    2550 3300
+	-1   0    0    -1
+$EndComp
+Wire Wire Line
+	2450 3800 2450 3950
+Wire Wire Line
+	2750 3600 2950 3600
+Connection ~ 2950 3600
+Wire Wire Line
+	2950 3600 2950 3500
 $EndSCHEMATC
