File: com/uc.sch (KiCad schematic (older format))
At the start: 46 parts, among them U8 STM32F407VG, Y1 8M

Commit message: full schematic
Parts:
- C70, C71, C72, C73, C74, C75, C76, C77, C78, C79, C80, C81, C82, C85, C86: symbol device:C -> com-rescue:C-device
- C83, C84: footprint espitall:C_0603 -> espitall:C_0805; symbol device:C -> com-rescue:C-device
- J1, J2: renamed from J?; symbol conn:Conn_01x02 -> com-rescue:Conn_01x02-conn
- J3: renamed from J?; symbol conn:Conn_01x05 -> com-rescue:Conn_01x05-conn
- R1, R10, R11, R12, R13, R14, R15, R16, R17, R18, R19, R2, R20, R3, R4, R5, R6, R7, R8, R9: renamed from R?; footprint (none) -> espitall:R_0603; symbol device:R -> com-rescue:R-device
- R34, R35: symbol device:R -> com-rescue:R-device
- SW1: renamed from SW?; symbol switches:SW_DIP_x08 -> com-rescue:SW_DIP_x08-switches
- Y1: symbol device:Crystal -> com-rescue:Crystal-device
- gave numbers to parts that had none: 1

Commit message: footprint assignation
Parts:
- removed J3: Conn_01x05, symbol com-rescue:Conn_01x05-conn
- added J3: Conn_01x04, Socket_Strips:Socket_Strip_Straight_1x04_Pitch2.54mm, symbol Connector_Generic:Conn_01x04
- D1: footprint (none) -> espitall:XGURUGX10D
- J1, J2: footprint (none) -> espitall:R_0603_HandSoldering
- SW1: footprint (none) -> Buttons_Switches_THT:SW_DIP_x8_W7.62mm_Slide
Connections:
- wire segments 273 -> 271
Changed lines of the file:
@@
-$EndComp
-$Comp
-L power:+5V #PWR0203
-U 1 1 556032C9
-P 1150 5400
-F 0 "#PWR0203" H 1150 5250 50  0001 C CNN
-F 1 "+5V" H 1150 5540 50  0000 C CNN
-F 2 "" H 1150 5400 60  0000 C CNN
-F 3 "" H 1150 5400 60  0000 C CNN
-	1    1150 5400
-	1    0    0    -1
 $EndComp
 $Comp
@@
 Wire Wire Line
 	1300 5950 1300 5600
-Wire Wire Line
-	1150 5400 1150 5850
-Wire Wire Line
-	1150 5850 1100 5850
 Wire Wire Line
 	13400 8050 14450 8050
@@
 F 0 "J2" H 2030 1292 50  0000 L CNN
 F 1 "Conn_01x02" H 2030 1201 50  0000 L CNN
-F 2 "" H 1950 1300 50  0001 C CNN
+F 2 "espitall:R_0603_HandSoldering" H 1950 1300 50  0001 C CNN
 F 3 "~" H 1950 1300 50  0001 C CNN
 	1    1950 1300
@@
 F 0 "J1" H 1230 1292 50  0000 L CNN
 F 1 "Conn_01x02" H 1230 1201 50  0000 L CNN
-F 2 "" H 1150 1300 50  0001 C CNN
+F 2 "espitall:R_0603_HandSoldering" H 1150 1300 50  0001 C CNN
 F 3 "~" H 1150 1300 50  0001 C CNN
 	1    1150 1300
@@
 Wire Wire Line
 	1350 1400 1350 1750
-$Comp
-L com-rescue:Conn_01x05-conn J3
-U 1 1 5B044264
-P 900 6050
-F 0 "J3" H 980 6092 50  0000 L CNN
-F 1 "Conn_01x05" H 980 6001 50  0000 L CNN
-F 2 "" H 900 6050 50  0001 C CNN
-F 3 "~" H 900 6050 50  0001 C CNN
-	1    900  6050
-	-1   0    0    -1
-$EndComp
 Wire Wire Line
 	650  5450 650  5550
@@
 F 0 "D1" H 673 11246 50  0000 R CNN
 F 1 "XGURUGX10D" H 673 11155 50  0000 R CNN
-F 2 "" V 900 11200 50  0001 C CNN
+F 2 "espitall:XGURUGX10D" V 900 11200 50  0001 C CNN
 F 3 "" V 900 11200 50  0001 C CNN
 	1    900  10900
@@
 F 0 "SW1" H 14150 4317 50  0000 C CNN
 F 1 "SW_DIP_x08" H 14150 4226 50  0000 C CNN
-F 2 "" H 14150 3650 50  0001 C CNN
+F 2 "Buttons_Switches_THT:SW_DIP_x8_W7.62mm_Slide" H 14150 3650 50  0001 C CNN
 F 3 "" H 14150 3650 50  0001 C CNN
 	1    14150 3650
@@
 Text HLabel 14450 7350 2    60   Output ~ 0
 rf_sdn_3v3
+$Comp
+L Connector_Generic:Conn_01x04 J3
+U 1 1 5AFDF091
+P 900 6050
+F 0 "J3" H 980 6042 50  0000 L CNN
+F 1 "Conn_01x04" H 980 5951 50  0000 L CNN
+F 2 "Socket_Strips:Socket_Strip_Straight_1x04_Pitch2.54mm" H 900 6050 50  0001 C CNN
+F 3 "~" H 900 6050 50  0001 C CNN
+	1    900  6050
+	-1   0    0    -1
+$EndComp
 $EndSCHEMATC

Commit message: add CAN output on com board
Parts:
- removed C78, C79: 100n, espitall:C_0603, symbol com-rescue:C-device
- removed C83, C84: 4u7, espitall:C_0805, symbol com-rescue:C-device
- removed J2: Conn_01x02, espitall:R_0603_HandSoldering, symbol com-rescue:Conn_01x02-conn
- removed R35: 10k, espitall:R_0603, symbol com-rescue:R-device
Connections:
- net labels added: can_rx_3v3, can_tx_3v3, led_c1_10_3v3, led_c1_1_3v3, led_c1_2_3v3, led_c1_3_3v3, led_c1_4_3v3, led_c1_5_3v3, led_c1_6_3v3, led_c1_7_3v3, led_c1_8_3v3, led_c1_9_3v3, led_c2_10_3v3, led_c2_1_3v3, led_c2_2_3v3, led_c2_3_3v3, led_c2_4_3v3, led_c2_5_3v3, led_c2_6_3v3, led_c2_7_3v3, led_c2_8_3v3, led_c2_9_3v3, sw1_3v3, sw2_3v3, sw3_3v3, sw4_3v3, sw5_3v3, sw6_3v3, sw7_3v3, sw8_3v3
- net labels removed: +5V
- wire segments 271 -> 241
Other:
- moved on the sheet: SW1

Commit message: com board: silkscreen and 3d
Parts:
- SW1: footprint Buttons_Switches_THT:SW_DIP_x8_W7.62mm_Slide -> espitall:SW_DIP_x8_W7.62mm_Slide
Changed lines of the file:
@@
 encoding utf-8
 Sheet 4 5
-Title "Brain"
-Date "2017-05-28"
-Rev "2018"
+Title "Com"
+Date "2018-05-27"
+Rev "2019"
 Comp "Cocobot"
 Comment1 "Board for eurobot 2018 (French edition)"
@@
 P 900 10900
 F 0 "D1" H 673 11246 50  0000 R CNN
-F 1 "XGURUGX10D" H 673 11155 50  0000 R CNN
+F 1 "XGURUGX10D" H 5100 11000 50  0000 R CNN
 F 2 "espitall:XGURUGX10D" V 900 11200 50  0001 C CNN
 F 3 "" V 900 11200 50  0001 C CNN
@@
 F 0 "SW1" H 14800 2117 50  0000 C CNN
 F 1 "SW_DIP_x08" H 14800 2026 50  0000 C CNN
-F 2 "Buttons_Switches_THT:SW_DIP_x8_W7.62mm_Slide" H 14800 1450 50  0001 C CNN
+F 2 "espitall:SW_DIP_x8_W7.62mm_Slide" H 14800 1450 50  0001 C CNN
 F 3 "" H 14800 1450 50  0001 C CNN
 	1    14800 1450

Commit message: add electrical protection on CAN bus
Parts:
- added C14: 100n, espitall:C_0603, symbol Device:C
- added R25, R26: 2k2, espitall:R_0603, symbol Device:R
- added U6: 24LC64T-I, espitall:SOT-23-5, symbol espitall:24LC64T-I
Connections:
- wire segments 241 -> 234
