File: brain_2019/encoders.sch (KiCad schematic (older format))
At the start: 8 parts, among them J7 JST_PH_S4B-PH-SM4-TB_04x2.00m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, J8 JST_PH_S4B-PH-SM4-TB_04x2.00m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

Commit message: brain 2019 layout
Parts:
- C22: value C -> 100n
- gave numbers to parts that had none: 1
Changed lines of the file:
@@
 P 7750 2000
 F 0 "C22" V 7498 2000 50  0000 C CNN
-F 1 "C" V 7589 2000 50  0000 C CNN
+F 1 "100n" V 7589 2000 50  0000 C CNN
 F 2 "espitall:C_0603" H 7788 1850 50  0001 C CNN
 F 3 "~" H 7750 2000 50  0001 C CNN
@@
 	5950 4450 6400 4450
 $Comp
-L espitall:MC74VHC244DTG U?
+L espitall:MC74VHC244DTG U5
 U 1 1 5B1EDE70
 P 7400 2900
-F 0 "U?" H 7150 3600 50  0000 C CNN
+F 0 "U5" H 7150 3600 50  0000 C CNN
 F 1 "MC74VHC244DTG" H 7800 2250 50  0000 C CNN
 F 2 "espitall:TSSOP-20_4.4x6.5mm_Pitch0.65mm" H 7000 3450 50  0001 C CNN
