File: brain_2019/io.sch (KiCad schematic (older format))
At the start: 2 parts, among them J9 JST_PH_S2B-PH-SM4-TB_02x2.00m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

Commit message: brain 2019 layout
Parts:
- R12: value R -> 10k
Changed lines of the file:
@@
 P 3700 2450
 F 0 "R12" H 3770 2496 50  0000 L CNN
-F 1 "R" H 3770 2405 50  0000 L CNN
+F 1 "10k" H 3770 2405 50  0000 L CNN
 F 2 "espitall:R_0603" V 3630 2450 50  0001 C CNN
 F 3 "~" H 3700 2450 50  0001 C CNN
