File: brain_2019/uc.sch (KiCad schematic (older format))
At the start: 22 parts, among them J5 Conn_01x02, J6 Conn_01x04, U4 STM32F407VG, Y1 8M

Commit message: brain 2019 layout
Parts:
- removed D4: LED, espitall:LED_0805, symbol Device:LED
- removed R7: 220, espitall:R_0603, symbol Device:R
- added C23: 100n, espitall:C_0603, symbol Device:C
- added R13, R14: 2k2, espitall:R_0603, symbol Device:R
- added U6: 24LC64T-I, espitall:SOT-23-5, symbol espitall:24LC64T-I
Connections:
- wire segments 112 -> 125
Changed lines of the file:
@@
 	-1   0    0    -1
 $EndComp
-Text Label 13500 5050 0    60   ~ 0
+Text HLabel 13800 5050 2    60   Output ~ 0
 can_tx_3v3
-Text Label 13500 5150 0    60   ~ 0
+Text HLabel 13800 5150 2    60   Input ~ 0
 can_rx_3v3
-Text HLabel 14450 5050 2    60   Output ~ 0
-can_tx_3v3
-Text HLabel 14450 5150 2    60   Input ~ 0
-can_rx_3v3
-Wire Wire Line
-	13400 5050 14450 5050
-Wire Wire Line
-	13400 5150 14450 5150
+Wire Wire Line
+	13400 5050 13800 5050
+Wire Wire Line
+	13400 5150 13800 5150
 Wire Wire Line
 	1750 1850 1750 2600
-Wire Wire Line
-	14450 5100 14450 5050
 Text HLabel 13800 6850 2    50   Input ~ 0
 vbatmon_0-3v3
 Wire Wire Line
 	13800 6850 13400 6850
-Text HLabel 13800 8150 2    60   Output ~ 0
+Text HLabel 13800 5250 2    60   Output ~ 0
 spi_gyro_~cs~_3v3
 Wire Wire Line
-	13400 8150 13800 8150
+	13400 5250 13800 5250
 Text HLabel 3000 6550 0    50   Input ~ 0
 enc_l_A_3v3
@@
 	3000 5150 3400 5150
 Wire Wire Line
-	13400 7050 13800 7050
-Text HLabel 13800 7050 2    50   Input ~ 0
+	13400 4050 13800 4050
+Text HLabel 13800 4050 2    50   Input ~ 0
 starter_3v3
-$Comp
-L power:GND #PWR039
-U 1 1 5B1CABEE
-P 2750 9400
-F 0 "#PWR039" H 2750 9150 50  0001 C CNN
-F 1 "GND" H 2750 9250 50  0000 C CNN
-F 2 "" H 2750 9400 60  0000 C CNN
-F 3 "" H 2750 9400 60  0000 C CNN
-	1    2750 9400
-	1    0    0    -1
-$EndComp
-$Comp
-L Device:LED D4
-U 1 1 5B1CDCE4
-P 2750 8950
-F 0 "D4" V 2788 8833 50  0000 R CNN
-F 1 "LED" V 2697 8833 50  0000 R CNN
-F 2 "espitall:LED_0805" H 2750 8950 50  0001 C CNN
-F 3 "~" H 2750 8950 50  0001 C CNN
-	1    2750 8950
-	0    -1   -1   0
-$EndComp
-Wire Wire Line
-	2750 9100 2750 9400
-$Comp
-L Device:R R7
-U 1 1 5B1D0C8C
-P 2750 8450
-F 0 "R7" H 2820 8496 50  0000 L CNN
-F 1 "220" H 2820 8405 50  0000 L CNN
-F 2 "espitall:R_0603" V 2680 8450 50  0001 C CNN
-F 3 "~" H 2750 8450 50  0001 C CNN
-	1    2750 8450
-	1    0    0    -1
-$EndComp
-Wire Wire Line
-	2750 8600 2750 8800
-Wire Wire Line
-	2750 8300 2750 7950
-Wire Wire Line
-	2750 7950 3400 7950
 $Comp
 L power:GND #PWR038
@@
 Wire Wire Line
 	2400 8600 2400 8800
-Wire Wire Line
-	3400 7850 2400 7850
-Wire Wire Line
-	2400 7850 2400 8300
+$Comp
+L espitall:24LC64T-I U6
+U 1 1 5B1D735A
+P 1250 7450
+F 0 "U6" H 920 7496 50  0000 R CNN
+F 1 "24LC64T-I" H 920 7405 50  0000 R CNN
+F 2 "espitall:SOT-23-5" H 1300 7600 50  0001 C CNN
+F 3 "" H 1400 7700 50  0001 C CNN
+	1    1250 7450
+	1    0    0    -1
+$EndComp
+Wire Wire Line
+	3400 7450 2100 7450
+Wire Wire Line
+	1850 7550 1850 7350
+Wire Wire Line
+	1850 7350 1650 7350
+Wire Wire Line
+	1650 7550 1750 7550
+Wire Wire Line
+	1750 7550 1750 7650
+Wire Wire Line
+	1750 7650 3400 7650
+$Comp
+L Device:R R13
+U 1 1 5B1E6581
+P 1850 7050
+F 0 "R13" H 1920 7096 50  0000 L CNN
+F 1 "2k2" H 1920 7005 50  0000 L CNN
+F 2 "espitall:R_0603" V 1780 7050 50  0001 C CNN
+F 3 "~" H 1850 7050 50  0001 C CNN
+	1    1850 7050
+	1    0    0    -1
+$EndComp
+$Comp
+L Device:R R14
+U 1 1 5B1E65E3
+P 2100 7050
+F 0 "R14" H 2170 7096 50  0000 L CNN
+F 1 "2k2" H 2170 7005 50  0000 L CNN
+F 2 "espitall:R_0603" V 2030 7050 50  0001 C CNN
+F 3 "~" H 2100 7050 50  0001 C CNN
+	1    2100 7050
+	1    0    0    -1
+$EndComp
+$Comp
+L power:+3V3 #PWR0101
+U 1 1 5B1E665D
+P 1850 6800
+F 0 "#PWR0101" H 1850 6650 50  0001 C CNN
+F 1 "+3V3" H 1850 6940 50  0000 C CNN
+F 2 "" H 1850 6800 60  0000 C CNN
+F 3 "" H 1850 6800 60  0000 C CNN
+	1    1850 6800
+	1    0    0    -1
+$EndComp
+Wire Wire Line
+	1850 6800 1850 6900
+$Comp
+L power:+3V3 #PWR0102
+U 1 1 5B1EA768
+P 2100 6800
+F 0 "#PWR0102" H 2100 6650 50  0001 C CNN
+F 1 "+3V3" H 2100 6940 50  0000 C CNN
+F 2 "" H 2100 6800 60  0000 C CNN
+F 3 "" H 2100 6800 60  0000 C CNN
+	1    2100 6800
+	1    0    0    -1
+$EndComp
+Wire Wire Line
+	2100 6800 2100 6900
+$Comp
+L power:+3V3 #PWR0103
+U 1 1 5B1EE965
+P 1250 6800
+F 0 "#PWR0103" H 1250 6650 50  0001 C CNN
+F 1 "+3V3" H 1250 6940 50  0000 C CNN
+F 2 "" H 1250 6800 60  0000 C CNN
+F 3 "" H 1250 6800 60  0000 C CNN
+	1    1250 6800
+	1    0    0    -1
+$EndComp
+Wire Wire Line
+	1250 6800 1250 6950
+Wire Wire Line
+	1850 7200 1850 7350
+Connection ~ 1850 7350
+$Comp
+L Device:C C23
+U 1 1 5B1FFBD5
+P 1000 6950
+F 0 "C23" V 748 6950 50  0000 C CNN
+F 1 "100n" V 839 6950 50  0000 C CNN
+F 2 "espitall:C_0603" H 1038 6800 50  0001 C CNN
+F 3 "~" H 1000 6950 50  0001 C CNN
+	1    1000 6950
+	0    1    1    0
+$EndComp
+$Comp
+L power:GND #PWR0104
+U 1 1 5B1FFC9A
+P 700 7050
+F 0 "#PWR0104" H 700 6800 50  0001 C CNN
+F 1 "GND" H 700 6900 50  0000 C CNN
+F 2 "" H 700 7050 60  0000 C CNN
+F 3 "" H 700 7050 60  0000 C CNN
+	1    700  7050
+	1    0    0    -1
+$EndComp
+Wire Wire Line
+	700  7050 700  6950
+Wire Wire Line
+	700  6950 850  6950
+Wire Wire Line
+	1150 6950 1250 6950
+Connection ~ 1250 6950
+Wire Wire Line
+	1250 6950 1250 7150
+$Comp
+L power:GND #PWR0105
+U 1 1 5B20931B
+P 1250 9400
+F 0 "#PWR0105" H 1250 9150 50  0001 C CNN
+F 1 "GND" H 1250 9250 50  0000 C CNN
+F 2 "" H 1250 9400 60  0000 C CNN
+F 3 "" H 1250 9400 60  0000 C CNN
+	1    1250 9400
+	1    0    0    -1
+$EndComp
+Wire Wire Line
+	1250 7750 1250 9400
+Wire Wire Line
+	1850 7550 3400 7550
+Wire Wire Line
+	2100 7450 2100 7200
+Connection ~ 2100 7450
+Wire Wire Line
+	2100 7450 1650 7450
+Wire Wire Line
+	3400 7750 2400 7750
+Wire Wire Line
+	2400 7750 2400 8300
 $EndSCHEMATC
