File: brain_2019/can.sch (KiCad schematic (older format))
At the start: 11 parts, among them J1 CocobotCAN, J2 CocobotCAN, U1 MAX3051ESA

Commit message: brain 2019 layout
Parts:
- gave numbers to parts that had none: 2
Changed lines of the file:
@@
 	5950 3600 6650 3600
 $Comp
-L espitall:NUP2105LT1G D?
+L espitall:NUP2105LT1G D1
 U 1 1 5B1ED698
 P 7150 4200
-F 0 "D?" H 7150 4416 50  0000 C CNN
+F 0 "D1" H 7150 4416 50  0000 C CNN
 F 1 "NUP2105LT1G" H 7150 4325 50  0000 C CNN
 F 2 "espitall:SOT-23" H 7000 4200 50  0001 C CNN
@@
 $EndComp
 $Comp
-L espitall:DR331-113BE FL?
+L espitall:DR331-113BE FL1
 U 1 1 5B1C2674
 P 5050 3500
-F 0 "FL?" H 5050 3778 50  0000 C CNN
+F 0 "FL1" H 5050 3778 50  0000 C CNN
 F 1 "DR331-113BE" H 5050 3687 50  0000 C CNN
 F 2 "espitall:DR331" H 5050 3540 50  0001 C CNN
 F 3 "" V 5050 3540 50  0000 C CNN
 	1    5050 3500
-	1    0    0    -1
+	1    0    0    1
 $EndComp
 $EndSCHEMATC

Commit message: Update brain 2019 with new CAN connector
Parts:
- J1, J2: footprint espitall:JST_PH_S4B-PH-SM4-TB_04x2.00mm_Angled -> espitall:JST_PH_S5B-PH-SM4-TB_05x2.00mm_Angled
Connections:
- wire segments 57 -> 61
Changed lines of the file:
@@
 Connection ~ 2150 3700
-$Comp
-L espitall:CocobotCAN J1
-U 1 1 5B1D7055
-P 8000 3450
-F 0 "J1" H 8279 3370 50  0000 L CNN
-F 1 "CocobotCAN" H 8279 3279 50  0000 L CNN
-F 2 "espitall:JST_PH_S4B-PH-SM4-TB_04x2.00mm_Angled" H 7950 3650 50  0001 C CNN
-F 3 "~" H 8000 3450 50  0001 C CNN
-	1    8000 3450
-	1    0    0    -1
-$EndComp
 $Comp
 L power:GND #PWR010
@@
 $EndComp
 Wire Wire Line
-	8100 3850 8100 3950
-Wire Wire Line
-	8100 3950 7650 3950
-Wire Wire Line
-	7650 3950 7650 3650
-Wire Wire Line
-	7650 3650 7800 3650
-Connection ~ 8100 3950
-Wire Wire Line
-	8100 3950 8100 4450
-$Comp
-L espitall:CocobotCAN J2
-U 1 1 5B1D7321
-P 9100 3450
-F 0 "J2" H 9379 3370 50  0000 L CNN
-F 1 "CocobotCAN" H 9379 3279 50  0000 L CNN
-F 2 "espitall:JST_PH_S4B-PH-SM4-TB_04x2.00mm_Angled" H 9050 3650 50  0001 C CNN
-F 3 "~" H 9100 3450 50  0001 C CNN
-	1    9100 3450
-	1    0    0    -1
-$EndComp
+	7700 3650 7800 3650
 $Comp
 L power:GND #PWR011
@@
 $EndComp
 Wire Wire Line
-	9200 4450 9200 3950
-Wire Wire Line
-	9200 3950 8800 3950
-Wire Wire Line
-	8800 3950 8800 3650
-Wire Wire Line
 	8800 3650 8900 3650
-Connection ~ 9200 3950
-Wire Wire Line
-	9200 3950 9200 3850
-Wire Wire Line
-	8900 3550 7800 3550
-Wire Wire Line
-	7800 3550 7200 3550
 Wire Wire Line
 	6650 3550 6650 3600
 Wire Wire Line
 	3650 3600 4400 3600
-Connection ~ 7800 3550
 Wire Wire Line
 	6650 3400 6650 3450
@@
 Wire Wire Line
 	3650 3400 4050 3400
-Wire Wire Line
-	8900 3450 7800 3450
-Connection ~ 7800 3450
 Wire Wire Line
 	7800 3350 8900 3350
@@
 	7100 3850 7100 3450
 Connection ~ 7100 3450
-Wire Wire Line
-	7100 3450 7800 3450
 $Comp
 L Device:C C2
@@
 	1    0    0    1
 $EndComp
+Wire Wire Line
+	7100 3450 7800 3450
+Wire Wire Line
+	7200 3550 7800 3550
+$Comp
+L espitall:CocobotCAN J1
+U 1 1 5B243B36
+P 8000 3450
+F 0 "J1" H 8319 3320 50  0000 L CNN
+F 1 "CocobotCAN" H 8319 3229 50  0000 L CNN
+F 2 "espitall:JST_PH_S5B-PH-SM4-TB_05x2.00mm_Angled" H 7950 3650 50  0001 C CNN
+F 3 "~" H 8000 3450 50  0001 C CNN
+	1    8000 3450
+	1    0    0    -1
+$EndComp
+Connection ~ 7800 3450
+Wire Wire Line
+	7800 3450 8900 3450
+Connection ~ 7800 3550
+Wire Wire Line
+	7800 3550 8900 3550
+Wire Wire Line
+	8100 3950 8100 4350
+Wire Wire Line
+	7800 3750 7700 3750
+Connection ~ 7700 3750
+Wire Wire Line
+	7700 3750 7700 3650
+Wire Wire Line
+	7700 4350 8100 4350
+Wire Wire Line
+	7700 3750 7700 4350
+Connection ~ 8100 4350
+Wire Wire Line
+	8100 4350 8100 4450
+$Comp
+L espitall:CocobotCAN J2
+U 1 1 5B2460BB
+P 9100 3450
+F 0 "J2" H 9419 3320 50  0000 L CNN
+F 1 "CocobotCAN" H 9419 3229 50  0000 L CNN
+F 2 "espitall:JST_PH_S5B-PH-SM4-TB_05x2.00mm_Angled" H 9050 3650 50  0001 C CNN
+F 3 "~" H 9100 3450 50  0001 C CNN
+	1    9100 3450
+	1    0    0    -1
+$EndComp
+Wire Wire Line
+	8900 3750 8800 3750
+Connection ~ 8800 3750
+Wire Wire Line
+	8800 3750 8800 3650
+Wire Wire Line
+	9200 3950 9200 4350
+Wire Wire Line
+	9200 4350 8800 4350
+Wire Wire Line
+	8800 3750 8800 4350
+Connection ~ 9200 4350
+Wire Wire Line
+	9200 4350 9200 4450
 $EndSCHEMATC
