File: canexpander/canexpander.sch (KiCad schematic (older format))
At the start: 8 parts, among them J1 CocobotCAN, J2 CocobotCAN, J3 CocobotCAN, J4 CocobotCAN, J5 CocobotCAN, J6 Conn_01x01, J7 Conn_01x01

Commit message: Add protection diodes on CANexpander board
Parts:
- added D1: NUP2105LT1G, espitall:SOT-23, symbol espitall:NUP2105LT1G
Connections:
- wire segments 48 -> 56
Changed lines of the file:
@@
 EESchema Schematic File Version 4
+LIBS:canexpander-cache
 EELAYER 26 0
 EELAYER END
@@
 L espitall:CocobotCAN J1
 U 1 1 5B0ACFB2
-P 3500 3600
-F 0 "J1" H 3520 3925 50  0000 C CNN
-F 1 "CocobotCAN" H 3520 3834 50  0000 C CNN
-F 2 "espitall:JST_PH_S4B-PH-SM4-TB_04x2.00mm_Angled" H 3450 3800 50  0001 C CNN
-F 3 "~" H 3500 3600 50  0001 C CNN
-	1    3500 3600
+P 2400 3600
+F 0 "J1" H 2420 3925 50  0000 C CNN
+F 1 "CocobotCAN" H 2420 3834 50  0000 C CNN
+F 2 "espitall:JST_PH_S4B-PH-SM4-TB_04x2.00mm_Angled" H 2350 3800 50  0001 C CNN
+F 3 "~" H 2400 3600 50  0001 C CNN
+	1    2400 3600
 	-1   0    0    -1
 $EndComp
@@
 $EndComp
 Wire Wire Line
-	3700 3500 4450 3500
+	2600 3500 4450 3500
 Wire Wire Line
 	7350 3600 6950 3600
 Wire Wire Line
-	3700 3700 4250 3700
+	2600 3700 2850 3700
 Wire Wire Line
 	7350 3800 6100 3800
@@
 Connection ~ 4150 3800
 Wire Wire Line
-	4150 3800 3850 3800
+	4150 3800 2700 3800
 Wire Wire Line
 	4250 3700 4250 4350
@@
 Connection ~ 4350 3600
 Wire Wire Line
-	4350 3600 3700 3600
+	4350 3600 3800 3600
 Wire Wire Line
 	4450 3500 4450 4350
@@
 L power:GND #PWR0101
 U 1 1 5B0ADDDD
-P 3400 5150
-F 0 "#PWR0101" H 3400 4900 50  0001 C CNN
-F 1 "GND" H 3405 4977 50  0000 C CNN
-F 2 "" H 3400 5150 50  0001 C CNN
-F 3 "" H 3400 5150 50  0001 C CNN
-	1    3400 5150
-	1    0    0    -1
-$EndComp
-Wire Wire Line
-	3400 5150 3400 5000
-Wire Wire Line
-	3950 4650 3400 4650
-Connection ~ 3400 4650
-Wire Wire Line
-	3400 4650 3400 4100
-Wire Wire Line
-	3400 5000 4800 5000
+P 2300 5150
+F 0 "#PWR0101" H 2300 4900 50  0001 C CNN
+F 1 "GND" H 2305 4977 50  0000 C CNN
+F 2 "" H 2300 5150 50  0001 C CNN
+F 3 "" H 2300 5150 50  0001 C CNN
+	1    2300 5150
+	1    0    0    -1
+$EndComp
+Wire Wire Line
+	2300 5150 2300 5000
+Wire Wire Line
+	3950 4650 3300 4650
+Connection ~ 2300 4650
+Wire Wire Line
+	2300 4650 2300 4100
+Wire Wire Line
+	2300 5000 4800 5000
 Wire Wire Line
 	5750 5000 5750 4650
 Wire Wire Line
 	5750 4650 5900 4650
-Connection ~ 3400 5000
-Wire Wire Line
-	3400 5000 3400 4650
+Connection ~ 2300 5000
+Wire Wire Line
+	2300 5000 2300 4650
 Wire Wire Line
 	5000 4650 4800 4650
@@
 	4800 5000 5750 5000
 Wire Wire Line
-	3850 3800 3850 4100
-Wire Wire Line
-	3850 4100 3400 4100
-Connection ~ 3850 3800
-Wire Wire Line
-	3850 3800 3700 3800
-Connection ~ 3400 4100
-Wire Wire Line
-	3400 4100 3400 4000
+	2700 3800 2700 4100
+Wire Wire Line
+	2700 4100 2300 4100
+Connection ~ 2700 3800
+Wire Wire Line
+	2700 3800 2600 3800
+Connection ~ 2300 4100
+Wire Wire Line
+	2300 4100 2300 4000
 $Comp
 L Connector_Generic:Conn_01x01 J6
@@
 	7650 4000 7650 5000
 Connection ~ 5750 5000
+$Comp
+L espitall:NUP2105LT1G D1
+U 1 1 5B201D11
+P 3300 4150
+F 0 "D1" H 3300 4366 50  0000 C CNN
+F 1 "NUP2105LT1G" H 3300 4275 50  0000 C CNN
+F 2 "espitall:SOT-23" H 3150 4150 50  0001 C CNN
+F 3 "~" H 3150 4150 50  0001 C CNN
+	1    3300 4150
+	1    0    0    -1
+$EndComp
+Wire Wire Line
+	3300 4300 3300 4650
+Connection ~ 3300 4650
+Wire Wire Line
+	3300 4650 2300 4650
+Wire Wire Line
+	2950 4150 2850 4150
+Wire Wire Line
+	2850 4150 2850 3700
+Connection ~ 2850 3700
+Wire Wire Line
+	2850 3700 4250 3700
+Wire Wire Line
+	3650 4150 3800 4150
+Wire Wire Line
+	3800 4150 3800 3600
+Connection ~ 3800 3600
+Wire Wire Line
+	3800 3600 2600 3600
 $EndSCHEMATC

Commit message: add step on gitignore
Parts:
- added J8: CocobotCAN, espitall:JST_PH_S5B-PH-SM4-TB_05x2.00mm_Angled, symbol espitall:CocobotCAN
- J1, J2, J3, J4, J5: footprint espitall:JST_PH_S4B-PH-SM4-TB_04x2.00mm_Angled -> espitall:JST_PH_S5B-PH-SM4-TB_05x2.00mm_Angled
Connections:
- wire segments 56 -> 89
