File: canivo/canivo.kicad_pcb (KiCad board)
At the start: 2 copper layers, 36 x 16 mm, 0 parts

Commit message: Canivo layout
Parts:
- added C1: 100n, espitall:C_0603, B.Cu at (57.2, 51.7)
- added C2: 100n, espitall:C_0603, B.Cu at (57.2, 54.6)
- added C3: 100n, espitall:C_0603, B.Cu at (66.0, 59.6)
- added C4: 100n, espitall:C_0603, F.Cu at (60.9, 51.3)
- added C5: 100n, espitall:C_0603, B.Cu at (59.4, 55.3)
- added C6: 100n, espitall:C_0603, B.Cu at (53.4, 57.9)
- added C7: 100n, espitall:C_0603, F.Cu at (68.9, 61.4)
- added J1: Conn_01x02, Pin_Headers:Pin_Header_Straight_1x02_Pitch2.54mm, F.Cu at (51.6, 56.2)
- added J2: Conn_01x04, Pin_Headers:Pin_Header_Straight_1x04_Pitch2.54mm, F.Cu at (63.6, 64.6)
- added J3: Conn_01x02, espitall:R_0603, F.Cu at (51.1, 61.8)
- added J4: Conn_01x01, Pin_Headers:Pin_Header_Straight_1x01_Pitch2.54mm, F.Cu at (78.5, 53.2)
- added J5: Conn_01x01, Pin_Headers:Pin_Header_Straight_1x01_Pitch2.54mm, F.Cu at (78.7, 62.5)
- added J6: Conn_01x03, Pin_Headers:Pin_Header_Straight_1x03_Pitch2.54mm, F.Cu at (84.7, 60.4)
- added J7: Conn_01x05, Pin_Headers:Pin_Header_Straight_1x05_Pitch2.54mm, F.Cu at (55.2, 62.3)
- added Q1: DMC3025LSD, espitall:SOIC-8_3.9x4.9mm_Pitch1.27mm, B.Cu at (71.1, 55.5)
- added Q2: DMC3025LSD, espitall:SOIC-8_3.9x4.9mm_Pitch1.27mm, B.Cu at (71.1, 61.0)
- added R1: 0.05, espitall:R_2010, B.Cu at (64.1, 54.5)
- added R2: 1k, espitall:R_0603, F.Cu at (62.5, 51.2)
- added R3: 100k, espitall:R_0603, F.Cu at (70.7, 59.6)
- added R4: 100k, espitall:R_0603, F.Cu at (70.7, 54.3)
- added R5: 1k, espitall:R_0603, F.Cu at (64.1, 51.2)
- added R6: 10k, espitall:R_0603, F.Cu at (52.8, 61.8)
- added R7: 100k, espitall:R_0603, F.Cu at (70.7, 56.9)
- added R8: 100k, espitall:R_0603, F.Cu at (70.7, 62.2)
- added R9: 10, espitall:R_0603, F.Cu at (68.9, 58.5)
- added U1: LM3480IM3-3.3, espitall:SOT-23, B.Cu at (59.7, 51.9)
- added U2: ZXCT1009FTA, espitall:SOT-23, B.Cu at (63.2, 51.6)
- added U3: STM32F042F6P6, espitall:TSSOP-20_4.4x6.5mm_Pitch0.65mm, B.Cu at (61.2, 59.6)
- added U4: ISO1050DW, espitall:SOIC-16W_7.5x10.3mm_Pitch1.27mm, F.Cu at (62.4, 57.7)
Routing:
- net GND: track 0.00 -> 125.0 mm, vias 0 -> 5
- net Net-(J6-Pad2): track 0.00 -> 46.0 mm, vias 0 -> 3
- net +3V3: track 0.00 -> 45.0 mm, vias 0 -> 5
- net Net-(J6-Pad1): track 0.00 -> 40.9 mm, vias 0 -> 2
- net Net-(D1-Pad1): track 0.00 -> 23.8 mm, vias 0 -> 2
- net Net-(D2-Pad2): track 0.00 -> 20.4 mm, vias 0 -> 1
- net Net-(D1-Pad2): track 0.00 -> 20.2 mm, vias 0 -> 2
- net Net-(C6-Pad2): track 0.00 -> 18.3 mm
- net +5P: track 0.00 -> 17.6 mm
- net Net-(J2-Pad2): track 0.00 -> 13.5 mm
- net Net-(J3-Pad2): track 0.00 -> 13.0 mm, vias 0 -> 1
- net Net-(Q2-Pad2): track 0.00 -> 12.5 mm, vias 0 -> 3
- net Net-(J2-Pad3): track 0.00 -> 11.0 mm
- net Net-(Q1-Pad2): track 0.00 -> 9.78 mm, vias 0 -> 2
- net Net-(C6-Pad1): track 0.00 -> 7.65 mm
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- added copper zone on B.Cu, net GND
- added copper zone on F.Cu, net GND
- added copper zone on B.Cu, net Net-(D1-Pad1)
Other:
- board text added: "CANivo"
- board text added: "Cocobot 2019"
- board text added: "D1/D2/D3/D4 sont à placer sur la 3ème couche de composants ;)"
