File: canivo/canivo.sch (KiCad schematic (older format))
At the start: 4 parts

Commit message: CANivo schematic
Parts:
- removed U?: LM3940IMP-3.3, espitall:SOT-223-3_TabPin2, symbol espitall:LM3940IMP-3.3
- added C? (x6): 100n, espitall:C_0603, symbol Device:C
- added J?: Conn_01x03, symbol Connector_Generic:Conn_01x03
- added J?: Conn_01x02, symbol Connector_Generic:Conn_01x02
- added J?: Conn_01x04, symbol Connector_Generic:Conn_01x04
- added J?: CocobotCAN, espitall:JST_PH_S4B-PH-SM4-TB_04x2.00mm_Angled, symbol espitall:CocobotCAN
- added J? (x2): Conn_01x01, symbol Connector_Generic:Conn_01x01
- added Q? (x4): DMC3025LSD, espitall:SOIC-8_3.9x4.9mm_Pitch1.27mm, symbol espitall:DMC3025LSD
- added R?: 10k, espitall:R_0603, symbol Device:R
- added R?: 10, espitall:R_0603, symbol Device:R
- added R? (x4): 100k, espitall:R_0603, symbol Device:R
- added R?: 0.05, symbol Device:R
- added R? (x2): 1k, espitall:R_0603, symbol Device:R
- added U?: ISO1050DW, espitall:SOIC-16W_7.5x10.3mm_Pitch1.27mm, symbol espitall:ISO1050DW
- added U?: ZXCT1009FTA, espitall:SOT-23, symbol espitall:ZXCT1009FTA
- added U?: LM3480IM3-3.3, espitall:SOT-23, symbol espitall:LM3480IM3-3.3
- C?: value C -> 100n; footprint (none) -> espitall:C_0603
Connections:
- wire segments 16 -> 165

Commit message: Canivo layout
Parts:
- removed J?: JST_PH_S2B-PH-SM4-TB_02x2.00mm_Angled, espitall:JST_PH_S2B-PH-SM4-TB_02x2.00mm_Angled, symbol espitall:JST_PH_S2B-PH-SM4-TB_02x2.00mm_Angled
- removed J?: CocobotCAN, espitall:JST_PH_S4B-PH-SM4-TB_04x2.00mm_Angled, symbol espitall:CocobotCAN
- added D1, D2, D3, D4: D, symbol Device:D
- added J1: Conn_01x02, Pin_Headers:Pin_Header_Straight_1x02_Pitch2.54mm, symbol Connector_Generic:Conn_01x02
- added J7: Conn_01x05, Pin_Headers:Pin_Header_Straight_1x05_Pitch2.54mm, symbol Connector_Generic:Conn_01x05
- J2: renamed from J?; footprint (none) -> Pin_Headers:Pin_Header_Straight_1x04_Pitch2.54mm
- J3: renamed from J?; footprint (none) -> espitall:R_0603
- J4, J5: renamed from J?; footprint (none) -> Pin_Headers:Pin_Header_Straight_1x01_Pitch2.54mm
- J6: renamed from J?; footprint (none) -> Pin_Headers:Pin_Header_Straight_1x03_Pitch2.54mm
- R1: renamed from R?; footprint (none) -> espitall:R_2010
- gave numbers to parts that had none: 21
Connections:
- wire segments 165 -> 185
