File: meca_2019/meca_2019.kicad_pcb (KiCad board)
At the start: 2 copper layers, 54 x 50 mm, 60 parts, among them J1 CocobotCAN, J2 CocobotCAN, J3 JST_PH_S6B-PH-SM4-TB_06x2.00m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, J4 JST_PH_S2B-PH-SM4-TB_02x2.00m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, J5 Conn_01x02, J6 Conn_01x04, J7 JST_PH_S4B-PH-SM4-TB_04x2.00m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, J8 JST_PH_S4B-PH-SM4-TB_04x2.00m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, J9 JST_PH_S2B-PH-SM4-TB_02x2.00m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, U1 MAX3051ESA, U2 TSR1-2450, U3 LM3940IMP-3.3, U4 STM32F407VG, U5 MC74VHC244DTG, U6 24LC64T-I, Y1 8M

Commit message: meca 2019 board
Parts:
- removed C9: 10u, espitall:C_0603
- added C24: 100n, espitall:C_0603, F.Cu at (60.6, 70.6)
- added C25: 100n, espitall:C_0603, B.Cu at (88.3, 68.7)
- added C26: 100n, espitall:C_0603, F.Cu at (61.6, 88.5)
- added C27: 100n, espitall:C_0603, F.Cu at (61.5, 80.5)
- added C28: 100n, espitall:C_0603, F.Cu at (75.4, 80.3)
- added C29: 100n, espitall:C_0603, F.Cu at (75.4, 88.5)
- added J10: Conn_01x03, espitall:Pin_Header_Straight_1x03_Pitch2.54mm, F.Cu at (92.2, 70.0)
- added J11: Conn_01x03, espitall:Pin_Header_Straight_1x03_Pitch2.54mm, F.Cu at (92.2, 72.5)
- added J12: Conn_01x03, espitall:Pin_Header_Straight_1x03_Pitch2.54mm, F.Cu at (92.2, 75.0)
- added J13: Conn_01x03, espitall:Pin_Header_Straight_1x03_Pitch2.54mm, F.Cu at (92.2, 80.1)
- added J14: Conn_01x03, espitall:Pin_Header_Straight_1x03_Pitch2.54mm, F.Cu at (92.2, 82.7)
- added J15: Conn_01x03, espitall:Pin_Header_Straight_1x03_Pitch2.54mm, F.Cu at (92.2, 85.2)
- added J16: Conn_01x03, espitall:Pin_Header_Straight_1x03_Pitch2.54mm, F.Cu at (92.2, 77.6)
- added J17: Conn_01x03, espitall:Pin_Header_Straight_1x03_Pitch2.54mm, F.Cu at (92.2, 87.7)
- added J18: Conn_01x03, espitall:Pin_Header_Straight_1x03_Pitch2.54mm, F.Cu at (92.2, 90.3)
- added J19: Conn_01x03, espitall:Pin_Header_Straight_1x03_Pitch2.54mm, F.Cu at (92.2, 92.8)
- added J20: Conn_01x03, espitall:Pin_Header_Straight_1x03_Pitch2.54mm, F.Cu at (92.2, 95.4)
- added J21: Conn_01x03, espitall:Pin_Header_Straight_1x03_Pitch2.54mm, F.Cu at (64.7, 81.7)
- added J22: Conn_01x03, espitall:Pin_Header_Straight_1x03_Pitch2.54mm, F.Cu at (67.2, 81.7)
- added J23: Conn_01x03, espitall:Pin_Header_Straight_1x03_Pitch2.54mm, F.Cu at (69.8, 81.7)
- added J24: Conn_01x03, espitall:Pin_Header_Straight_1x03_Pitch2.54mm, F.Cu at (72.3, 81.7)
- added R15: R, espitall:R_0603, F.Cu at (75.4, 81.9)
- added R16: R, espitall:R_0603, F.Cu at (75.4, 85.3)
- added R17: R, espitall:R_0603, F.Cu at (75.4, 86.9)
- added R18: 10k, espitall:R_0603, F.Cu at (64.7, 75.3)
- added R7: 10k, espitall:R_0603, F.Cu at (51.9, 78.4)
- C10, C11, C12, C13, C14, C17, C20, C22, C23, C7, C8, J1, R3, R8, R9, U3, U6: moved to F.Cu
- C18, C19, D1, FL1, U1, U4, Y1: moved to B.Cu
- J4: value JST_PH_S2B-PH-SM4-TB_02x2.00mm_Angled -> JST_PH_S6B-PH-SM4-TB_06x2.00mm_Angled; footprint espitall:JST_PH_S2B-PH-SM4-TB_02x2.00mm_Angled -> espitall:JST_PH_S6B-PH-SM4-TB_06x2.00mm_Angled
- J5: value Conn_01x02 -> Conn_01x03; footprint espitall:R_0603_HandSoldering -> espitall:Pin_Header_Straight_1x03_Pitch2.54mm
- J6: footprint Socket_Strips:Socket_Strip_Straight_1x04_Pitch2.54mm -> espitall:Socket_Strip_Straight_1x04_Pitch2.54mm
- J7, J8: value JST_PH_S4B-PH-SM4-TB_04x2.00mm_Angled -> Conn_01x03; footprint espitall:JST_PH_S4B-PH-SM4-TB_04x2.00mm_Angled -> espitall:Pin_Header_Straight_1x03_Pitch2.54mm
- J9: value JST_PH_S2B-PH-SM4-TB_02x2.00mm_Angled -> Conn_01x03; footprint espitall:JST_PH_S2B-PH-SM4-TB_02x2.00mm_Angled -> espitall:Pin_Header_Straight_1x03_Pitch2.54mm
- R12: value 10k -> R; moved to F.Cu
- R2: value 10k -> 200k; moved to B.Cu
- R4: value 1k -> 2k2; moved to B.Cu
- R5: value 10k -> 2k2; moved to B.Cu
- U2: value TSR1-2450 -> PCA9306; footprint espitall:TSR-1 -> espitall:SO-8
- U5: value MC74VHC244DTG -> PCA9685; footprint espitall:TSSOP-20_4.4x6.5mm_Pitch0.65mm -> espitall:TSSOP-28_4.4x9.7mm_Pitch0.65mm; moved to F.Cu
- moved H3 47.3 mm to (54.0, 85.0)
- moved H2 46.0 mm to (54.0, 54.0)
- moved R9 44.0 mm to (61.6, 86.9)
- moved R8 42.4 mm to (61.6, 85.3)
- moved H1 42.0 mm to (96.0, 54.0)
- moved J4 41.9 mm to (77.0, 94.5), turned to 0 degrees
- moved J5 37.5 mm to (92.2, 62.3), turned to 90 degrees
- moved J8 37.2 mm to (92.2, 67.4), turned to 90 degrees
- moved C1 36.0 mm to (59.1, 57.1)
- moved U1 34.0 mm to (63.4, 54.6)
- moved H4 32.9 mm to (85.0, 85.0)
- moved C18 32.8 mm to (80.5, 66.5)
- moved R1 31.7 mm to (67.7, 51.8)
- moved C15 31.0 mm to (53.2, 63.7), turned to 180 degrees
- moved C16 29.6 mm to (70.2, 59.6)
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Connections:
- C22 pad 1: GND -> +3V3
- C22 pad 2: +3V3 -> GND
- C6 pad 1: +BATT -> +5V
- H1 pad 1: (no net) -> Net-(H1-Pad1)
- H2 pad 1: (no net) -> Net-(H2-Pad1)
- H3 pad 1: (no net) -> Net-(H3-Pad1)
- H4 pad 1: (no net) -> Net-(H4-Pad1)
- J1 pad 1: Net-(J1-Pad1) -> +5V
- J2 pad 1: Net-(J1-Pad1) -> +5V
- J3 pad 1: +3V3 -> /uc/pump_1_3v3
- J3 pad 2: /Gyro/mosi_3v3 -> /uc/solenoid_1_3v3
- J3 pad 3: /Gyro/miso_3v3 -> /uc/solenoid_2_3v3
- J3 pad 4: /Gyro/sck_3v3 -> /uc/solenoid_3_3v3
- J3 pad 5: /uc/spi_gyro_~cs~_3v3 -> /uc/solenoid_4_3v3
- J4 pad 1: +BATT -> /uc/pump_2_3v3
- J4 pad 2: GND -> /uc/solenoid_5_3v3
- J5 pad 1: +3V3 -> /Servo/S0
- J5 pad 2: /uc/BOOT0_3v3 -> Net-(J10-Pad2)
- J6 pad 1: +3V3 -> /uc/BOOT0_3v3
- J7 pad 1: +5V -> /Servo/S1
- J7 pad 2: /Encoders/enc_l_A_5v -> Net-(J10-Pad2)
- J7 pad 3: /Encoders/enc_l_B_5v -> GND
- J8 pad 1: +5V -> /Servo/S2
- J8 pad 2: /Encoders/enc_r_A_5v -> Net-(J10-Pad2)
- J8 pad 3: /Encoders/enc_r_B_5v -> GND
- J9 pad 1: /IO/starter_3v3 -> Net-(J9-Pad1)
- J9 pad 2: GND -> Net-(J10-Pad2)
- R10 pad 1: +5V -> Net-(J22-Pad2)
- R10 pad 2: /Encoders/enc_r_A_5v -> /Sensor/ana_2_0-3v3
- R11 pad 1: +5V -> GND
- R11 pad 2: /Encoders/enc_r_B_5v -> /Sensor/ana_2_0-3v3
- R12 pad 1: +3V3 -> Net-(J23-Pad2)
- R12 pad 2: /IO/starter_3v3 -> /Sensor/ana_3_0-3v3
- R13 pad 2: Net-(R13-Pad2) -> /Servo/sda_3v3
- R14 pad 2: Net-(R14-Pad2) -> /Servo/scl_3v3
- R2 pad 1: +BATT -> +5V
- R2 pad 2: /Supply/vbatmon_0-3v3 -> Net-(C24-Pad1)
- R4 pad 1: /Supply/vbatmon_0-3v3 -> +5V
- R4 pad 2: GND -> Net-(R4-Pad2)
- R5 pad 1: /uc/BOOT0_3v3 -> +5V
- R5 pad 2: GND -> Net-(R5-Pad2)
- R8 pad 1: +5V -> Net-(J21-Pad2)
- R8 pad 2: /Encoders/enc_l_A_5v -> /Sensor/ana_1_0-3v3
- R9 pad 1: +5V -> GND
- R9 pad 2: /Encoders/enc_l_B_5v -> /Sensor/ana_1_0-3v3
- U2 pad 1: +BATT -> GND
- U2 pad 2: GND -> +3V3
- U2 pad 3: +5V -> /Servo/scl_3v3
- U4 pad 1: (no net) -> Net-(U4-Pad1)
- U4 pad 15: /Supply/vbatmon_0-3v3 -> Net-(U4-Pad15)
- U4 pad 16: (no net) -> Net-(U4-Pad16)
- U4 pad 17: (no net) -> Net-(U4-Pad17)
- U4 pad 18: (no net) -> Net-(U4-Pad18)
- U4 pad 2: (no net) -> Net-(U4-Pad2)
- U4 pad 23: /Encoders/enc_r_A_3v3 -> Net-(U4-Pad23)
- U4 pad 24: /Encoders/enc_r_B_3v3 -> Net-(U4-Pad24)
- U4 pad 25: (no net) -> Net-(R6-Pad1)
- U4 pad 26: (no net) -> Net-(U4-Pad26)
- U4 pad 29: (no net) -> /Sensor/ana_3_0-3v3
- U4 pad 3: (no net) -> Net-(U4-Pad3)
- U4 pad 30: (no net) -> /Sensor/ana_4_0-3v3
- U4 pad 31: (no net) -> /Sensor/ana_1_0-3v3
- U4 pad 32: (no net) -> /Sensor/ana_2_0-3v3
- U4 pad 33: (no net) -> Net-(U4-Pad33)
- U4 pad 34: (no net) -> Net-(U4-Pad34)
- U4 pad 35: (no net) -> Net-(U4-Pad35)
- U4 pad 36: (no net) -> Net-(U4-Pad36)
- U4 pad 37: GND -> /uc/BOOT1_3v3
- U4 pad 38: (no net) -> Net-(U4-Pad38)
- U4 pad 39: /IO/starter_3v3 -> Net-(U4-Pad39)
- U4 pad 4: (no net) -> Net-(U4-Pad4)
- U4 pad 40: (no net) -> Net-(U4-Pad40)
- U4 pad 41: (no net) -> Net-(U4-Pad41)
- U4 pad 42: (no net) -> Net-(U4-Pad42)
- U4 pad 43: (no net) -> Net-(U4-Pad43)
- U4 pad 44: (no net) -> /uc/pump_2_3v3
- U4 pad 45: (no net) -> /uc/solenoid_5_3v3
- U4 pad 46: (no net) -> /uc/solenoid_6_3v3
- U4 pad 47: (no net) -> /uc/solenoid_7_3v3
- U4 pad 48: (no net) -> /uc/solenoid_8_3v3
- U4 pad 5: (no net) -> Net-(U4-Pad5)
- U4 pad 51: (no net) -> /uc/solenoid_4_3v3
- U4 pad 52: (no net) -> /uc/solenoid_3_3v3
- U4 pad 53: (no net) -> Net-(U4-Pad53)
- U4 pad 54: (no net) -> /uc/solenoid_2_3v3
- U4 pad 55: (no net) -> Net-(U4-Pad55)
- U4 pad 56: (no net) -> Net-(U4-Pad56)
- U4 pad 57: (no net) -> /uc/solenoid_1_3v3
- U4 pad 58: (no net) -> /uc/pump_1_3v3
- U4 pad 59: (no net) -> Net-(U4-Pad59)
- U4 pad 60: (no net) -> Net-(U4-Pad60)
- U4 pad 61: (no net) -> Net-(U4-Pad61)
- U4 pad 62: (no net) -> Net-(U4-Pad62)
- U4 pad 63: (no net) -> Net-(U4-Pad63)
- U4 pad 64: (no net) -> Net-(U4-Pad64)
- U4 pad 65: (no net) -> Net-(U4-Pad65)
- U4 pad 66: (no net) -> Net-(U4-Pad66)
- U4 pad 67: (no net) -> Net-(U4-Pad67)
- U4 pad 7: (no net) -> Net-(U4-Pad7)
- U4 pad 70: (no net) -> Net-(U4-Pad70)
- U4 pad 71: (no net) -> Net-(U4-Pad71)
- U4 pad 72: (no net) -> Net-(U4-Pad72)
- U4 pad 76: (no net) -> Net-(U4-Pad76)
- U4 pad 77: /Encoders/enc_l_A_3v3 -> Net-(U4-Pad77)
- U4 pad 78: /Gyro/sck_3v3 -> Net-(U4-Pad78)
- U4 pad 79: /Gyro/miso_3v3 -> Net-(U4-Pad79)
- U4 pad 8: (no net) -> Net-(U4-Pad8)
- U4 pad 80: /Gyro/mosi_3v3 -> Net-(U4-Pad80)
- U4 pad 81: /CAN/can_tx_3v3 -> /CAN/can_rx_3v3
- U4 pad 82: /CAN/can_rx_3v3 -> /CAN/can_tx_3v3
- U4 pad 83: /uc/spi_gyro_~cs~_3v3 -> Net-(U4-Pad83)
- U4 pad 84: (no net) -> Net-(U4-Pad84)
- U4 pad 85: (no net) -> Net-(U4-Pad85)
- U4 pad 86: (no net) -> Net-(U4-Pad86)
- U4 pad 87: (no net) -> Net-(U4-Pad87)
- U4 pad 88: (no net) -> Net-(U4-Pad88)
- U4 pad 89: /Encoders/enc_l_B_3v3 -> Net-(U4-Pad89)
- U4 pad 9: (no net) -> Net-(U4-Pad9)
- U4 pad 90: (no net) -> Net-(U4-Pad90)
- U4 pad 91: (no net) -> Net-(U4-Pad91)
- U4 pad 92: Net-(R14-Pad2) -> /Servo/scl_3v3
- U4 pad 93: Net-(R13-Pad2) -> /Servo/sda_3v3
- U4 pad 96: Net-(R6-Pad1) -> Net-(U4-Pad96)
- U4 pad 97: (no net) -> Net-(U4-Pad97)
- U4 pad 98: (no net) -> Net-(U4-Pad98)
- U5 pad 1: GND -> +5V
- U5 pad 10: GND -> /Servo/S4
- U5 pad 11: GND -> /Servo/S5
- U5 pad 12: /Encoders/enc_r_B_3v3 -> /Servo/S6
- U5 pad 13: GND -> /Servo/S7
- U5 pad 14: /Encoders/enc_r_A_3v3 -> GND
- U5 pad 15: GND -> /Servo/S8
- U5 pad 16: /Encoders/enc_l_B_3v3 -> /Servo/S9
- U5 pad 17: GND -> /Servo/S10
- U5 pad 18: /Encoders/enc_l_A_3v3 -> /Servo/S11
- U5 pad 19: GND -> /Servo/S12
- U5 pad 2: /Encoders/enc_l_A_5v -> +5V
- U5 pad 20: +3V3 -> Net-(U5-Pad20)
- U5 pad 3: (no net) -> +5V
- U5 pad 4: /Encoders/enc_l_B_5v -> +5V
- U5 pad 5: (no net) -> GND
- U5 pad 6: /Encoders/enc_r_A_5v -> /Servo/S0
- U5 pad 7: (no net) -> /Servo/S1
- U5 pad 8: /Encoders/enc_r_B_5v -> /Servo/S2
- U5 pad 9: (no net) -> /Servo/S3
- U6 pad 1: Net-(R14-Pad2) -> /Servo/scl_3v3
- U6 pad 3: Net-(R13-Pad2) -> /Servo/sda_3v3
- U6 pad 5: Net-(U4-Pad95) -> Net-(U4-Pad77)
Routing:
- net /Encoders/enc_l_A_5v: track 70.1 -> 0.00 mm, vias 1 -> 0
- net /Encoders/enc_l_B_5v: track 65.0 -> 0.00 mm, vias 1 -> 0
- net +3V3: track 169.1 -> 106.5 mm, vias 13 -> 8
- net /Supply/vbatmon_0-3v3: track 56.7 -> 0.00 mm, vias 6 -> 0
- net /Encoders/enc_r_B_3v3: track 47.3 -> 0.00 mm, vias 3 -> 0
- net /Encoders/enc_r_A_3v3: track 46.3 -> 0.00 mm, vias 3 -> 0
- net Net-(R5-Pad2): track 0.00 -> 41.0 mm, vias 0 -> 2
- net Net-(R4-Pad2): track 0.00 -> 38.3 mm, vias 0 -> 2
- net /uc/solenoid_8_3v3: track 0.00 -> 36.7 mm, vias 0 -> 1
- net /uc/solenoid_7_3v3: track 0.00 -> 33.4 mm, vias 0 -> 1
- net /uc/solenoid_6_3v3: track 0.00 -> 30.4 mm, vias 0 -> 1
- net +5V: track 63.1 -> 92.3 mm, vias 1 -> 7
- net /uc/solenoid_5_3v3: track 0.00 -> 27.4 mm, vias 0 -> 1
- net /uc/pump_1_3v3: track 0.00 -> 24.9 mm, vias 0 -> 1
- net /Servo/S12: track 0.00 -> 24.6 mm, vias 0 -> 1
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Other:
- board size 54 x 50 mm -> 50 x 50 mm
- board text added: "A1"
- board text added: "A2"
- board text added: "A3"
- board text added: "A4"
- board text added: "Cocobot"
- board text added: "MECA 2019"
- board text added: "P1"
- board text added: "P2"
- board text added: "S"
- board text added: "S0"
- board text added: "S1"
- board text added: "S10"
- board text added: "S11"
- board text added: "S12"
- board text added: "S2"
- board text added: "S3"
- board text added: "S4"
- board text added: "S5"
- board text added: "S6"
- board text added: "S7"
- board text added: "S8"
- board text added: "S9"
- board text removed: "Brain 2019 Cocobot"
- board text removed: "CAN"
- board text removed: "ENC L"
- board text removed: "ENC R"
- board text removed: "Gyro"
- board text removed: "PWR"
- board text removed: "Starter"
