File: meca_2019/sensor.sch (KiCad schematic (older format))
At the start: 16 parts, among them J21 Conn_01x03, J22 Conn_01x03, J23 Conn_01x03, J24 Conn_01x03

Commit message: meca 2019 board
Parts:
- J21, J22, J23, J24: footprint (none) -> espitall:Pin_Header_Straight_1x03_Pitch2.54mm
Changed lines of the file:
@@
 F 0 "J21" H 1730 1742 50  0000 L CNN
 F 1 "Conn_01x03" H 1730 1651 50  0000 L CNN
-F 2 "" H 1650 1700 50  0001 C CNN
+F 2 "espitall:Pin_Header_Straight_1x03_Pitch2.54mm" H 1650 1700 50  0001 C CNN
 F 3 "~" H 1650 1700 50  0001 C CNN
 	1    1650 1700
@@
 F 0 "J22" H 1730 2892 50  0000 L CNN
 F 1 "Conn_01x03" H 1730 2801 50  0000 L CNN
-F 2 "" H 1650 2850 50  0001 C CNN
+F 2 "espitall:Pin_Header_Straight_1x03_Pitch2.54mm" H 1650 2850 50  0001 C CNN
 F 3 "~" H 1650 2850 50  0001 C CNN
 	1    1650 2850
@@
 F 0 "J23" H 1730 4092 50  0000 L CNN
 F 1 "Conn_01x03" H 1730 4001 50  0000 L CNN
-F 2 "" H 1650 4050 50  0001 C CNN
+F 2 "espitall:Pin_Header_Straight_1x03_Pitch2.54mm" H 1650 4050 50  0001 C CNN
 F 3 "~" H 1650 4050 50  0001 C CNN
 	1    1650 4050
@@
 F 0 "J24" H 1730 5292 50  0000 L CNN
 F 1 "Conn_01x03" H 1730 5201 50  0000 L CNN
-F 2 "" H 1650 5250 50  0001 C CNN
+F 2 "espitall:Pin_Header_Straight_1x03_Pitch2.54mm" H 1650 5250 50  0001 C CNN
 F 3 "~" H 1650 5250 50  0001 C CNN
 	1    1650 5250
