File: meca_2019/servo.sch (KiCad schematic (older format))
At the start: 23 parts, among them J10 Conn_01x03, J11 Conn_01x03, J12 Conn_01x03, J13 Conn_01x03, J14 Conn_01x03, J15 Conn_01x03, J16 Conn_01x03, J17 Conn_01x03, J18 Conn_01x03, J19 Conn_01x03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

Commit message: meca 2019 board
Parts:
- J10, J11, J12, J13, J14, J15, J16, J17, J18, J19, J20, J5, J7, J8, J9: footprint (none) -> espitall:Pin_Header_Straight_1x03_Pitch2.54mm
- R2: footprint (none) -> espitall:R_0603
- U2: footprint (none) -> espitall:SO-8
- U5: footprint (none) -> espitall:TSSOP-28_4.4x9.7mm_Pitch0.65mm
Connections:
- wire segments 153 -> 156
