File: canon_2019/control.sch (KiCad schematic (older format))
At the start: 21 parts

Commit message: canon 2019 layout (2 layers)
Parts:
- removed C? (x2): 22p, symbol Device:C
- removed Y?: 8M, symbol Device:Crystal
- added C4: 100n, espitall:C_0603, symbol Device:C
- added J3: CocobotCAN, espitall:JST_PH_S5B-PH-SM4-TB_05x2.00mm_Angled, symbol espitall:CocobotCAN
- added U2: MAX3051, Housings_SOIC:SOIC-8_3.9x4.9mm_Pitch1.27mm, symbol Interface_UART:MAX3051
- C12, C13, C5, C6, C7, C8, C9: renamed from C?; footprint (none) -> espitall:C_0603
- D3: renamed from D?; footprint (none) -> espitall:LED_0805
- J4: renamed from J?; footprint (none) -> Pin_Headers:Pin_Header_Straight_1x04_Pitch2.54mm
- R10, R11, R5, R6, R7, R8, R9: renamed from R?; footprint (none) -> espitall:R_0603
- U3: renamed from U?; footprint Package_QFP:LQFP-64_10x10mm_P0.5mm -> Housings_QFP:LQFP-64_10x10mm_Pitch0.5mm
- U4: renamed from U?; footprint TO_SOT_Packages_SMD:SOT-323_SC-70 -> TO_SOT_Packages_SMD:SOT-353_SC-70-5
Connections:
- net labels added: can_rx, can_tx
- wire segments 105 -> 136
