File: canon_2019/phase.sch (KiCad schematic (older format))
At the start: 10 parts

Commit message: schematic of canon board 2019
Parts:
- added C?: 100n, symbol Device:C
- added R? (x2): 5m, Resistors_SMD:R_1206, symbol Device:R
- added U?: INA240A1PW, Package_SO:TSSOP-8_4.4x3mm_P0.65mm, symbol Amplifier_Current:INA240A1PW
Connections:
- net labels added: +3V3, I_0-3v3, PH, REF_1v65
- wire segments 53 -> 82
Other:
- note added: "Current monitor"
- note added: "Driver\n"
- note added: "Half bridge"

Commit message: canon 2019 layout (2 layers)
Parts:
- C16, C17, C18: renamed from C?; footprint (none) -> espitall:C_0603
- D4, D5, D6: renamed from D?; footprint (none) -> Diodes_SMD:D_SOD-523
- Q3, Q4: renamed from Q?; footprint (none) -> TO_SOT_Packages_SMD:SOT-669_LFPAK
- R12, R15: renamed from R?; footprint (none) -> espitall:R_0603
- U5: renamed from U?; footprint (none) -> espitall:SOIC-8_3.9x4.9mm_Pitch1.27mm
- U6: renamed from U?; footprint Package_SO:TSSOP-8_4.4x3mm_P0.65mm -> Housings_SSOP:TSSOP-8_4.4x3mm_Pitch0.65mm
- gave numbers to parts that had none: 2
