File: pompette_2019/pompette_2019.kicad_pcb (KiCad board)
At the start: 2 copper layers, 34 x 50 mm, 45 parts, among them J1 Conn_01x01, J2 Conn_01x02, J3 Conn_01x01, J4 Conn_01x02, J5 Conn_01x02, J6 JST_PH_S6B-PH-SM4-TB_06x2.00m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, J7 Conn_01x02, J8 Conn_01x02, Q1 DMG4466SSS-13, Q2 DMG4466SSS-13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

Commit message: Layout of Pompette 2019
Parts:
- moved J2 2.60 mm to (79.0, 93.7), turned to 90 degrees
Routing:
- net +BATT: track 20.5 -> 88.8 mm, vias 0 -> 1
- net GND: track 50.1 -> 98.6 mm, vias 0 -> 15
- net Net-(D1-Pad2): track 0.00 -> 26.4 mm
- net Net-(D3-Pad2): track 0.00 -> 22.9 mm
- net Net-(D4-Pad2): track 0.00 -> 22.8 mm
- net Net-(D2-Pad2): track 0.00 -> 22.4 mm
- net Net-(D5-Pad2): track 0.00 -> 22.3 mm
- net Net-(D5-Pad1): track 0.00 -> 12.0 mm
- net Net-(D4-Pad1): track 0.00 -> 11.0 mm
- net Net-(D3-Pad1): track 0.00 -> 10.6 mm
- net Net-(D2-Pad1): track 0.00 -> 10.6 mm
- added copper zone on F.Cu, net +BATT
- added copper zone on B.Cu, net GND
- added copper zone on F.Cu, net GND
- added copper zone on F.Cu, net Net-(D1-Pad2)
- added copper zone on F.Cu, net Net-(D2-Pad1)
- added copper zone on F.Cu, net Net-(D2-Pad2)
- added copper zone on F.Cu, net Net-(D3-Pad1)
- added copper zone on F.Cu, net Net-(D3-Pad2)
- added copper zone on F.Cu, net Net-(D4-Pad1)
- added copper zone on F.Cu, net Net-(D4-Pad2)
- added copper zone on F.Cu, net Net-(D5-Pad1)
- added copper zone on F.Cu, net Net-(D5-Pad2)
Other:
- board text added: "GND"
- board text added: "P1"
- board text added: "Pompette 2019 Cocobot"
- board text added: "S1"
- board text added: "S2"
- board text added: "S3"
- board text added: "S4"
- board text added: "Vbat"

Commit message: Modifications after review
Parts:
- added R20: 470k, espitall:R_0603, B.Cu at (75.7, 73.5)
- added R21: 470k, espitall:R_0603, B.Cu at (54.6, 73.6)
- added R22: 470k, espitall:R_0603, B.Cu at (65.8, 73.6)
- added R23: 470k, espitall:R_0603, F.Cu at (63.0, 73.7)
- added R24: 470k, espitall:R_0603, F.Cu at (75.0, 73.5)
- R1, R15, R16, R7, R8: value 10k -> 1k
- R10, R11, R18, R19, R3: value 1k -> 10k
Routing:
- net Net-(R23-Pad2): track 0.00 -> 3.83 mm
- net Net-(Q5-PadG): track 6.40 -> 9.75 mm
- net Net-(R20-Pad2): track 0.00 -> 2.67 mm
- net Net-(R22-Pad2): track 0.00 -> 2.64 mm
- net Net-(Q4-PadG): track 6.87 -> 9.43 mm
- net Net-(R21-Pad2): track 0.00 -> 2.39 mm
- net Net-(R24-Pad2): track 0.00 -> 2.31 mm
- net Net-(Q1-PadG): track 10.9 -> 12.7 mm, vias 1 -> 2
- net Net-(Q2-PadG): track 16.8 -> 18.3 mm, vias 1 -> 2
- net Net-(Q3-PadG): track 14.6 -> 15.3 mm, vias 1 -> 2
