File: pompette_2019/pompette_2019.sch (KiCad schematic (older format))
At the start: 46 parts, among them J1 Conn_01x01, J2 Conn_01x02, J3 Conn_01x01, J4 Conn_01x02, J5 Conn_01x02, J6 JST_PH_S6B-PH-SM4-TB_06x2.00m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, J7 Conn_01x02, J8 Conn_01x02, Q1 DMG4466SSS-13, Q2 DMG4466SSS-13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

Commit message: Modifications after review
Parts:
- added R20, R21, R22, R23, R24: 470k, espitall:R_0603, symbol Device:R
- R1, R15, R16, R7, R8: value 10k -> 1k
- R10, R11, R18, R19, R3: value 1k -> 10k
Connections:
- wire segments 137 -> 177
Changed lines of the file:
@@
 P 6550 1800
 F 0 "R3" H 6620 1846 50  0000 L CNN
-F 1 "1k" H 6620 1755 50  0000 L CNN
+F 1 "10k" H 6620 1755 50  0000 L CNN
 F 2 "espitall:R_0603" V 6480 1800 50  0001 C CNN
 F 3 "~" H 6550 1800 50  0001 C CNN
@@
 $EndComp
 Wire Wire Line
-	6250 1550 6550 1550
+	6250 1550 6400 1550
 Wire Wire Line
 	6550 1650 6550 1550
@@
 P 6550 1000
 F 0 "R1" H 6620 1046 50  0000 L CNN
-F 1 "10k" H 6620 955 50  0000 L CNN
+F 1 "1k" H 6620 955 50  0000 L CNN
 F 2 "espitall:R_0603" V 6480 1000 50  0001 C CNN
 F 3 "~" H 6550 1000 50  0001 C CNN
@@
 P 6550 4000
 F 0 "R10" H 6620 4046 50  0000 L CNN
-F 1 "1k" H 6620 3955 50  0000 L CNN
+F 1 "10k" H 6620 3955 50  0000 L CNN
 F 2 "espitall:R_0603" V 6480 4000 50  0001 C CNN
 F 3 "~" H 6550 4000 50  0001 C CNN
@@
 $EndComp
 Wire Wire Line
-	6250 3750 6550 3750
+	6250 3750 6400 3750
 Wire Wire Line
 	6550 3850 6550 3750
@@
 P 6550 3200
 F 0 "R7" H 6620 3246 50  0000 L CNN
-F 1 "10k" H 6620 3155 50  0000 L CNN
+F 1 "1k" H 6620 3155 50  0000 L CNN
 F 2 "espitall:R_0603" V 6480 3200 50  0001 C CNN
 F 3 "~" H 6550 3200 50  0001 C CNN
@@
 P 9750 4000
 F 0 "R11" H 9820 4046 50  0000 L CNN
-F 1 "1k" H 9820 3955 50  0000 L CNN
+F 1 "10k" H 9820 3955 50  0000 L CNN
 F 2 "espitall:R_0603" V 9680 4000 50  0001 C CNN
 F 3 "~" H 9750 4000 50  0001 C CNN
@@
 	1    0    0    -1
 $EndComp
-Wire Wire Line
-	9450 3750 9750 3750
 Wire Wire Line
 	9750 3850 9750 3750
@@
 P 9750 3200
 F 0 "R8" H 9820 3246 50  0000 L CNN
-F 1 "10k" H 9820 3155 50  0000 L CNN
+F 1 "1k" H 9820 3155 50  0000 L CNN
 F 2 "espitall:R_0603" V 9680 3200 50  0001 C CNN
 F 3 "~" H 9750 3200 50  0001 C CNN
@@
 P 6550 6200
 F 0 "R18" H 6620 6246 50  0000 L CNN
-F 1 "1k" H 6620 6155 50  0000 L CNN
+F 1 "10k" H 6620 6155 50  0000 L CNN
 F 2 "espitall:R_0603" V 6480 6200 50  0001 C CNN
 F 3 "~" H 6550 6200 50  0001 C CNN
@@
 	1    0    0    -1
 $EndComp
-Wire Wire Line
-	6250 5950 6550 5950
 Wire Wire Line
 	6550 6050 6550 5950
@@
 P 6550 5400
 F 0 "R15" H 6620 5446 50  0000 L CNN
-F 1 "10k" H 6620 5355 50  0000 L CNN
+F 1 "1k" H 6620 5355 50  0000 L CNN
 F 2 "espitall:R_0603" V 6480 5400 50  0001 C CNN
 F 3 "~" H 6550 5400 50  0001 C CNN
@@
 P 9750 6200
 F 0 "R19" H 9820 6246 50  0000 L CNN
-F 1 "1k" H 9820 6155 50  0000 L CNN
+F 1 "10k" H 9820 6155 50  0000 L CNN
 F 2 "espitall:R_0603" V 9680 6200 50  0001 C CNN
 F 3 "~" H 9750 6200 50  0001 C CNN
@@
 	1    0    0    -1
 $EndComp
-Wire Wire Line
-	9450 5950 9750 5950
 Wire Wire Line
 	9750 6050 9750 5950
@@
 P 9750 5400
 F 0 "R16" H 9820 5446 50  0000 L CNN
-F 1 "10k" H 9820 5355 50  0000 L CNN
+F 1 "1k" H 9820 5355 50  0000 L CNN
 F 2 "espitall:R_0603" V 9680 5400 50  0001 C CNN
 F 3 "~" H 9750 5400 50  0001 C CNN
@@
 	-1   0    0    1
 $EndComp
+$Comp
+L Device:R R20
+U 1 1 5C94336B
+P 6150 1800
+F 0 "R20" H 6220 1846 50  0000 L CNN
+F 1 "470k" H 6220 1755 50  0000 L CNN
+F 2 "espitall:R_0603" V 6080 1800 50  0001 C CNN
+F 3 "~" H 6150 1800 50  0001 C CNN
+	1    6150 1800
+	0    1    1    0
+$EndComp
+Wire Wire Line
+	6300 1800 6400 1800
+Wire Wire Line
+	6400 1800 6400 1550
+Connection ~ 6400 1550
+Wire Wire Line
+	6400 1550 6550 1550
+Wire Wire Line
+	6250 1350 6300 1350
+Wire Wire Line
+	6300 1350 6300 1700
+Wire Wire Line
+	6300 1700 5950 1700
+Wire Wire Line
+	5950 1700 5950 1800
+Wire Wire Line
+	5950 1800 6000 1800
+$Comp
+L Device:R R21
+U 1 1 5C9547BD
+P 6150 4000
+F 0 "R21" H 6220 4046 50  0000 L CNN
+F 1 "470k" H 6220 3955 50  0000 L CNN
+F 2 "espitall:R_0603" V 6080 4000 50  0001 C CNN
+F 3 "~" H 6150 4000 50  0001 C CNN
+	1    6150 4000
+	0    1    1    0
+$EndComp
+Wire Wire Line
+	6300 4000 6400 4000
+Wire Wire Line
+	6400 4000 6400 3750
+Wire Wire Line
+	6300 3550 6300 3900
+Wire Wire Line
+	6300 3900 5950 3900
+Wire Wire Line
+	5950 3900 5950 4000
+Wire Wire Line
+	5950 4000 6000 4000
+$Comp
+L Device:R R22
+U 1 1 5C95AA5E
+P 9350 4000
+F 0 "R22" H 9420 4046 50  0000 L CNN
+F 1 "470k" H 9420 3955 50  0000 L CNN
+F 2 "espitall:R_0603" V 9280 4000 50  0001 C CNN
+F 3 "~" H 9350 4000 50  0001 C CNN
+	1    9350 4000
+	0    1    1    0
+$EndComp
+Wire Wire Line
+	9500 4000 9600 4000
+Wire Wire Line
+	9600 4000 9600 3750
+Wire Wire Line
+	9500 3550 9500 3900
+Wire Wire Line
+	9500 3900 9150 3900
+Wire Wire Line
+	9150 3900 9150 4000
+Wire Wire Line
+	9150 4000 9200 4000
+$Comp
+L Device:R R23
+U 1 1 5C961594
+P 6150 6200
+F 0 "R23" H 6220 6246 50  0000 L CNN
+F 1 "470k" H 6220 6155 50  0000 L CNN
+F 2 "espitall:R_0603" V 6080 6200 50  0001 C CNN
+F 3 "~" H 6150 6200 50  0001 C CNN
+	1    6150 6200
+	0    1    1    0
+$EndComp
+Wire Wire Line
+	6300 6200 6400 6200
+Wire Wire Line
+	6400 6200 6400 5950
+Wire Wire Line
+	6300 5750 6300 6100
+Wire Wire Line
+	6300 6100 5950 6100
+Wire Wire Line
+	5950 6100 5950 6200
+Wire Wire Line
+	5950 6200 6000 6200
+$Comp
+L Device:R R24
+U 1 1 5C9688B0
+P 9350 6200
+F 0 "R24" H 9420 6246 50  0000 L CNN
+F 1 "470k" H 9420 6155 50  0000 L CNN
+F 2 "espitall:R_0603" V 9280 6200 50  0001 C CNN
+F 3 "~" H 9350 6200 50  0001 C CNN
+	1    9350 6200
+	0    1    1    0
+$EndComp
+Wire Wire Line
+	9500 6200 9600 6200
+Wire Wire Line
+	9600 6200 9600 5950
+Wire Wire Line
+	9500 5750 9500 6100
+Wire Wire Line
+	9500 6100 9150 6100
+Wire Wire Line
+	9150 6100 9150 6200
+Wire Wire Line
+	9150 6200 9200 6200
+Wire Wire Line
+	9500 5750 9450 5750
+Wire Wire Line
+	6300 5750 6250 5750
+Wire Wire Line
+	6250 5950 6400 5950
+Connection ~ 6400 5950
+Wire Wire Line
+	6400 5950 6550 5950
+Wire Wire Line
+	9450 5950 9600 5950
+Connection ~ 9600 5950
+Wire Wire Line
+	9600 5950 9750 5950
+Wire Wire Line
+	9450 3550 9500 3550
+Wire Wire Line
+	9450 3750 9600 3750
+Connection ~ 9600 3750
+Wire Wire Line
+	9600 3750 9750 3750
+Wire Wire Line
+	6400 3750 6550 3750
+Connection ~ 6400 3750
+Wire Wire Line
+	6300 3550 6250 3550
 $EndSCHEMATC
